File: pcb/badge/badge.sch (KiCad schematic (older format))
At the start: 1 part

Commit message: feat: add some initial connections to the mp3 player module
Parts:
- added C? (x2): 33pF, symbol Device:C
- added R?: 1M, symbol Device:R
- added Y?: 12.288M, symbol Device:Crystal
Connections:
- net labels added: +1V8, +3V3, GND, GNDA, GNDD, LEFT, RIGHT, VDDA
- wire segments 0 -> 47
Other:
- moved on the sheet: IC?

Commit message: feat: add audio jack (TRRS) connector
also assign footprints to symbols
Parts:
- added J1: AudioJack4_Ground, Connector_Audio:Jack_3.5mm_PJ320D_Horizontal, symbol Connector:AudioJack4_Ground
- C1, C2: renamed from C?; footprint (none) -> Capacitor_SMD:C_0603_1608Metric
- IC1: renamed from IC?; footprint QFP50P900X900X160-48N -> COM-08892:QFP50P900X900X160-48N
- R1: renamed from R?; footprint (none) -> Resistor_SMD:R_0603_1608Metric
- Y1: renamed from Y?; footprint (none) -> Crystal:Crystal_SMD_3225-4Pin_3.2x2.5mm
Connections:
- net labels added: GBUF
- wire segments 47 -> 51
Changed lines of the file:
@@
 EESchema Schematic File Version 4
+LIBS:badge-cache
 EELAYER 26 0
 EELAYER END
@@
 $EndDescr
 $Comp
-L COM-08892:COM-08892 IC?
+L COM-08892:COM-08892 IC1
 U 1 1 5BF74A63
 P 7950 1950
-F 0 "IC?" H 10391 1296 50  0000 L CNN
+F 0 "IC1" H 10391 1296 50  0000 L CNN
 F 1 "COM-08892" H 10391 1205 50  0000 L CNN
-F 2 "QFP50P900X900X160-48N" H 10200 2450 50  0001 L CNN
+F 2 "COM-08892:QFP50P900X900X160-48N" H 10200 2450 50  0001 L CNN
 F 3 "https://www.google.co.jp/url?sa=t&rct=j&q=&esrc=s&source=web&cd=1&cad=rja&uact=8&ved=0ahUKEwiAkKC8ipDWAhWEWrwKHciZB0kQFggpMAA&url=https%3A%2F%2Fwww.sparkfun.com%2Fdatasheets%2FComponents%2FSMD%2Fvs1053.pdf&usg=AFQjCNGfjeIOxgMtdfoxEnZ7Zp1IsEDwzA" H 10200 2350 50  0001 L CNN
 F 4 "SparkFun Accessories MP3 and MIDI Codec - VS1053B" H 10200 2250 50  0001 L CNN "Description"
@@
 Connection ~ 9350 4150
 $Comp
-L power:GNDD #PWR?
+L power:GNDD #PWR0101
 U 1 1 5BF74F90
 P 9350 4250
-F 0 "#PWR?" H 9350 4000 50  0001 C CNN
+F 0 "#PWR0101" H 9350 4000 50  0001 C CNN
 F 1 "GNDD" H 9354 4095 50  0000 C CNN
 F 2 "" H 9350 4250 50  0001 C CNN
@@
 	7950 2250 7700 2250
 $Comp
-L power:GNDD #PWR?
+L power:GNDD #PWR0102
 U 1 1 5BF751E2
 P 7700 2250
-F 0 "#PWR?" H 7700 2000 50  0001 C CNN
+F 0 "#PWR0102" H 7700 2000 50  0001 C CNN
 F 1 "GNDD" V 7704 2140 50  0000 R CNN
 F 2 "" H 7700 2250 50  0001 C CNN
@@
 $EndComp
 $Comp
-L power:+3V3 #PWR?
+L power:+3V3 #PWR0103
 U 1 1 5BF752EA
 P 10600 2350
-F 0 "#PWR?" H 10600 2200 50  0001 C CNN
+F 0 "#PWR0103" H 10600 2200 50  0001 C CNN
 F 1 "+3V3" V 10615 2478 50  0000 L CNN
 F 2 "" H 10600 2350 50  0001 C CNN
@@
 	10600 2350 10350 2350
 $Comp
-L power:+1V8 #PWR?
+L power:+1V8 #PWR0104
 U 1 1 5BF753E2
 P 10600 2450
-F 0 "#PWR?" H 10600 2300 50  0001 C CNN
+F 0 "#PWR0104" H 10600 2300 50  0001 C CNN
 F 1 "+1V8" V 10615 2578 50  0000 L CNN
 F 2 "" H 10600 2450 50  0001 C CNN
@@
 	7950 2450 7700 2450
 $Comp
-L power:+3V3 #PWR?
+L power:+3V3 #PWR0105
 U 1 1 5BF75578
 P 7700 2450
-F 0 "#PWR?" H 7700 2300 50  0001 C CNN
+F 0 "#PWR0105" H 7700 2300 50  0001 C CNN
 F 1 "+3V3" V 7715 2578 50  0000 L CNN
 F 2 "" H 7700 2450 50  0001 C CNN
@@
 $EndComp
 $Comp
-L power:+1V8 #PWR?
+L power:+1V8 #PWR0106
 U 1 1 5BF7562E
 P 7700 2350
-F 0 "#PWR?" H 7700 2200 50  0001 C CNN
+F 0 "#PWR0106" H 7700 2200 50  0001 C CNN
 F 1 "+1V8" V 7715 2478 50  0000 L CNN
 F 2 "" H 7700 2350 50  0001 C CNN
@@
 	7800 2350 7950 2350
 $Comp
-L power:+1V8 #PWR?
+L power:+1V8 #PWR0107
 U 1 1 5BF75901
 P 9650 4250
-F 0 "#PWR?" H 9650 4100 50  0001 C CNN
+F 0 "#PWR0107" H 9650 4100 50  0001 C CNN
 F 1 "+1V8" H 9665 4423 50  0000 C CNN
 F 2 "" H 9650 4250 50  0001 C CNN
@@
 	9650 4250 9650 4050
 $Comp
-L power:+3V3 #PWR?
+L power:+3V3 #PWR0108
 U 1 1 5BF75AF4
 P 8650 4250
-F 0 "#PWR?" H 8650 4100 50  0001 C CNN
+F 0 "#PWR0108" H 8650 4100 50  0001 C CNN
 F 1 "+3V3" H 8665 4423 50  0000 C CNN
 F 2 "" H 8650 4250 50  0001 C CNN
@@
 	9250 1250 9250 1100
 $Comp
-L power:GNDA #PWR?
+L power:GNDA #PWR0109
 U 1 1 5BF76469
 P 9250 950
-F 0 "#PWR?" H 9250 700 50  0001 C CNN
+F 0 "#PWR0109" H 9250 700 50  0001 C CNN
 F 1 "GNDA" H 9255 777 50  0000 C CNN
 F 2 "" H 9250 950 50  0001 C CNN
@@
 RIGHT
 $Comp
-L power:GNDA #PWR?
+L power:GNDA #PWR0110
 U 1 1 5BF778A7
 P 8650 950
-F 0 "#PWR?" H 8650 700 50  0001 C CNN
+F 0 "#PWR0110" H 8650 700 50  0001 C CNN
 F 1 "GNDA" H 8655 777 50  0000 C CNN
 F 2 "" H 8650 950 50  0001 C CNN
@@
 	9250 1100 9250 950
 $Comp
-L power:GNDA #PWR?
+L power:GNDA #PWR0111
 U 1 1 5BF7800C
 P 9650 950
-F 0 "#PWR?" H 9650 700 50  0001 C CNN
+F 0 "#PWR0111" H 9650 700 50  0001 C CNN
 F 1 "GNDA" H 9655 777 50  0000 C CNN
 F 2 "" H 9650 950 50  0001 C CNN
@@
 	9650 950  9650 1250
 $Comp
-L power:VDDA #PWR?
+L power:VDDA #PWR0112
 U 1 1 5BF7874B
 P 9550 1100
-F 0 "#PWR?" H 9550 950 50  0001 C CNN
+F 0 "#PWR0112" H 9550 950 50  0001 C CNN
 F 1 "VDDA" H 9567 1273 50  0000 C CNN
 F 2 "" H 9550 1100 50  0001 C CNN
@@
 	9550 1100 9550 1250
 $Comp
-L power:VDDA #PWR?
+L power:VDDA #PWR0113
 U 1 1 5BF78A5D
 P 8950 850
-F 0 "#PWR?" H 8950 700 50  0001 C CNN
+F 0 "#PWR0113" H 8950 700 50  0001 C CNN
 F 1 "VDDA" H 8967 1023 50  0000 C CNN
 F 2 "" H 8950 850 50  0001 C CNN
@@
 	9050 4050 9050 4500
 $Comp
-L Device:R R?
+L Device:R R1
 U 1 1 5BF7A612
 P 9000 4650
-F 0 "R?" V 8900 4650 50  0000 C CNN
+F 0 "R1" V 8900 4650 50  0000 C CNN
 F 1 "1M" V 9000 4650 50  0000 C CNN
-F 2 "" V 8930 4650 50  0001 C CNN
+F 2 "Resistor_SMD:R_0603_1608Metric" V 8930 4650 50  0001 C CNN
 F 3 "~" H 9000 4650 50  0001 C CNN
 	1    9000 4650
@@
 	9150 4500 9150 4650
 $Comp
-L Device:Crystal Y?
+L Device:Crystal Y1
 U 1 1 5BF7CBFA
 P 9000 4900
-F 0 "Y?" H 9000 4900 50  0000 C CNN
+F 0 "Y1" H 9000 4900 50  0000 C CNN
 F 1 "12.288M" H 9000 4750 50  0000 C CNN
-F 2 "" H 9000 4900 50  0001 C CNN
+F 2 "Crystal:Crystal_SMD_3225-4Pin_3.2x2.5mm" H 9000 4900 50  0001 C CNN
 F 3 "~" H 9000 4900 50  0001 C CNN
 	1    9000 4900
@@
 Connection ~ 8850 4650
 $Comp
-L Device:C C?
+L Device:C C2
 U 1 1 5BF7E640
 P 9300 4900
-F 0 "C?" H 9415 4946 50  0000 L CNN
+F 0 "C2" H 9415 4946 50  0000 L CNN
 F 1 "33pF" H 9415 4855 50  0000 L CNN
-F 2 "" H 9338 4750 50  0001 C CNN
+F 2 "Capacitor_SMD:C_0603_1608Metric" H 9338 4750 50  0001 C CNN
 F 3 "~" H 9300 4900 50  0001 C CNN
 	1    9300 4900
@@
 $EndComp
 $Comp
-L Device:C C?
+L Device:C C1
 U 1 1 5BF7E6E4
 P 8700 4900
-F 0 "C?" H 8500 4950 50  0000 L CNN
+F 0 "C1" H 8500 4950 50  0000 L CNN
 F 1 "33pF" H 8400 4850 50  0000 L CNN
-F 2 "" H 8738 4750 50  0001 C CNN
+F 2 "Capacitor_SMD:C_0603_1608Metric" H 8738 4750 50  0001 C CNN
 F 3 "~" H 8700 4900 50  0001 C CNN
 	1    8700 4900
@@
 	8700 5200 8700 5050
 $Comp
-L power:GND #PWR?
+L power:GND #PWR0114
 U 1 1 5BF8086D
 P 9000 5200
-F 0 "#PWR?" H 9000 4950 50  0001 C CNN
+F 0 "#PWR0114" H 9000 4950 50  0001 C CNN
 F 1 "GND" H 9005 5027 50  0000 C CNN
 F 2 "" H 9000 5200 50  0001 C CNN
@@
 	9000 5200 8700 5200
 Connection ~ 9000 5200
+$Comp
+L Connector:AudioJack4_Ground J1
+U 1 1 5BF87719
+P 7050 1200
+F 0 "J1" H 7016 1542 50  0000 C CNN
+F 1 "AudioJack4_Ground" H 7016 1451 50  0000 C CNN
+F 2 "Connector_Audio:Jack_3.5mm_PJ320D_Horizontal" H 7050 1200 50  0001 C CNN
+F 3 "~" H 7050 1200 50  0001 C CNN
+	1    7050 1200
+	0    1    1    0
+$EndComp
+Wire Wire Line
+	6850 1400 6850 1700
+Text Label 6850 1700 1    50   ~ 0
+LEFT
+Wire Wire Line
+	6950 1400 6950 1700
+Text Label 6950 1700 1    50   ~ 0
+RIGHT
+Wire Wire Line
+	9150 1250 9150 1050
+Text Label 9150 1250 1    50   ~ 0
+GBUF
+Wire Wire Line
+	7050 1400 7050 1700
+Text Label 7050 1700 1    50   ~ 0
+GBUF
 $EndSCHEMATC

Commit message: Add MP3 breakout
Parts:
- added J?: Conn_01x08_Male, symbol Connector:Conn_01x08_Male
Connections:
- net labels added: DREQ, MISO, MOSI, SCLK, XRESET, xCS, xDCS
- wire segments 51 -> 66
Changed lines of the file:
@@
 EESchema Schematic File Version 4
-LIBS:badge-cache
 EELAYER 26 0
 EELAYER END
@@
 U 1 1 5BF74A63
 P 7950 1950
-F 0 "IC1" H 10391 1296 50  0000 L CNN
-F 1 "COM-08892" H 10391 1205 50  0000 L CNN
+F 0 "IC1" H 9100 1500 50  0000 L CNN
+F 1 "COM-08892" H 8950 1600 50  0000 L CNN
 F 2 "COM-08892:QFP50P900X900X160-48N" H 10200 2450 50  0001 L CNN
 F 3 "https://www.google.co.jp/url?sa=t&rct=j&q=&esrc=s&source=web&cd=1&cad=rja&uact=8&ved=0ahUKEwiAkKC8ipDWAhWEWrwKHciZB0kQFggpMAA&url=https%3A%2F%2Fwww.sparkfun.com%2Fdatasheets%2FComponents%2FSMD%2Fvs1053.pdf&usg=AFQjCNGfjeIOxgMtdfoxEnZ7Zp1IsEDwzA" H 10200 2350 50  0001 L CNN
@@
 Text Label 7050 1700 1    50   ~ 0
 GBUF
+$Comp
+L Connector:Conn_01x08_Male J?
+U 1 1 5C0E7589
+P 5100 3400
+F 0 "J?" H 5206 3878 50  0000 C CNN
+F 1 "Conn_01x08_Male" H 5206 3787 50  0000 C CNN
+F 2 "" H 5100 3400 50  0001 C CNN
+F 3 "~" H 5100 3400 50  0001 C CNN
+	1    5100 3400
+	1    0    0    -1
+$EndComp
+$Comp
+L power:GND #PWR?
+U 1 1 5C0E8288
+P 5700 3100
+F 0 "#PWR?" H 5700 2850 50  0001 C CNN
+F 1 "GND" V 5705 2972 50  0000 R CNN
+F 2 "" H 5700 3100 50  0001 C CNN
+F 3 "" H 5700 3100 50  0001 C CNN
+	1    5700 3100
+	0    -1   -1   0
+$EndComp
+Wire Wire Line
+	5300 3100 5700 3100
+Wire Wire Line
+	5300 3200 5750 3200
+Wire Wire Line
+	5300 3300 5750 3300
+Wire Wire Line
+	5300 3400 5700 3400
+Wire Wire Line
+	5300 3600 5800 3600
+Wire Wire Line
+	5300 3700 5800 3700
+Wire Wire Line
+	5300 3800 5800 3800
+Wire Wire Line
+	5300 3500 5750 3500
+Text Label 5450 3200 0    50   ~ 0
+MOSI
+Text Label 5350 3300 0    50   ~ 0
+MISO
+Text Label 5400 3400 0    50   ~ 0
+SCLK
+Text Label 5400 3500 0    50   ~ 0
+XRESET
+Text Label 5350 3600 0    50   ~ 0
+DREQ
+Text Label 5400 3700 0    50   ~ 0
+xDCS
+Text Label 5450 3800 0    50   ~ 0
+xCS
+Wire Wire Line
+	7950 2150 7500 2150
+Text Label 7550 2150 0    50   ~ 0
+XRESET
+Wire Wire Line
+	10350 2550 10700 2550
+Text Label 10400 2550 0    50   ~ 0
+MISO
+Wire Wire Line
+	10350 2650 10750 2650
+Text Label 10550 2650 0    50   ~ 0
+MOSI
+Text Label 10550 2750 0    50   ~ 0
+SCLK
+Wire Wire Line
+	10350 2750 10800 2750
+Wire Wire Line
+	7950 2650 7550 2650
+Text Label 7700 2650 0    50   ~ 0
+DREQ
+Wire Wire Line
+	8550 4050 8550 4250
+Text Label 8550 4200 1    50   ~ 0
+xDCS
+Wire Wire Line
+	9550 4050 9550 4350
+Text Label 9550 4200 1    50   ~ 0
+xCS
 $EndSCHEMATC

Commit message: Finish mp3 chip schematic
Parts:
- added C? (x2): 10nF, symbol Device:C
- added C?: 47nF, symbol Device:C
- added C?: 1uF, symbol Device:C
- added C? (x14): 100nF, symbol Device:C
- added C? (x2): 10uF, symbol Device:CP1
- added C?: 100uF, symbol Device:CP1
- added J?: Conn_01x04_Male, symbol Connector:Conn_01x04_Male
- added R? (x2): 100k, symbol Device:R
- added R? (x3): 20R, symbol Device:R
- added U?: AMS1117-1.8, Package_TO_SOT_SMD:SOT-223-3_TabPin2, symbol Regulator_Linear:AMS1117-1.8
- added U?: AMS1117-3.3, Package_TO_SOT_SMD:SOT-223-3_TabPin2, symbol Regulator_Linear:AMS1117-3.3
Connections:
- net labels added: +5V, GPIO-R
- net labels removed: GNDD, VDDA
- wire segments 66 -> 153
Other:
- note added: "Connect GND to GNDA together as close to the chip as possible"
- note added: "Put these next to the chip"
- moved on the sheet: C1, C2, IC1, J1, J?, R1, Y1

Commit message: Assign footprints
Parts:
- C10, C13, C14, C15, C17, C18, C19, C20, C21, C22, C23, C3, C4, C5, C6, C7, C8, C9: renamed from C?; footprint (none) -> Capacitor_SMD:C_0603_1608Metric
- C11, C12, C16: renamed from C?; footprint (none) -> Capacitor_Tantalum_SMD:CP_EIA-3216-18_Kemet-A
- IC1: value COM-08892 -> VS1053B; footprint COM-08892:QFP50P900X900X160-48N -> Package_QFP:LQFP-48_7x7mm_P0.5mm
- J2: renamed from J?; footprint (none) -> Connector_PinSocket_2.54mm:PinSocket_1x04_P2.54mm_Vertical
- J3: renamed from J?; footprint (none) -> Connector_PinHeader_2.54mm:PinHeader_1x08_P2.54mm_Vertical
- R2, R3, R4, R5, R6: renamed from R?; footprint (none) -> Resistor_SMD:R_0603_1608Metric
- gave numbers to parts that had none: 2

Commit message: Start PCB layout
Parts:
- added R7: 0, Jumper:SolderJumper-2_P1.3mm_Bridged2Bar_RoundedPad1.0x1.5mm, symbol Device:R
- C11, C16: footprint Capacitor_Tantalum_SMD:CP_EIA-3216-18_Kemet-A -> Capacitor_SMD:C_0603_1608Metric
- J1: footprint Connector_Audio:Jack_3.5mm_PJ320D_Horizontal -> audio:Jack_3.5mm_PJ320D_Horizontal
Connections:
- wire segments 153 -> 154
Changed lines of the file:
@@
 U 1 1 5BF87719
 P 6550 1200
-F 0 "J1" H 6516 1542 50  0000 C CNN
-F 1 "AudioJack4_Ground" H 6516 1451 50  0000 C CNN
-F 2 "Connector_Audio:Jack_3.5mm_PJ320D_Horizontal" H 6550 1200 50  0001 C CNN
+F 0 "J1" V 6470 1405 50  0000 L CNN
+F 1 "AudioJack4_Ground" V 6561 1405 50  0000 L CNN
+F 2 "audio:Jack_3.5mm_PJ320D_Horizontal" H 6550 1200 50  0001 C CNN
 F 3 "~" H 6550 1200 50  0001 C CNN
 	1    6550 1200
@@
 $EndComp
 Wire Wire Line
-	5700 5050 5700 4850
+	5700 5050 5700 5000
 $Comp
 L power:GNDA #PWR0124
 U 1 1 5C16DB3C
-P 5700 4850
-F 0 "#PWR0124" H 5700 4600 50  0001 C CNN
-F 1 "GNDA" H 5705 4677 50  0000 C CNN
-F 2 "" H 5700 4850 50  0001 C CNN
-F 3 "" H 5700 4850 50  0001 C CNN
-	1    5700 4850
+P 5700 4600
+F 0 "#PWR0124" H 5700 4350 50  0001 C CNN
+F 1 "GNDA" H 5705 4427 50  0000 C CNN
+F 2 "" H 5700 4600 50  0001 C CNN
+F 3 "" H 5700 4600 50  0001 C CNN
+	1    5700 4600
 	-1   0    0    1
 $EndComp
@@
 F 0 "C11" H 3315 5146 50  0000 L CNN
 F 1 "10uF" H 3315 5055 50  0000 L CNN
-F 2 "Capacitor_Tantalum_SMD:CP_EIA-3216-18_Kemet-A" H 3200 5100 50  0001 C CNN
+F 2 "Capacitor_SMD:C_0603_1608Metric" H 3200 5100 50  0001 C CNN
 F 3 "~" H 3200 5100 50  0001 C CNN
 	1    3200 5100
@@
 F 0 "C16" H 3915 6546 50  0000 L CNN
 F 1 "10uF" H 3915 6455 50  0000 L CNN
-F 2 "Capacitor_Tantalum_SMD:CP_EIA-3216-18_Kemet-A" H 3800 6500 50  0001 C CNN
+F 2 "Capacitor_SMD:C_0603_1608Metric" H 3800 6500 50  0001 C CNN
 F 3 "~" H 3800 6500 50  0001 C CNN
 	1    3800 6500
@@
 Wire Wire Line
 	1400 1800 1600 1800
+$Comp
+L Device:R R7
+U 1 1 5C26550C
+P 5700 4850
+F 0 "R7" H 5770 4896 50  0000 L CNN
+F 1 "0" H 5770 4805 50  0000 L CNN
+F 2 "Jumper:SolderJumper-2_P1.3mm_Bridged2Bar_RoundedPad1.0x1.5mm" V 5630 4850 50  0001 C CNN
+F 3 "~" H 5700 4850 50  0001 C CNN
+	1    5700 4850
+	1    0    0    -1
+$EndComp
+Wire Wire Line
+	5700 4600 5700 4700
 $EndSCHEMATC

Commit message: Finish initial PCB layout
This is only the sound module
Parts:
- added R8, R9: 100k, Resistor_SMD:R_0603_1608Metric, symbol Device:R
Connections:
- wire segments 154 -> 157
Changed lines of the file:
@@
 EESchema Schematic File Version 4
+LIBS:badge-cache
 EELAYER 26 0
 EELAYER END
@@
 Connection ~ 10150 2800
 Wire Wire Line
-	10500 2800 10500 2500
-Text Label 10250 2500 0    50   ~ 0
+	10500 2800 10500 2550
+Text Label 7750 3800 1    50   ~ 0
 GPIO-R
-Text Label 7700 3700 1    50   ~ 0
-GPIO-R
-Wire Wire Line
-	10150 3600 10400 3600
-Text Label 10100 3600 0    50   ~ 0
-GPIO-R
+Wire Wire Line
+	10150 3600 10300 3600
 $Comp
 L power:GND #PWR0113
@@
 Wire Wire Line
 	5700 4600 5700 4700
+$Comp
+L Device:R R8
+U 1 1 5C104117
+P 10300 3750
+F 0 "R8" H 10370 3796 50  0000 L CNN
+F 1 "100k" H 10370 3705 50  0000 L CNN
+F 2 "Resistor_SMD:R_0603_1608Metric" V 10230 3750 50  0001 C CNN
+F 3 "~" H 10300 3750 50  0001 C CNN
+	1    10300 3750
+	1    0    0    -1
+$EndComp
+$Comp
+L power:GND #PWR0141
+U 1 1 5C1139F1
+P 10300 3950
+F 0 "#PWR0141" H 10300 3700 50  0001 C CNN
+F 1 "GND" H 10305 3777 50  0000 C CNN
+F 2 "" H 10300 3950 50  0001 C CNN
+F 3 "" H 10300 3950 50  0001 C CNN
+	1    10300 3950
+	1    0    0    -1
+$EndComp
+Wire Wire Line
+	10300 3900 10300 3950
+$Comp
+L Device:R R9
+U 1 1 5C11B744
+P 10650 2550
+F 0 "R9" H 10720 2596 50  0000 L CNN
+F 1 "100k" H 10720 2505 50  0000 L CNN
+F 2 "Resistor_SMD:R_0603_1608Metric" V 10580 2550 50  0001 C CNN
+F 3 "~" H 10650 2550 50  0001 C CNN
+	1    10650 2550
+	0    1    1    0
+$EndComp
+Connection ~ 10500 2550
+Wire Wire Line
+	10500 2550 10500 2500
+$Comp
+L power:GND #PWR0142
+U 1 1 5C11B7E7
+P 10900 2550
+F 0 "#PWR0142" H 10900 2300 50  0001 C CNN
+F 1 "GND" H 10905 2377 50  0000 C CNN
+F 2 "" H 10900 2550 50  0001 C CNN
+F 3 "" H 10900 2550 50  0001 C CNN
+	1    10900 2550
+	0    -1   -1   0
+$EndComp
+Wire Wire Line
+	10900 2550 10800 2550
 $EndSCHEMATC

Commit message: Move MP3 schematic to a new sheet
- add micro usb connector
- add ebyte module
Parts:
- removed C1, C2: 33pF, Capacitor_SMD:C_0603_1608Metric, symbol Device:C
- removed C10, C13, C14, C15, C17, C18, C19, C3, C4, C5, C6, C7, C8, C9: 100nF, Capacitor_SMD:C_0603_1608Metric, symbol Device:C
- removed C11, C16: 10uF, Capacitor_SMD:C_0603_1608Metric, symbol Device:CP1
- removed C12: 100uF, Capacitor_Tantalum_SMD:CP_EIA-3216-18_Kemet-A, symbol Device:CP1
- removed C20, C21: 10nF, Capacitor_SMD:C_0603_1608Metric, symbol Device:C
- removed C22: 47nF, Capacitor_SMD:C_0603_1608Metric, symbol Device:C
- removed C23: 1uF, Capacitor_SMD:C_0603_1608Metric, symbol Device:C
- removed IC1: VS1053B, Package_QFP:LQFP-48_7x7mm_P0.5mm, symbol COM-08892:COM-08892
- removed J1: AudioJack4_Ground, audio:Jack_3.5mm_PJ320D_Horizontal, symbol Connector:AudioJack4_Ground
- removed J2: Conn_01x04_Male, Connector_PinSocket_2.54mm:PinSocket_1x04_P2.54mm_Vertical, symbol Connector:Conn_01x04_Male
- removed J3: Conn_01x08_Male, Connector_PinHeader_2.54mm:PinHeader_1x08_P2.54mm_Vertical, symbol Connector:Conn_01x08_Male
- removed R1: 1M, Resistor_SMD:R_0603_1608Metric, symbol Device:R
- removed R2, R3, R4: 20R, Resistor_SMD:R_0603_1608Metric, symbol Device:R
- removed R5, R6, R8, R9: 100k, Resistor_SMD:R_0603_1608Metric, symbol Device:R
- removed R7: 0, Jumper:SolderJumper-2_P1.3mm_Bridged2Bar_RoundedPad1.0x1.5mm, symbol Device:R
- removed U1: AMS1117-1.8, Package_TO_SOT_SMD:SOT-223-3_TabPin2, symbol Regulator_Linear:AMS1117-1.8
- removed U2: AMS1117-3.3, Package_TO_SOT_SMD:SOT-223-3_TabPin2, symbol Regulator_Linear:AMS1117-3.3
- removed Y1: 12.288M, Crystal:Crystal_SMD_3225-4Pin_3.2x2.5mm, symbol Device:Crystal
- added J?: USB_B_Micro, symbol Connector:USB_B_Micro
- added U?: E73-2G4M08S1C, symbol ebyte:E73-2G4M08S1C
Connections:
- net labels added: +3.3V, D+, D-
- net labels removed: +1V8, +3V3, +5V, DREQ, GBUF, GNDA, GPIO-R, LEFT, MISO, MOSI, RIGHT, SCLK, XRESET, xCS, xDCS
- wire segments 157 -> 7
- no-connect marks 0 -> 3
Other:
- note removed: "Connect GND to GNDA together as close to the chip as possible"
- note removed: "Put these next to the chip"
