File: pcb/badge/badge.sch (KiCad schematic (older format))
At the start: 2 parts

Commit message: Fix names in MP3 sheet
Add programming connector
Parts:
- added J?: Conn_01x04_Male, symbol Connector:Conn_01x04_Male
- added J?: Conn_01x08_Male, symbol Connector:Conn_01x08_Male
- J4: renamed from J?; footprint (none) -> Connector_USB:USB_Micro-B_Molex-105017-0001
- U3: renamed from U?; footprint (none) -> EBYTE:E73-2G4M08S1C
Connections:
- net labels added: MISO, MOSI, SCLK, SNDCS, SNDDREQ, SNDRESET, SNDxDCS, SWCLK, SWDCLK, SWDIO, VCC
- wire segments 7 -> 27
Other:
- moved on the sheet: U3
Changed lines of the file:
@@
 $EndDescr
 $Sheet
-S 800  800  1200 550
+S 1600 750  1200 550
 U 5C1D48B0
 F0 "SheetMP3" 50
 F1 "MP3.sch" 50
-F2 "MISO" I R 2000 900 50
-F3 "MOSI" I R 2000 1050 50
-F4 "SCLK" I R 2000 1200 50
-F5 "XRESET" I L 800 1150 50
-F6 "DREQ" O L 800 1050 50
-F7 "xDCS" I L 800 900 50
-F8 "xCS" I L 800 1250 50
+F2 "MISO" I R 2800 850 50
+F3 "MOSI" I R 2800 1000 50
+F4 "SCLK" I R 2800 1150 50
+F5 "XRESET" I L 1600 1200 50
+F6 "DREQ" O L 1600 1000 50
+F7 "xDCS" I L 1600 850 50
+F8 "xCS" I R 2800 1250 50
 $EndSheet
 $Comp
-L ebyte:E73-2G4M08S1C U?
+L ebyte:E73-2G4M08S1C U3
 U 1 1 5C1F197E
-P 4400 3250
-F 0 "U?" H 4575 2228 50  0000 C CNN
-F 1 "E73-2G4M08S1C" H 4575 2137 50  0000 C CNN
-F 2 "" H 4300 3300 50  0001 C CNN
-F 3 "" H 4300 3300 50  0001 C CNN
-	1    4400 3250
-	1    0    0    -1
-$EndComp
-$Comp
-L power:GND #PWR?
+P 4700 3250
+F 0 "U3" H 4875 2228 50  0000 C CNN
+F 1 "E73-2G4M08S1C" H 4875 2137 50  0000 C CNN
+F 2 "EBYTE:E73-2G4M08S1C" H 4600 3300 50  0001 C CNN
+F 3 "" H 4600 3300 50  0001 C CNN
+	1    4700 3250
+	1    0    0    -1
+$EndComp
+$Comp
+L power:GND #PWR0101
 U 1 1 5C1F19F6
-P 4350 2150
-F 0 "#PWR?" H 4350 1900 50  0001 C CNN
-F 1 "GND" H 4355 1977 50  0000 C CNN
-F 2 "" H 4350 2150 50  0001 C CNN
-F 3 "" H 4350 2150 50  0001 C CNN
-	1    4350 2150
+P 4650 2150
+F 0 "#PWR0101" H 4650 1900 50  0001 C CNN
+F 1 "GND" H 4655 1977 50  0000 C CNN
+F 2 "" H 4650 2150 50  0001 C CNN
+F 3 "" H 4650 2150 50  0001 C CNN
+	1    4650 2150
 	-1   0    0    1
 $EndComp
 $Comp
-L power:GND #PWR?
+L power:GND #PWR0102
 U 1 1 5C1F1A1C
-P 5500 3550
-F 0 "#PWR?" H 5500 3300 50  0001 C CNN
-F 1 "GND" V 5505 3422 50  0000 R CNN
-F 2 "" H 5500 3550 50  0001 C CNN
-F 3 "" H 5500 3550 50  0001 C CNN
-	1    5500 3550
+P 5800 3550
+F 0 "#PWR0102" H 5800 3300 50  0001 C CNN
+F 1 "GND" V 5805 3422 50  0000 R CNN
+F 2 "" H 5800 3550 50  0001 C CNN
+F 3 "" H 5800 3550 50  0001 C CNN
+	1    5800 3550
 	0    -1   -1   0
 $EndComp
 $Comp
-L power:+3.3V #PWR?
+L power:+3.3V #PWR0103
 U 1 1 5C1F1A4A
-P 4200 2050
-F 0 "#PWR?" H 4200 1900 50  0001 C CNN
-F 1 "+3.3V" H 4215 2223 50  0000 C CNN
-F 2 "" H 4200 2050 50  0001 C CNN
-F 3 "" H 4200 2050 50  0001 C CNN
-	1    4200 2050
-	1    0    0    -1
-$EndComp
-Wire Wire Line
-	4200 2050 4200 2150
-Wire Wire Line
-	4500 2150 4500 2000
-$Comp
-L power:+3.3V #PWR?
+P 4500 2050
+F 0 "#PWR0103" H 4500 1900 50  0001 C CNN
+F 1 "+3.3V" H 4515 2223 50  0000 C CNN
+F 2 "" H 4500 2050 50  0001 C CNN
+F 3 "" H 4500 2050 50  0001 C CNN
+	1    4500 2050
+	1    0    0    -1
+$EndComp
+Wire Wire Line
+	4500 2050 4500 2150
+Wire Wire Line
+	4800 2150 4800 2000
+$Comp
+L power:+3.3V #PWR0104
 U 1 1 5C1F1A95
-P 4500 2000
-F 0 "#PWR?" H 4500 1850 50  0001 C CNN
-F 1 "+3.3V" H 4515 2173 50  0000 C CNN
-F 2 "" H 4500 2000 50  0001 C CNN
-F 3 "" H 4500 2000 50  0001 C CNN
-	1    4500 2000
-	1    0    0    -1
-$EndComp
-NoConn ~ 4050 2150
+P 4800 2000
+F 0 "#PWR0104" H 4800 1850 50  0001 C CNN
+F 1 "+3.3V" H 4800 2150 50  0000 C CNN
+F 2 "" H 4800 2000 50  0001 C CNN
+F 3 "" H 4800 2000 50  0001 C CNN
+	1    4800 2000
+	1    0    0    -1
+$EndComp
+NoConn ~ 4350 2150
 Wire Wire Line
 	3100 2950 3650 2950
@@
 NoConn ~ 2700 3550
 $Comp
-L power:GND #PWR?
+L power:GND #PWR0105
 U 1 1 5C1F1C91
 P 2800 3550
-F 0 "#PWR?" H 2800 3300 50  0001 C CNN
+F 0 "#PWR0105" H 2800 3300 50  0001 C CNN
 F 1 "GND" H 2805 3377 50  0000 C CNN
 F 2 "" H 2800 3550 50  0001 C CNN
@@
 D+
 $Comp
-L Connector:USB_B_Micro J?
+L Connector:USB_B_Micro J4
 U 1 1 5C1F1B13
 P 2800 3150
-F 0 "J?" H 2855 3617 50  0000 C CNN
+F 0 "J4" H 2855 3617 50  0000 C CNN
 F 1 "USB_B_Micro" H 2855 3526 50  0000 C CNN
-F 2 "" H 2950 3100 50  0001 C CNN
+F 2 "Connector_USB:USB_Micro-B_Molex-105017-0001" H 2950 3100 50  0001 C CNN
 F 3 "~" H 2950 3100 50  0001 C CNN
 	1    2800 3150
 	1    0    0    -1
 $EndComp
+Wire Wire Line
+	2800 850  3100 850
+Wire Wire Line
+	2800 1000 3100 1000
+Wire Wire Line
+	2800 1150 3100 1150
+Text Label 2850 850  0    50   ~ 0
+MISO
+Text Label 2900 1000 0    50   ~ 0
+MOSI
+Text Label 2900 1150 0    50   ~ 0
+SCLK
+Wire Wire Line
+	2800 1250 3100 1250
+Text Label 2850 1250 0    50   ~ 0
+SNDCS
+Wire Wire Line
+	1600 850  1400 850
+Wire Wire Line
+	1600 1000 1400 1000
+Wire Wire Line
+	1600 1200 1400 1200
+Text Label 1550 850  2    50   ~ 0
+SNDxDCS
+Text Label 1500 1000 2    50   ~ 0
+SNDDREQ
+Text Label 1550 1200 2    50   ~ 0
+SNDRESET
+Wire Wire Line
+	5800 4000 6100 4000
+Wire Wire Line
+	5800 3400 6100 3400
+Wire Wire Line
+	4950 2150 4950 1700
+Wire Wire Line
+	3650 3400 3450 3400
+Wire Wire Line
+	3650 3550 3400 3550
+Wire Wire Line
+	5800 3850 6150 3850
+Wire Wire Line
+	5800 4150 6100 4150
+Text Label 5850 4150 0    50   ~ 0
+MOSI
+Text Label 5850 4000 0    50   ~ 0
+MISO
+Text Label 5850 3850 0    50   ~ 0
+SCLK
+Text Label 5850 3400 0    50   ~ 0
+SNDCS
+Text Label 4950 2100 1    50   ~ 0
+SNDRESET
+Text Label 3600 3400 2    50   ~ 0
+SNDDREQ
+Text Label 3600 3550 2    50   ~ 0
+SNDxDCS
+$Comp
+L Connector:Conn_01x04_Male J?
+U 1 1 5C1C7A0F
+P 1250 2400
+F 0 "J?" H 1356 2678 50  0000 C CNN
+F 1 "Conn_01x04_Male" H 1350 2800 50  0000 C CNN
+F 2 "" H 1250 2400 50  0001 C CNN
+F 3 "~" H 1250 2400 50  0001 C CNN
+	1    1250 2400
+	1    0    0    -1
+$EndComp
+Wire Wire Line
+	1450 2300 1800 2300
+Wire Wire Line
+	1450 2400 1800 2400
+Wire Wire Line
+	1450 2500 1800 2500
+Wire Wire Line
+	1450 2600 1800 2600
+Text Label 1500 2300 0    50   ~ 0
+VCC
+Text Label 1500 2400 0    50   ~ 0
+SWDIO
+Text Label 1500 2500 0    50   ~ 0
+SWCLK
+Text Label 1500 2600 0    50   ~ 0
+GND
+$Comp
+L power:+3.3V #PWR?
+U 1 1 5C1C8FC9
+P 1800 2300
+F 0 "#PWR?" H 1800 2150 50  0001 C CNN
+F 1 "+3.3V" H 1815 2473 50  0000 C CNN
+F 2 "" H 1800 2300 50  0001 C CNN
+F 3 "" H 1800 2300 50  0001 C CNN
+	1    1800 2300
+	0    1    1    0
+$EndComp
+Wire Wire Line
+	3650 3850 3250 3850
+Wire Wire Line
+	3650 3700 3250 3700
+Text Label 3350 3700 0    50   ~ 0
+SWDIO
+Text Label 3300 3850 0    50   ~ 0
+SWDCLK
+$Comp
+L power:GND #PWR?
+U 1 1 5C1CA857
+P 1800 2600
+F 0 "#PWR?" H 1800 2350 50  0001 C CNN
+F 1 "GND" H 1805 2427 50  0000 C CNN
+F 2 "" H 1800 2600 50  0001 C CNN
+F 3 "" H 1800 2600 50  0001 C CNN
+	1    1800 2600
+	0    -1   -1   0
+$EndComp
+$Comp
+L Connector:Conn_01x08_Male J?
+U 1 1 5C1CAC01
+P 950 3750
+F 0 "J?" H 1056 4228 50  0000 C CNN
+F 1 "Conn_01x08_Male" H 1056 4137 50  0000 C CNN
+F 2 "" H 950 3750 50  0001 C CNN
+F 3 "~" H 950 3750 50  0001 C CNN
+	1    950  3750
+	1    0    0    -1
+$EndComp

Commit message: Add schematic for E paper display
Parts:
- J5: renamed from J?; footprint (none) -> Connector_PinHeader_2.54mm:PinHeader_1x08_P2.54mm_Vertical
- J6: renamed from J?; footprint (none) -> Connector_PinHeader_2.54mm:PinHeader_1x04_P2.54mm_Vertical
Connections:
- net labels added: DISPBUSY, DISPCS, DISPDC, DISPRST
- wire segments 27 -> 39
Other:
- moved on the sheet: J4, J5
Changed lines of the file:
@@
 $Descr A4 11693 8268
 encoding utf-8
-Sheet 1 2
+Sheet 1 3
 Title ""
 Date ""
@@
 U 1 1 5C1F197E
 P 4700 3250
-F 0 "U3" H 4875 2228 50  0000 C CNN
+F 0 "U3" H 4850 2050 50  0000 C CNN
 F 1 "E73-2G4M08S1C" H 4875 2137 50  0000 C CNN
 F 2 "EBYTE:E73-2G4M08S1C" H 4600 3300 50  0001 C CNN
@@
 NoConn ~ 4350 2150
 Wire Wire Line
-	3100 2950 3650 2950
-Wire Wire Line
-	3100 3150 3250 3150
-Text Label 3150 3150 0    50   ~ 0
+	3100 2800 3650 2800
+Wire Wire Line
+	3100 3000 3250 3000
+Text Label 3150 3000 0    50   ~ 0
 D+
 Wire Wire Line
-	3100 3250 3250 3250
-Text Label 3150 3250 0    50   ~ 0
+	3100 3100 3250 3100
+Text Label 3150 3100 0    50   ~ 0
 D-
-NoConn ~ 3100 3350
-NoConn ~ 2700 3550
+NoConn ~ 3100 3200
+NoConn ~ 2700 3400
 $Comp
 L power:GND #PWR0105
 U 1 1 5C1F1C91
-P 2800 3550
-F 0 "#PWR0105" H 2800 3300 50  0001 C CNN
-F 1 "GND" H 2805 3377 50  0000 C CNN
-F 2 "" H 2800 3550 50  0001 C CNN
-F 3 "" H 2800 3550 50  0001 C CNN
-	1    2800 3550
-	1    0    0    -1
-$EndComp
+P 2800 3400
+F 0 "#PWR0105" H 2800 3150 50  0001 C CNN
+F 1 "GND" H 2805 3227 50  0000 C CNN
+F 2 "" H 2800 3400 50  0001 C CNN
+F 3 "" H 2800 3400 50  0001 C CNN
+	1    2800 3400
+	1    0    0    -1
+$EndComp
+Wire Wire Line
+	3650 2950 3500 2950
+Text Label 3550 2950 0    50   ~ 0
+D-
 Wire Wire Line
 	3650 3100 3500 3100
-Text Label 3550 3100 0    50   ~ 0
-D-
-Wire Wire Line
-	3650 3250 3500 3250
-Text Label 3500 3250 0    50   ~ 0
+Text Label 3500 3100 0    50   ~ 0
 D+
 $Comp
 L Connector:USB_B_Micro J4
 U 1 1 5C1F1B13
-P 2800 3150
-F 0 "J4" H 2855 3617 50  0000 C CNN
-F 1 "USB_B_Micro" H 2855 3526 50  0000 C CNN
-F 2 "Connector_USB:USB_Micro-B_Molex-105017-0001" H 2950 3100 50  0001 C CNN
-F 3 "~" H 2950 3100 50  0001 C CNN
-	1    2800 3150
+P 2800 3000
+F 0 "J4" H 2855 3467 50  0000 C CNN
+F 1 "USB_B_Micro" H 2855 3376 50  0000 C CNN
+F 2 "Connector_USB:USB_Micro-B_Molex-105017-0001" H 2950 2950 50  0001 C CNN
+F 3 "~" H 2950 2950 50  0001 C CNN
+	1    2800 3000
 	1    0    0    -1
 $EndComp
@@
 SNDRESET
 Wire Wire Line
+	5800 3850 6100 3850
+Wire Wire Line
+	5800 3400 6100 3400
+Wire Wire Line
+	4950 2150 4950 1700
+Wire Wire Line
+	3650 3250 3450 3250
+Wire Wire Line
+	3650 3400 3400 3400
+Wire Wire Line
+	5800 3700 6150 3700
+Wire Wire Line
 	5800 4000 6100 4000
-Wire Wire Line
-	5800 3400 6100 3400
-Wire Wire Line
-	4950 2150 4950 1700
-Wire Wire Line
-	3650 3400 3450 3400
-Wire Wire Line
-	3650 3550 3400 3550
-Wire Wire Line
-	5800 3850 6150 3850
-Wire Wire Line
-	5800 4150 6100 4150
-Text Label 5850 4150 0    50   ~ 0
+Text Label 5850 4000 0    50   ~ 0
 MOSI
-Text Label 5850 4000 0    50   ~ 0
+Text Label 5850 3850 0    50   ~ 0
 MISO
-Text Label 5850 3850 0    50   ~ 0
+Text Label 5850 3700 0    50   ~ 0
 SCLK
 Text Label 5850 3400 0    50   ~ 0
@@
 Text Label 4950 2100 1    50   ~ 0
 SNDRESET
+Text Label 3600 3250 2    50   ~ 0
+SNDDREQ
 Text Label 3600 3400 2    50   ~ 0
-SNDDREQ
-Text Label 3600 3550 2    50   ~ 0
 SNDxDCS
 $Comp
-L Connector:Conn_01x04_Male J?
+L Connector:Conn_01x04_Male J6
 U 1 1 5C1C7A0F
 P 1250 2400
-F 0 "J?" H 1356 2678 50  0000 C CNN
+F 0 "J6" H 1356 2678 50  0000 C CNN
 F 1 "Conn_01x04_Male" H 1350 2800 50  0000 C CNN
-F 2 "" H 1250 2400 50  0001 C CNN
+F 2 "Connector_PinHeader_2.54mm:PinHeader_1x04_P2.54mm_Vertical" H 1250 2400 50  0001 C CNN
 F 3 "~" H 1250 2400 50  0001 C CNN
 	1    1250 2400
@@
 GND
 $Comp
-L power:+3.3V #PWR?
+L power:+3.3V #PWR0148
 U 1 1 5C1C8FC9
 P 1800 2300
-F 0 "#PWR?" H 1800 2150 50  0001 C CNN
+F 0 "#PWR0148" H 1800 2150 50  0001 C CNN
 F 1 "+3.3V" H 1815 2473 50  0000 C CNN
 F 2 "" H 1800 2300 50  0001 C CNN
@@
 $EndComp
 Wire Wire Line
-	3650 3850 3250 3850
-Wire Wire Line
 	3650 3700 3250 3700
-Text Label 3350 3700 0    50   ~ 0
+Wire Wire Line
+	3650 3550 3250 3550
+Text Label 3350 3550 0    50   ~ 0
 SWDIO
-Text Label 3300 3850 0    50   ~ 0
+Text Label 3300 3700 0    50   ~ 0
 SWDCLK
 $Comp
-L power:GND #PWR?
+L power:GND #PWR0149
 U 1 1 5C1CA857
 P 1800 2600
-F 0 "#PWR?" H 1800 2350 50  0001 C CNN
+F 0 "#PWR0149" H 1800 2350 50  0001 C CNN
 F 1 "GND" H 1805 2427 50  0000 C CNN
 F 2 "" H 1800 2600 50  0001 C CNN
@@
 $EndComp
 $Comp
-L Connector:Conn_01x08_Male J?
+L Connector:Conn_01x08_Male J5
 U 1 1 5C1CAC01
-P 950 3750
-F 0 "J?" H 1056 4228 50  0000 C CNN
-F 1 "Conn_01x08_Male" H 1056 4137 50  0000 C CNN
-F 2 "" H 950 3750 50  0001 C CNN
-F 3 "~" H 950 3750 50  0001 C CNN
-	1    950  3750
-	1    0    0    -1
-$EndComp
+P 7850 2200
+F 0 "J5" H 7956 2678 50  0000 C CNN
+F 1 "Conn_01x08_Male" H 7900 2800 50  0000 C CNN
+F 2 "Connector_PinHeader_2.54mm:PinHeader_1x08_P2.54mm_Vertical" H 7850 2200 50  0001 C CNN
+F 3 "~" H 7850 2200 50  0001 C CNN
+	1    7850 2200
+	1    0    0    -1
+$EndComp
+Wire Wire Line
+	8050 1900 8500 1900
+Wire Wire Line
+	8050 2000 8500 2000
+Text Label 8100 2100 0    50   ~ 0
+MOSI
+Text Label 8100 2200 0    50   ~ 0
+SCLK
+Text Label 8100 2300 0    50   ~ 0
+DISPCS
+Text Label 8100 2400 0    50   ~ 0
+DISPDC
+Text Label 8100 2500 0    50   ~ 0
+DISPRST
+Text Label 8100 2600 0    50   ~ 0
+DISPBUSY
+$Comp
+L power:GND #PWR0150
+U 1 1 5C21556B
+P 8500 2000
+F 0 "#PWR0150" H 8500 1750 50  0001 C CNN
+F 1 "GND" V 8505 1872 50  0000 R CNN
+F 2 "" H 8500 2000 50  0001 C CNN
+F 3 "" H 8500 2000 50  0001 C CNN
+	1    8500 2000
+	0    -1   -1   0
+$EndComp
+$Comp
+L power:+3.3V #PWR0151
+U 1 1 5C215595
+P 8500 1900
+F 0 "#PWR0151" H 8500 1750 50  0001 C CNN
+F 1 "+3.3V" V 8500 2150 50  0000 C CNN
+F 2 "" H 8500 1900 50  0001 C CNN
+F 3 "" H 8500 1900 50  0001 C CNN
+	1    8500 1900
+	0    1    1    0
+$EndComp
+Wire Wire Line
+	5400 2150 5400 1800
+Wire Wire Line
+	5250 2150 5250 1800
+Text Label 5400 2100 1    50   ~ 0
+DISPCS
+Text Label 5250 2100 1    50   ~ 0
+DISPDC
+Wire Wire Line
+	4350 4300 4350 4750
+Text Label 4350 4650 1    50   ~ 0
+DISPRST
+Text Label 4500 4700 1    50   ~ 0
+DISPBUSY
+Wire Wire Line
+	4500 4300 4500 4750
+$Sheet
+S 9100 1650 1750 1500
+U 5C21B929
+F0 "Epaper" 50
+F1 "Epaper.sch" 50
+F2 "DIN" I L 9100 2100 50
+F3 "CLK" I L 9100 2200 50
+F4 "CS" I L 9100 2300 50
+F5 "DC" I L 9100 2400 50
+F6 "RST" I L 9100 2500 50
+F7 "BUSY" O L 9100 2600 50
+$EndSheet
+Wire Wire Line
+	8050 2300 9100 2300
+Wire Wire Line
+	8050 2400 9100 2400
+Wire Wire Line
+	8050 2500 9100 2500
+Wire Wire Line
+	8050 2600 9100 2600
+Wire Wire Line
+	8050 2200 9100 2200
+Wire Wire Line
+	8050 2100 9100 2100
 $EndSCHEMATC

Commit message: Fix ERC problems
Connections:
- net labels removed: SWCLK
Changed lines of the file:
@@
 	1450 2400 1800 2400
-Wire Wire Line
-	1450 2500 1800 2500
 Wire Wire Line
 	1450 2600 1800 2600
@@
 SWDIO
 Text Label 1500 2500 0    50   ~ 0
-SWCLK
+SWDCLK
 Text Label 1500 2600 0    50   ~ 0
 GND
@@
 Wire Wire Line
 	8050 2100 9100 2100
+Wire Wire Line
+	1450 2500 1800 2500
 $EndSCHEMATC

Commit message: Add touch button symbols + footprints
Parts:
- added U4: touch-slider-4pin, touch-buttons:TouchSlider-4_50x10mm, symbol touch-buttons:touch-slider-4pin
- added U5, U6: touch-button, touch-buttons:TOUCH-CIRCLE, symbol touch-buttons:touch-button
Connections:
- net labels added: TouchBTN1, TouchBTN2
- wire segments 39 -> 53
Changed lines of the file:
@@
 U 1 1 5C1F197E
 P 4700 3250
-F 0 "U3" H 4850 2050 50  0000 C CNN
-F 1 "E73-2G4M08S1C" H 4875 2137 50  0000 C CNN
+F 0 "U3" H 4700 3250 50  0000 C CNN
+F 1 "E73-2G4M08S1C" H 4650 3400 50  0000 C CNN
 F 2 "EBYTE:E73-2G4M08S1C" H 4600 3300 50  0001 C CNN
 F 3 "" H 4600 3300 50  0001 C CNN
@@
 SNDRESET
 Wire Wire Line
-	5800 3850 6100 3850
+	5400 2150 5400 1850
 Wire Wire Line
 	5800 3400 6100 3400
@@
 	3650 3400 3400 3400
 Wire Wire Line
-	5800 3700 6150 3700
+	5250 2150 5250 1800
 Wire Wire Line
 	5800 4000 6100 4000
 Text Label 5850 4000 0    50   ~ 0
 MOSI
-Text Label 5850 3850 0    50   ~ 0
+Text Label 5400 2100 1    50   ~ 0
 MISO
-Text Label 5850 3700 0    50   ~ 0
+Text Label 5250 2100 1    50   ~ 0
 SCLK
 Text Label 5850 3400 0    50   ~ 0
@@
 $EndComp
 Wire Wire Line
-	5400 2150 5400 1800
-Wire Wire Line
-	5250 2150 5250 1800
-Text Label 5400 2100 1    50   ~ 0
+	4950 4300 4950 4650
+Wire Wire Line
+	5100 4300 5100 4650
+Text Label 4950 4350 3    50   ~ 0
 DISPCS
-Text Label 5250 2100 1    50   ~ 0
+Text Label 5100 4350 3    50   ~ 0
 DISPDC
 Wire Wire Line
@@
 Wire Wire Line
 	1450 2500 1800 2500
+$Comp
+L power:GND #PWR0162
+U 1 1 5C2E4386
+P 5250 4300
+F 0 "#PWR0162" H 5250 4050 50  0001 C CNN
+F 1 "GND" H 5255 4127 50  0000 C CNN
+F 2 "" H 5250 4300 50  0001 C CNN
+F 3 "" H 5250 4300 50  0001 C CNN
+	1    5250 4300
+	1    0    0    -1
+$EndComp
+$Comp
+L touch-buttons:touch-button U5
+U 1 1 5C2E49F6
+P 7100 4050
+F 0 "U5" H 7482 4042 50  0000 L CNN
+F 1 "touch-button" H 7482 3951 50  0000 L CNN
+F 2 "touch-buttons:TOUCH-CIRCLE" H 7100 4050 50  0001 C CNN
+F 3 "" H 7100 4050 50  0001 C CNN
+	1    7100 4050
+	1    0    0    -1
+$EndComp
+$Comp
+L touch-buttons:touch-button U6
+U 1 1 5C2E4A86
+P 8450 4050
+F 0 "U6" H 8832 4042 50  0000 L CNN
+F 1 "touch-button" H 8832 3951 50  0000 L CNN
+F 2 "touch-buttons:TOUCH-CIRCLE" H 8450 4050 50  0001 C CNN
+F 3 "" H 8450 4050 50  0001 C CNN
+	1    8450 4050
+	1    0    0    -1
+$EndComp
+$Comp
+L touch-buttons:touch-slider-4pin U4
+U 1 1 5C2E4B1E
+P 6600 2900
+F 0 "U4" V 6554 3077 50  0000 L CNN
+F 1 "touch-slider-4pin" V 6645 3077 50  0000 L CNN
+F 2 "touch-buttons:TouchSlider-4_50x10mm" H 6600 2900 50  0001 C CNN
+F 3 "" H 6600 2900 50  0001 C CNN
+	1    6600 2900
+	0    1    1    0
+$EndComp
+Wire Wire Line
+	6350 3200 5800 3200
+Wire Wire Line
+	5800 3200 5800 3250
+Wire Wire Line
+	6350 3000 5800 3000
+Wire Wire Line
+	5800 3000 5800 3100
+Wire Wire Line
+	5800 2950 5800 2900
+Wire Wire Line
+	5800 2900 6350 2900
+Wire Wire Line
+	6350 2900 6350 2800
+Wire Wire Line
+	6350 2600 6100 2600
+Wire Wire Line
+	6100 2600 6100 2800
+Wire Wire Line
+	6100 2800 5800 2800
+Wire Wire Line
+	7100 4500 7100 4950
+Wire Wire Line
+	8450 4500 8450 4950
+Text Label 7100 4900 1    50   ~ 0
+TouchBTN1
+Text Label 8450 4900 1    50   ~ 0
+TouchBTN2
+Text Label 6250 3700 2    50   ~ 0
+TouchBTN1
+Wire Wire Line
+	5800 3700 6350 3700
+Wire Wire Line
+	5800 3850 6350 3850
+Text Label 6300 3850 2    50   ~ 0
+TouchBTN2
 $EndSCHEMATC

Commit message: Routing the CPU
Connections:
- net labels added: +5V
- wire segments 53 -> 55
Changed lines of the file:
@@
 NoConn ~ 4350 2150
 Wire Wire Line
-	3100 2800 3650 2800
+	3100 2800 3300 2800
 Wire Wire Line
 	3100 3000 3250 3000
@@
 Text Label 5850 4000 0    50   ~ 0
 MOSI
-Text Label 5400 2100 1    50   ~ 0
+Text Label 4950 2050 1    50   ~ 0
 MISO
 Text Label 5250 2100 1    50   ~ 0
@@
 Text Label 5850 3400 0    50   ~ 0
 SNDCS
-Text Label 4950 2100 1    50   ~ 0
+Text Label 5400 2150 1    50   ~ 0
 SNDRESET
 Text Label 3600 3250 2    50   ~ 0
@@
 Wire Wire Line
 	5100 4300 5100 4650
+Text Label 5100 4350 3    50   ~ 0
+DISPCS
 Text Label 4950 4350 3    50   ~ 0
-DISPCS
-Text Label 5100 4350 3    50   ~ 0
 DISPDC
 Wire Wire Line
 	4350 4300 4350 4750
-Text Label 4350 4650 1    50   ~ 0
+Text Label 4500 4650 1    50   ~ 0
 DISPRST
-Text Label 4500 4700 1    50   ~ 0
+Text Label 4350 4700 1    50   ~ 0
 DISPBUSY
 Wire Wire Line
@@
 Text Label 6300 3850 2    50   ~ 0
 TouchBTN2
+Wire Wire Line
+	3300 2800 3300 2700
+Connection ~ 3300 2800
+Wire Wire Line
+	3300 2800 3650 2800
+$Comp
+L power:+5V #PWR?
+U 1 1 5C30DCF7
+P 3300 2700
+F 0 "#PWR?" H 3300 2550 50  0001 C CNN
+F 1 "+5V" H 3315 2873 50  0000 C CNN
+F 2 "" H 3300 2700 50  0001 C CNN
+F 3 "" H 3300 2700 50  0001 C CNN
+	1    3300 2700
+	1    0    0    -1
+$EndComp
 $EndSCHEMATC
