File: pcb/badge/badge.sch (KiCad schematic (older format))
At the start: 7 parts, among them J4 USB_B_Micro, J5 Conn_01x08_Male, J6 Conn_01x04_Male, U3 E73-2G4M08S1C, U4 touch-slider-4pin, U5 touch-button, U6 touch-button

Commit message: fix: add missing pin in E73 symbol
Pin #1 was missing (P1.11)
Connections:
- wire segments 55 -> 56
Other:
- moved on the sheet: J4, U4
Changed lines of the file:
@@
 L power:GND #PWR0101
 U 1 1 5C1F19F6
-P 4650 2150
-F 0 "#PWR0101" H 4650 1900 50  0001 C CNN
-F 1 "GND" H 4655 1977 50  0000 C CNN
-F 2 "" H 4650 2150 50  0001 C CNN
-F 3 "" H 4650 2150 50  0001 C CNN
-	1    4650 2150
-	-1   0    0    1
+P 4500 1600
+F 0 "#PWR0101" H 4500 1350 50  0001 C CNN
+F 1 "GND" H 4505 1427 50  0000 C CNN
+F 2 "" H 4500 1600 50  0001 C CNN
+F 3 "" H 4500 1600 50  0001 C CNN
+	1    4500 1600
+	0    -1   -1   0
 $EndComp
 $Comp
 L power:GND #PWR0102
 U 1 1 5C1F1A1C
-P 5800 3550
-F 0 "#PWR0102" H 5800 3300 50  0001 C CNN
-F 1 "GND" V 5805 3422 50  0000 R CNN
-F 2 "" H 5800 3550 50  0001 C CNN
-F 3 "" H 5800 3550 50  0001 C CNN
-	1    5800 3550
+P 5800 3450
+F 0 "#PWR0102" H 5800 3200 50  0001 C CNN
+F 1 "GND" V 5805 3322 50  0000 R CNN
+F 2 "" H 5800 3450 50  0001 C CNN
+F 3 "" H 5800 3450 50  0001 C CNN
+	1    5800 3450
 	0    -1   -1   0
 $EndComp
@@
 L power:+3.3V #PWR0103
 U 1 1 5C1F1A4A
-P 4500 2050
-F 0 "#PWR0103" H 4500 1900 50  0001 C CNN
-F 1 "+3.3V" H 4515 2223 50  0000 C CNN
-F 2 "" H 4500 2050 50  0001 C CNN
-F 3 "" H 4500 2050 50  0001 C CNN
-	1    4500 2050
-	1    0    0    -1
-$EndComp
-Wire Wire Line
-	4500 2050 4500 2150
-Wire Wire Line
-	4800 2150 4800 2000
+P 4350 1900
+F 0 "#PWR0103" H 4350 1750 50  0001 C CNN
+F 1 "+3.3V" H 4365 2073 50  0000 C CNN
+F 2 "" H 4350 1900 50  0001 C CNN
+F 3 "" H 4350 1900 50  0001 C CNN
+	1    4350 1900
+	1    0    0    -1
+$EndComp
 $Comp
 L power:+3.3V #PWR0104
 U 1 1 5C1F1A95
-P 4800 2000
-F 0 "#PWR0104" H 4800 1850 50  0001 C CNN
-F 1 "+3.3V" H 4800 2150 50  0000 C CNN
-F 2 "" H 4800 2000 50  0001 C CNN
-F 3 "" H 4800 2000 50  0001 C CNN
-	1    4800 2000
-	1    0    0    -1
-$EndComp
-NoConn ~ 4350 2150
-Wire Wire Line
-	3100 2800 3300 2800
-Wire Wire Line
-	3100 3000 3250 3000
-Text Label 3150 3000 0    50   ~ 0
+P 4650 1900
+F 0 "#PWR0104" H 4650 1750 50  0001 C CNN
+F 1 "+3.3V" H 4650 2050 50  0000 C CNN
+F 2 "" H 4650 1900 50  0001 C CNN
+F 3 "" H 4650 1900 50  0001 C CNN
+	1    4650 1900
+	1    0    0    -1
+$EndComp
+NoConn ~ 4200 2050
+Wire Wire Line
+	3100 2850 3300 2850
+Wire Wire Line
+	3100 3050 3250 3050
+Text Label 3150 3050 0    50   ~ 0
 D+
 Wire Wire Line
-	3100 3100 3250 3100
-Text Label 3150 3100 0    50   ~ 0
+	3100 3150 3250 3150
+Text Label 3150 3150 0    50   ~ 0
 D-
-NoConn ~ 3100 3200
-NoConn ~ 2700 3400
+NoConn ~ 3100 3250
+NoConn ~ 2700 3450
 $Comp
 L power:GND #PWR0105
 U 1 1 5C1F1C91
-P 2800 3400
-F 0 "#PWR0105" H 2800 3150 50  0001 C CNN
-F 1 "GND" H 2805 3227 50  0000 C CNN
-F 2 "" H 2800 3400 50  0001 C CNN
-F 3 "" H 2800 3400 50  0001 C CNN
-	1    2800 3400
-	1    0    0    -1
-$EndComp
-Wire Wire Line
-	3650 2950 3500 2950
-Text Label 3550 2950 0    50   ~ 0
+P 2800 3450
+F 0 "#PWR0105" H 2800 3200 50  0001 C CNN
+F 1 "GND" H 2805 3277 50  0000 C CNN
+F 2 "" H 2800 3450 50  0001 C CNN
+F 3 "" H 2800 3450 50  0001 C CNN
+	1    2800 3450
+	1    0    0    -1
+$EndComp
+Wire Wire Line
+	3650 3000 3500 3000
+Text Label 3550 3000 0    50   ~ 0
 D-
 Wire Wire Line
-	3650 3100 3500 3100
-Text Label 3500 3100 0    50   ~ 0
+	3650 3150 3500 3150
+Text Label 3500 3150 0    50   ~ 0
 D+
 $Comp
 L Connector:USB_B_Micro J4
 U 1 1 5C1F1B13
-P 2800 3000
-F 0 "J4" H 2855 3467 50  0000 C CNN
-F 1 "USB_B_Micro" H 2855 3376 50  0000 C CNN
-F 2 "Connector_USB:USB_Micro-B_Molex-105017-0001" H 2950 2950 50  0001 C CNN
-F 3 "~" H 2950 2950 50  0001 C CNN
-	1    2800 3000
+P 2800 3050
+F 0 "J4" H 2855 3517 50  0000 C CNN
+F 1 "USB_B_Micro" H 2855 3426 50  0000 C CNN
+F 2 "Connector_USB:USB_Micro-B_Molex-105017-0001" H 2950 3000 50  0001 C CNN
+F 3 "~" H 2950 3000 50  0001 C CNN
+	1    2800 3050
 	1    0    0    -1
 $EndComp
@@
 SNDRESET
 Wire Wire Line
-	5400 2150 5400 1850
-Wire Wire Line
-	5800 3400 6100 3400
-Wire Wire Line
-	4950 2150 4950 1700
-Wire Wire Line
-	3650 3250 3450 3250
-Wire Wire Line
-	3650 3400 3400 3400
-Wire Wire Line
-	5250 2150 5250 1800
-Wire Wire Line
-	5800 4000 6100 4000
-Text Label 5850 4000 0    50   ~ 0
+	5800 3300 6100 3300
+Wire Wire Line
+	4800 2050 4800 1700
+Wire Wire Line
+	3650 3300 3250 3300
+Wire Wire Line
+	3650 3450 3250 3450
+Wire Wire Line
+	5100 2050 5100 1700
+Wire Wire Line
+	5800 3900 6100 3900
+Text Label 5850 3900 0    50   ~ 0
 MOSI
-Text Label 4950 2050 1    50   ~ 0
+Text Label 4800 2000 1    50   ~ 0
 MISO
-Text Label 5250 2100 1    50   ~ 0
+Text Label 5100 2000 1    50   ~ 0
 SCLK
-Text Label 5850 3400 0    50   ~ 0
+Text Label 5850 3300 0    50   ~ 0
 SNDCS
-Text Label 5400 2150 1    50   ~ 0
+Text Label 5250 2000 1    50   ~ 0
 SNDRESET
-Text Label 3600 3250 2    50   ~ 0
+Text Label 3600 3300 2    50   ~ 0
 SNDDREQ
-Text Label 3600 3400 2    50   ~ 0
+Text Label 3600 3450 2    50   ~ 0
 SNDxDCS
 $Comp
@@
 $EndComp
 Wire Wire Line
-	3650 3700 3250 3700
-Wire Wire Line
-	3650 3550 3250 3550
-Text Label 3350 3550 0    50   ~ 0
+	3650 3750 3250 3750
+Wire Wire Line
+	3650 3600 3250 3600
+Text Label 3350 3600 0    50   ~ 0
 SWDIO
-Text Label 3300 3700 0    50   ~ 0
+Text Label 3300 3750 0    50   ~ 0
 SWDCLK
 $Comp
@@
 L touch-buttons:touch-slider-4pin U4
 U 1 1 5C2E4B1E
-P 6600 2900
-F 0 "U4" V 6554 3077 50  0000 L CNN
-F 1 "touch-slider-4pin" V 6645 3077 50  0000 L CNN
-F 2 "touch-buttons:TouchSlider-4_50x10mm" H 6600 2900 50  0001 C CNN
-F 3 "" H 6600 2900 50  0001 C CNN
-	1    6600 2900
+P 6600 2800
+F 0 "U4" V 6554 2977 50  0000 L CNN
+F 1 "touch-slider-4pin" V 6645 2977 50  0000 L CNN
+F 2 "touch-buttons:TouchSlider-4_50x10mm" H 6600 2800 50  0001 C CNN
+F 3 "" H 6600 2800 50  0001 C CNN
+	1    6600 2800
 	0    1    1    0
 $EndComp
 Wire Wire Line
-	6350 3200 5800 3200
-Wire Wire Line
-	5800 3200 5800 3250
-Wire Wire Line
-	6350 3000 5800 3000
-Wire Wire Line
-	5800 3000 5800 3100
-Wire Wire Line
-	5800 2950 5800 2900
-Wire Wire Line
-	5800 2900 6350 2900
-Wire Wire Line
-	6350 2900 6350 2800
-Wire Wire Line
-	6350 2600 6100 2600
-Wire Wire Line
-	6100 2600 6100 2800
-Wire Wire Line
-	6100 2800 5800 2800
+	6350 3100 5800 3100
+Wire Wire Line
+	6350 2900 5800 2900
+Wire Wire Line
+	5800 2800 6350 2800
+Wire Wire Line
+	6350 2800 6350 2700
+Wire Wire Line
+	6350 2500 6100 2500
+Wire Wire Line
+	6100 2500 6100 2700
+Wire Wire Line
+	6100 2700 5800 2700
 Wire Wire Line
 	7100 4500 7100 4950
@@
 Text Label 8450 4900 1    50   ~ 0
 TouchBTN2
-Text Label 6250 3700 2    50   ~ 0
+Text Label 6250 3600 2    50   ~ 0
 TouchBTN1
 Wire Wire Line
-	5800 3700 6350 3700
-Wire Wire Line
-	5800 3850 6350 3850
-Text Label 6300 3850 2    50   ~ 0
+	5800 3600 6350 3600
+Wire Wire Line
+	5800 3750 6350 3750
+Text Label 6250 3750 2    50   ~ 0
 TouchBTN2
 Wire Wire Line
-	3300 2800 3300 2700
-Connection ~ 3300 2800
-Wire Wire Line
-	3300 2800 3650 2800
-$Comp
-L power:+5V #PWR?
+	3300 2850 3300 2750
+Connection ~ 3300 2850
+Wire Wire Line
+	3300 2850 3650 2850
+$Comp
+L power:+5V #PWR0137
 U 1 1 5C30DCF7
-P 3300 2700
-F 0 "#PWR?" H 3300 2550 50  0001 C CNN
-F 1 "+5V" H 3315 2873 50  0000 C CNN
-F 2 "" H 3300 2700 50  0001 C CNN
-F 3 "" H 3300 2700 50  0001 C CNN
-	1    3300 2700
-	1    0    0    -1
-$EndComp
+P 3300 2750
+F 0 "#PWR0137" H 3300 2600 50  0001 C CNN
+F 1 "+5V" H 3315 2923 50  0000 C CNN
+F 2 "" H 3300 2750 50  0001 C CNN
+F 3 "" H 3300 2750 50  0001 C CNN
+	1    3300 2750
+	1    0    0    -1
+$EndComp
+Wire Wire Line
+	5800 3100 5800 3150
+Wire Wire Line
+	5800 2900 5800 3000
+Wire Wire Line
+	5800 2800 5800 2850
+Wire Wire Line
+	4650 1900 4650 2050
+Wire Wire Line
+	4500 1600 4500 2050
+Wire Wire Line
+	4350 1900 4350 2050
+Wire Wire Line
+	5250 1700 5250 2050
 $EndSCHEMATC

Commit message: Add power and indication LEDs
Parts:
- added D4, D5: LED, LED_SMD:LED_0603_1608Metric, symbol Device:LED
- added R12, R13: 470R, Resistor_SMD:R_0603_1608Metric, symbol Device:R
Connections:
- wire segments 56 -> 63
Changed lines of the file:
@@
 	0    1    1    0
 $EndComp
-Wire Wire Line
-	4950 4300 4950 4650
-Wire Wire Line
-	5100 4300 5100 4650
-Text Label 5100 4350 3    50   ~ 0
+Text Label 5100 4400 3    50   ~ 0
 DISPCS
 Text Label 4950 4350 3    50   ~ 0
 DISPDC
-Wire Wire Line
-	4350 4300 4350 4750
 Text Label 4500 4650 1    50   ~ 0
 DISPRST
 Text Label 4350 4700 1    50   ~ 0
 DISPBUSY
-Wire Wire Line
-	4500 4300 4500 4750
 $Sheet
 S 9100 1650 1750 1500
@@
 L power:GND #PWR0162
 U 1 1 5C2E4386
-P 5250 4300
-F 0 "#PWR0162" H 5250 4050 50  0001 C CNN
-F 1 "GND" H 5255 4127 50  0000 C CNN
-F 2 "" H 5250 4300 50  0001 C CNN
-F 3 "" H 5250 4300 50  0001 C CNN
-	1    5250 4300
+P 5250 4350
+F 0 "#PWR0162" H 5250 4100 50  0001 C CNN
+F 1 "GND" H 5255 4177 50  0000 C CNN
+F 2 "" H 5250 4350 50  0001 C CNN
+F 3 "" H 5250 4350 50  0001 C CNN
+	1    5250 4350
 	1    0    0    -1
 $EndComp
@@
 Wire Wire Line
 	5250 1700 5250 2050
+$Comp
+L Device:LED D5
+U 1 1 5C217B44
+P 6100 4200
+F 0 "D5" V 6045 4278 50  0000 L CNN
+F 1 "LED" V 6136 4278 50  0000 L CNN
+F 2 "LED_SMD:LED_0603_1608Metric" H 6100 4200 50  0001 C CNN
+F 3 "~" H 6100 4200 50  0001 C CNN
+	1    6100 4200
+	0    1    1    0
+$EndComp
+Wire Wire Line
+	5800 4050 6100 4050
+$Comp
+L Device:R R13
+U 1 1 5C218AF9
+P 6100 4650
+F 0 "R13" H 6170 4696 50  0000 L CNN
+F 1 "470R" H 6170 4605 50  0000 L CNN
+F 2 "Resistor_SMD:R_0603_1608Metric" V 6030 4650 50  0001 C CNN
+F 3 "~" H 6100 4650 50  0001 C CNN
+	1    6100 4650
+	1    0    0    -1
+$EndComp
+Wire Wire Line
+	6100 4350 6100 4500
+$Comp
+L power:+3.3V #PWR0138
+U 1 1 5C219A32
+P 6100 5000
+F 0 "#PWR0138" H 6100 4850 50  0001 C CNN
+F 1 "+3.3V" H 6115 5173 50  0000 C CNN
+F 2 "" H 6100 5000 50  0001 C CNN
+F 3 "" H 6100 5000 50  0001 C CNN
+	1    6100 5000
+	-1   0    0    1
+$EndComp
+Wire Wire Line
+	6100 4800 6100 5000
+$Comp
+L Device:LED D4
+U 1 1 5C21B86B
+P 2400 5600
+F 0 "D4" H 2392 5345 50  0000 C CNN
+F 1 "LED" H 2392 5436 50  0000 C CNN
+F 2 "LED_SMD:LED_0603_1608Metric" H 2400 5600 50  0001 C CNN
+F 3 "~" H 2400 5600 50  0001 C CNN
+	1    2400 5600
+	-1   0    0    1
+$EndComp
+$Comp
+L power:+3.3V #PWR0139
+U 1 1 5C21C876
+P 1750 5400
+F 0 "#PWR0139" H 1750 5250 50  0001 C CNN
+F 1 "+3.3V" H 1765 5573 50  0000 C CNN
+F 2 "" H 1750 5400 50  0001 C CNN
+F 3 "" H 1750 5400 50  0001 C CNN
+	1    1750 5400
+	1    0    0    -1
+$EndComp
+$Comp
+L Device:R R12
+U 1 1 5C21C8AD
+P 2000 5600
+F 0 "R12" V 1793 5600 50  0000 C CNN
+F 1 "470R" V 1884 5600 50  0000 C CNN
+F 2 "Resistor_SMD:R_0603_1608Metric" V 1930 5600 50  0001 C CNN
+F 3 "~" H 2000 5600 50  0001 C CNN
+	1    2000 5600
+	0    1    1    0
+$EndComp
+$Comp
+L power:GND #PWR0140
+U 1 1 5C21E734
+P 2800 5600
+F 0 "#PWR0140" H 2800 5350 50  0001 C CNN
+F 1 "GND" H 2805 5427 50  0000 C CNN
+F 2 "" H 2800 5600 50  0001 C CNN
+F 3 "" H 2800 5600 50  0001 C CNN
+	1    2800 5600
+	0    -1   -1   0
+$EndComp
+Wire Wire Line
+	2800 5600 2550 5600
+Wire Wire Line
+	2250 5600 2150 5600
+Wire Wire Line
+	1850 5600 1750 5600
+Wire Wire Line
+	1750 5600 1750 5400
+Wire Wire Line
+	5100 4350 5100 4700
+Wire Wire Line
+	4950 4350 4950 4700
+Wire Wire Line
+	4500 4350 4500 4700
+Wire Wire Line
+	4350 4350 4350 4700
 $EndSCHEMATC

Commit message: feat(pcb): add 2 neopixels
Parts:
- added D6, D7: WS2812B, LED_SMD:LED_WS2812B_PLCC4_5.0x5.0mm_P3.2mm, symbol LED:WS2812B
Connections:
- net labels added: NEOPIXEL
- wire segments 63 -> 72
- no-connect marks 3 -> 4
Changed lines of the file:
@@
 Wire Wire Line
 	4350 4350 4350 4700
+Text Label 4650 4750 1    50   ~ 0
+NEOPIXEL
+$Comp
+L LED:WS2812B D6
+U 1 1 5C2D8170
+P 4650 5350
+F 0 "D6" V 4604 5691 50  0000 L CNN
+F 1 "WS2812B" V 4695 5691 50  0000 L CNN
+F 2 "LED_SMD:LED_WS2812B_PLCC4_5.0x5.0mm_P3.2mm" H 4700 5050 50  0001 L TNN
+F 3 "https://cdn-shop.adafruit.com/datasheets/WS2812B.pdf" H 4750 4975 50  0001 L TNN
+	1    4650 5350
+	0    1    1    0
+$EndComp
+Wire Wire Line
+	4650 4350 4650 5050
+$Comp
+L LED:WS2812B D7
+U 1 1 5C2DBAD4
+P 4650 6000
+F 0 "D7" V 4604 6341 50  0000 L CNN
+F 1 "WS2812B" V 4695 6341 50  0000 L CNN
+F 2 "LED_SMD:LED_WS2812B_PLCC4_5.0x5.0mm_P3.2mm" H 4700 5700 50  0001 L TNN
+F 3 "https://cdn-shop.adafruit.com/datasheets/WS2812B.pdf" H 4750 5625 50  0001 L TNN
+	1    4650 6000
+	0    1    1    0
+$EndComp
+Wire Wire Line
+	4650 5650 4650 5700
+Wire Wire Line
+	4650 6300 4650 6350
+Wire Wire Line
+	4950 6000 4950 6300
+Connection ~ 4950 6000
+Wire Wire Line
+	4950 6000 4950 5350
+Wire Wire Line
+	4350 5350 4350 6000
+Wire Wire Line
+	4350 6000 4350 6350
+Connection ~ 4350 6000
+$Comp
+L power:+3.3V #PWR0163
+U 1 1 5C2E9FF8
+P 5400 6300
+F 0 "#PWR0163" H 5400 6150 50  0001 C CNN
+F 1 "+3.3V" H 5415 6473 50  0000 C CNN
+F 2 "" H 5400 6300 50  0001 C CNN
+F 3 "" H 5400 6300 50  0001 C CNN
+	1    5400 6300
+	0    1    1    0
+$EndComp
+Wire Wire Line
+	4950 6300 5400 6300
+$Comp
+L power:GND #PWR0164
+U 1 1 5C2EB8EF
+P 3900 6350
+F 0 "#PWR0164" H 3900 6100 50  0001 C CNN
+F 1 "GND" H 3905 6177 50  0000 C CNN
+F 2 "" H 3900 6350 50  0001 C CNN
+F 3 "" H 3900 6350 50  0001 C CNN
+	1    3900 6350
+	0    1    1    0
+$EndComp
+Wire Wire Line
+	4350 6350 3900 6350
+NoConn ~ 4650 6350
 $EndSCHEMATC
