File: pcb/badge/badge.sch (KiCad schematic (older format))
At the start: 17 parts, among them J2 SAO_CONN, J4 USB_B_Micro, J6 Conn_ARM_JTAG_SWD_10, SW1 SW_Push, SW2 SW_Push, SW3 SW_Push, U3 E73-2G4M08S1C, U4 TPS610986DSET

Commit message: Add Flash memory + connect battery and step-up IC
Parts:
- added C12: 100uF, Capacitor_Tantalum_SMD:CP_EIA-3216-18_Kemet-A, symbol Device:CP1
- added C16: 10uF, Capacitor_SMD:C_0603_1608Metric, symbol Device:C
- added C36: 1uF, Capacitor_SMD:C_0603_1608Metric, symbol Device:C
- added C37, C4, C6: 100nF, Capacitor_SMD:C_0603_1608Metric, symbol Device:C
- added L2: 4.7uH, Inductor_SMD:L_1210_3225Metric, symbol pspice:INDUCTOR
- added R14: 400R, Resistor_SMD:R_0603_1608Metric, symbol Device:R
- added SW4: SW_SPDT, Button_Switch_THT:SW_CuK_OS102011MA1QN1_SPDT_Angled, symbol Switch:SW_SPDT
- added U2: AMS1117-3.3, Package_TO_SOT_SMD:SOT-223-3_TabPin2, symbol Regulator_Linear:AMS1117-3.3
- added U5: GD25Q16C, Package_SO:SOIC-8_3.9x4.9mm_P1.27mm, symbol Memory_Flash:AT25SF081-SSHD-X
Connections:
- net labels added: +3V3, FLASH_SO, V_BAT
- wire segments 79 -> 119
- no-connect marks 4 -> 5
Other:
- moved on the sheet: BT1, D4, R12, U4

Commit message: Add vibrator
Parts:
- added BZ1: Buzzer, symbol Device:Buzzer
- added Q2: Si1308EDL, Package_TO_SOT_SMD:SOT-323_SC-70, symbol Device:Q_NMOS_GSD
Connections:
- net labels added: VIBRATOR
- wire segments 119 -> 123
- no-connect marks 5 -> 4
Changed lines of the file:
@@
 Wire Wire Line
 	4350 6200 3900 6200
-NoConn ~ 1450 7700
 $Comp
 L LED:WS2812B D8
@@
 NoConn ~ 9650 5700
 $Comp
-L power:+3V3 #PWR?
+L power:+3V3 #PWR0173
 U 1 1 5C557749
 P 9650 5800
-F 0 "#PWR?" H 9650 5650 50  0001 C CNN
+F 0 "#PWR0173" H 9650 5650 50  0001 C CNN
 F 1 "+3V3" V 9665 5928 50  0000 L CNN
 F 2 "" H 9650 5800 50  0001 C CNN
@@
 	0    1    1    0
 $EndComp
+$Comp
+L Device:Buzzer BZ1
+U 1 1 5C558E48
+P 1750 6600
+F 0 "BZ1" H 1903 6629 50  0000 L CNN
+F 1 "Buzzer" H 1903 6538 50  0000 L CNN
+F 2 "" V 1725 6700 50  0001 C CNN
+F 3 "~" V 1725 6700 50  0001 C CNN
+	1    1750 6600
+	1    0    0    -1
+$EndComp
+$Comp
+L power:+3V3 #PWR0174
+U 1 1 5C558FF1
+P 1600 6500
+F 0 "#PWR0174" H 1600 6350 50  0001 C CNN
+F 1 "+3V3" V 1615 6628 50  0000 L CNN
+F 2 "" H 1600 6500 50  0001 C CNN
+F 3 "" H 1600 6500 50  0001 C CNN
+	1    1600 6500
+	0    -1   -1   0
+$EndComp
+Wire Wire Line
+	1600 6500 1650 6500
+$Comp
+L Device:Q_NMOS_GSD Q?
+U 1 1 5C560203
+P 1300 6900
+AR Path="/5C21B929/5C560203" Ref="Q?"  Part="1"
+AR Path="/5C560203" Ref="Q2"  Part="1"
+F 0 "Q2" H 1505 6946 50  0000 L CNN
+F 1 "Si1308EDL" H 1505 6855 50  0000 L CNN
+F 2 "Package_TO_SOT_SMD:SOT-323_SC-70" H 1500 7000 50  0001 C CNN
+F 3 "~" H 1300 6900 50  0001 C CNN
+	1    1300 6900
+	1    0    0    -1
+$EndComp
+Wire Wire Line
+	1650 6700 1400 6700
+$Comp
+L power:GND #PWR0175
+U 1 1 5C567B60
+P 1400 7100
+F 0 "#PWR0175" H 1400 6850 50  0001 C CNN
+F 1 "GND" H 1405 6927 50  0000 C CNN
+F 2 "" H 1400 7100 50  0001 C CNN
+F 3 "" H 1400 7100 50  0001 C CNN
+	1    1400 7100
+	1    0    0    -1
+$EndComp
+Wire Wire Line
+	1100 6900 800  6900
+Text Label 850  6900 0    50   ~ 0
+VIBRATOR
+Wire Wire Line
+	4050 4350 4050 4750
+Text Label 4050 4750 1    50   ~ 0
+VIBRATOR
 $EndSCHEMATC

Commit message: PCB routing
Parts:
- BZ1: footprint (none) -> Connector_PinHeader_2.00mm:PinHeader_1x02_P2.00mm_Vertical
Changed lines of the file:
@@
 F 0 "BZ1" H 1903 6629 50  0000 L CNN
 F 1 "Buzzer" H 1903 6538 50  0000 L CNN
-F 2 "" V 1725 6700 50  0001 C CNN
+F 2 "Connector_PinHeader_2.00mm:PinHeader_1x02_P2.00mm_Vertical" V 1725 6700 50  0001 C CNN
 F 3 "~" V 1725 6700 50  0001 C CNN
 	1    1750 6600

Commit message: fix(pcb): change step-up resistor to 390R
400R is not a common value, 390 is.
Parts:
- R14: value 400R -> 390R
Changed lines of the file:
@@
 P 8100 5850
 F 0 "R14" H 8170 5896 50  0000 L CNN
-F 1 "400R" H 8170 5805 50  0000 L CNN
+F 1 "390R" H 8170 5805 50  0000 L CNN
 F 2 "Resistor_SMD:R_0603_1608Metric" V 8030 5850 50  0001 C CNN
 F 3 "~" H 8100 5850 50  0001 C CNN
@@
 F 3 "" H 8100 6400 50  0001 C CNN
 	1    8100 6400
-	1    0    0    -1
+	0    1    1    0
 $EndComp
 Wire Wire Line

Commit message: refactor(pcb): move power schematic to a separate sheet
Parts:
- removed BT1: Battery_Cell, AA_battery_clip:BK-53_MPD_AAClip, symbol Device:Battery_Cell
- removed C12: 100uF, Capacitor_Tantalum_SMD:CP_EIA-3216-18_Kemet-A, symbol Device:CP1
- removed C16: 10uF, Capacitor_SMD:C_0603_1608Metric, symbol Device:C
- removed C36: 1uF, Capacitor_SMD:C_0603_1608Metric, symbol Device:C
- removed C37, C4, C6: 100nF, Capacitor_SMD:C_0603_1608Metric, symbol Device:C
- removed L2: 4.7uH, Inductor_SMD:L_1210_3225Metric, symbol pspice:INDUCTOR
- removed R14: 390R, Resistor_SMD:R_0603_1608Metric, symbol Device:R
- removed SW4: SW_SPDT, Button_Switch_THT:SW_CuK_OS102011MA1QN1_SPDT_Angled, symbol Switch:SW_SPDT
- removed U2: AMS1117-3.3, Package_TO_SOT_SMD:SOT-223-3_TabPin2, symbol Regulator_Linear:AMS1117-3.3
- removed U4: TPS610986DSET, SON50P150X150X80-6N:SON50P150X150X80-6N, symbol regulator:TPS610986DSET
Connections:
- wire segments 123 -> 98
- no-connect marks 4 -> 3

Commit message: feat(pcb): add LIS2DH12TR accelerometer
Parts:
- added C38: 10uF, Capacitor_SMD:C_0603_1608Metric, symbol Device:C
- added C39: 100nF, Capacitor_SMD:C_0603_1608Metric, symbol Device:C
- added U7: LIS2DH12TR, Package_LGA:LGA-12_2x2mm_P0.5mm, symbol LIS2DH12TR:LIS2DH12TR
Connections:
- wire segments 98 -> 119
- no-connect marks 3 -> 5
Changed lines of the file:
@@
 Text Label 8750 5250 0    50   ~ 0
 V_BAT
+Wire Wire Line
+	6800 5300 6700 5300
+Wire Wire Line
+	6700 5300 6700 5200
+$Comp
+L power:+3.3V #PWR0177
+U 1 1 5C4C3434
+P 6700 5200
+F 0 "#PWR0177" H 6700 5050 50  0001 C CNN
+F 1 "+3.3V" H 6715 5373 50  0000 C CNN
+F 2 "" H 6700 5200 50  0001 C CNN
+F 3 "" H 6700 5200 50  0001 C CNN
+	1    6700 5200
+	1    0    0    -1
+$EndComp
+NoConn ~ 8200 5300
+NoConn ~ 8200 5400
+$Comp
+L power:GND #PWR0178
+U 1 1 5C4C88FE
+P 8250 6050
+F 0 "#PWR0178" H 8250 5800 50  0001 C CNN
+F 1 "GND" V 8255 5922 50  0000 R CNN
+F 2 "" H 8250 6050 50  0001 C CNN
+F 3 "" H 8250 6050 50  0001 C CNN
+	1    8250 6050
+	1    0    0    -1
+$EndComp
+Wire Wire Line
+	8250 6050 8250 6000
+Wire Wire Line
+	8250 6000 8200 6000
+Wire Wire Line
+	6800 5500 6500 5500
+Text Label 6500 5500 0    50   ~ 0
+SCL
+Wire Wire Line
+	6800 5600 6500 5600
+Text Label 6500 5600 0    50   ~ 0
+SDA
+Wire Wire Line
+	8200 5900 8250 5900
+Wire Wire Line
+	8250 5900 8250 6000
+Connection ~ 8250 6000
+$Comp
+L power:+3.3V #PWR0179
+U 1 1 5C4D72C9
+P 8400 4950
+F 0 "#PWR0179" H 8400 4800 50  0001 C CNN
+F 1 "+3.3V" H 8415 5123 50  0000 C CNN
+F 2 "" H 8400 4950 50  0001 C CNN
+F 3 "" H 8400 4950 50  0001 C CNN
+	1    8400 4950
+	1    0    0    -1
+$EndComp
+Wire Wire Line
+	8400 4950 8400 5000
+Wire Wire Line
+	8400 5000 8300 5000
+Wire Wire Line
+	8300 5100 8300 5000
+Connection ~ 8300 5000
+Wire Wire Line
+	8300 5000 8200 5000
+$Comp
+L Device:C C38
+U 1 1 5C4DE596
+P 8400 5500
+F 0 "C38" H 8515 5546 50  0000 L CNN
+F 1 "10uF" H 8515 5455 50  0000 L CNN
+F 2 "Capacitor_SMD:C_0603_1608Metric" H 8438 5350 50  0001 C CNN
+F 3 "~" H 8400 5500 50  0001 C CNN
+	1    8400 5500
+	1    0    0    -1
+$EndComp
+$Comp
+L Device:C C39
+U 1 1 5C4DE630
+P 8800 5500
+F 0 "C39" H 8915 5546 50  0000 L CNN
+F 1 "100nF" H 8915 5455 50  0000 L CNN
+F 2 "Capacitor_SMD:C_0603_1608Metric" H 8838 5350 50  0001 C CNN
+F 3 "~" H 8800 5500 50  0001 C CNN
+	1    8800 5500
+	1    0    0    -1
+$EndComp
+Wire Wire Line
+	8400 5100 8400 5350
+Wire Wire Line
+	8200 5100 8300 5100
+Connection ~ 8300 5100
+Wire Wire Line
+	8300 5100 8400 5100
+Connection ~ 8400 5350
+Wire Wire Line
+	8250 5650 8250 5900
+Connection ~ 8400 5650
+Wire Wire Line
+	8400 5650 8250 5650
+Connection ~ 8250 5900
+Wire Wire Line
+	8400 5350 8800 5350
+Wire Wire Line
+	8400 5650 8800 5650
+$Comp
+L power:GND #PWR0180
+U 1 1 5C4F7416
+P 6700 5750
+F 0 "#PWR0180" H 6700 5500 50  0001 C CNN
+F 1 "GND" V 6705 5622 50  0000 R CNN
+F 2 "" H 6700 5750 50  0001 C CNN
+F 3 "" H 6700 5750 50  0001 C CNN
+	1    6700 5750
+	1    0    0    -1
+$EndComp
+$Comp
+L LIS2DH12TR:LIS2DH12TR U7
+U 1 1 5C4C0967
+P 7500 5500
+F 0 "U7" H 7500 6270 50  0000 C CNN
+F 1 "LIS2DH12TR" H 7500 6179 50  0000 C CNN
+F 2 "Package_LGA:LGA-12_2x2mm_P0.5mm" H 7500 5500 50  0001 L BNN
+F 3 "497-14851-1-ND" H 7500 5500 50  0001 L BNN
+F 4 "LGA-12 STMicroelectronics" H 7500 5500 50  0001 L BNN "Field4"
+F 5 "https://www.digikey.com/product-detail/en/stmicroelectronics/LIS2DH12TR/497-14851-1-ND/4899838?utm_source=snapeda&utm_medium=aggregator&utm_campaign=symbol" H 7500 5500 50  0001 L BNN "Field5"
+F 6 "STMicroelectronics" H 7500 5500 50  0001 L BNN "Field6"
+F 7 "LIS2DH12TR" H 7500 5500 50  0001 L BNN "Field7"
+F 8 "MEMS digital output motion sensor: ultra low-power high performance 3-axes femto accelerometer" H 7500 5500 50  0001 L BNN "Field8"
+	1    7500 5500
+	1    0    0    -1
+$EndComp
+Wire Wire Line
+	6800 5700 6700 5700
+Wire Wire Line
+	6700 5700 6700 5750
 $EndSCHEMATC

Commit message: feat(pcb): add test-points for programming
add GND, SWCLK, SWDIO, 3V3 with standard 0.1" spacing
Parts:
- added TP1: TP_3V3, TestPoint:TestPoint_Pad_D1.5mm, symbol Connector:TestPoint
- added TP2: TP_SWDIO, TestPoint:TestPoint_Pad_D1.5mm, symbol Connector:TestPoint
- added TP3: TP_SWCLK, TestPoint:TestPoint_Pad_D1.5mm, symbol Connector:TestPoint
- added TP4: TP_GND, TestPoint:TestPoint_Pad_D1.5mm, symbol Connector:TestPoint
Connections:
- wire segments 119 -> 123
Changed lines of the file:
@@
 Wire Wire Line
 	6700 5700 6700 5750
+$Comp
+L Connector:TestPoint TP1
+U 1 1 5C5F862C
+P 4950 900
+F 0 "TP1" H 5008 1020 50  0000 L CNN
+F 1 "TP_3V3" H 5008 929 50  0000 L CNN
+F 2 "TestPoint:TestPoint_Pad_D1.5mm" H 5150 900 50  0001 C CNN
+F 3 "~" H 5150 900 50  0001 C CNN
+	1    4950 900
+	1    0    0    -1
+$EndComp
+$Comp
+L power:+3.3V #PWR0181
+U 1 1 5C5F8E6E
+P 4950 1100
+F 0 "#PWR0181" H 4950 950 50  0001 C CNN
+F 1 "+3.3V" H 4965 1273 50  0000 C CNN
+F 2 "" H 4950 1100 50  0001 C CNN
+F 3 "" H 4950 1100 50  0001 C CNN
+	1    4950 1100
+	-1   0    0    1
+$EndComp
+Wire Wire Line
+	4950 900  4950 1100
+$Comp
+L Connector:TestPoint TP2
+U 1 1 5C5FC8D2
+P 5400 900
+F 0 "TP2" H 5458 1020 50  0000 L CNN
+F 1 "TP_SWDIO" H 5458 929 50  0000 L CNN
+F 2 "TestPoint:TestPoint_Pad_D1.5mm" H 5600 900 50  0001 C CNN
+F 3 "~" H 5600 900 50  0001 C CNN
+	1    5400 900
+	1    0    0    -1
+$EndComp
+$Comp
+L Connector:TestPoint TP3
+U 1 1 5C5FC94C
+P 5850 900
+F 0 "TP3" H 5908 1020 50  0000 L CNN
+F 1 "TP_SWCLK" H 5908 929 50  0000 L CNN
+F 2 "TestPoint:TestPoint_Pad_D1.5mm" H 6050 900 50  0001 C CNN
+F 3 "~" H 6050 900 50  0001 C CNN
+	1    5850 900
+	1    0    0    -1
+$EndComp
+$Comp
+L Connector:TestPoint TP4
+U 1 1 5C5FC99E
+P 6300 900
+F 0 "TP4" H 6358 1020 50  0000 L CNN
+F 1 "TP_GND" H 6358 929 50  0000 L CNN
+F 2 "TestPoint:TestPoint_Pad_D1.5mm" H 6500 900 50  0001 C CNN
+F 3 "~" H 6500 900 50  0001 C CNN
+	1    6300 900
+	1    0    0    -1
+$EndComp
+Wire Wire Line
+	5400 900  5400 1250
+Wire Wire Line
+	5850 900  5850 1250
+$Comp
+L power:GND #PWR0182
+U 1 1 5C607C1C
+P 6300 1100
+F 0 "#PWR0182" H 6300 850 50  0001 C CNN
+F 1 "GND" H 6305 927 50  0000 C CNN
+F 2 "" H 6300 1100 50  0001 C CNN
+F 3 "" H 6300 1100 50  0001 C CNN
+	1    6300 1100
+	1    0    0    -1
+$EndComp
+Wire Wire Line
+	6300 900  6300 1100
+Text Label 5850 950  3    50   ~ 0
+SWDCLK
+Text Label 5400 1250 1    50   ~ 0
+SWDIO
 $EndSCHEMATC

Commit message: fix(pcb): add capacitor for the buzzer
Parts:
- added C40: 10uF, Capacitor_SMD:C_0603_1608Metric, symbol Device:C
Connections:
- wire segments 123 -> 127
Changed lines of the file:
@@
 L power:+3V3 #PWR0174
 U 1 1 5C558FF1
-P 1600 6500
-F 0 "#PWR0174" H 1600 6350 50  0001 C CNN
-F 1 "+3V3" V 1615 6628 50  0000 L CNN
-F 2 "" H 1600 6500 50  0001 C CNN
-F 3 "" H 1600 6500 50  0001 C CNN
-	1    1600 6500
+P 1250 6500
+F 0 "#PWR0174" H 1250 6350 50  0001 C CNN
+F 1 "+3V3" V 1265 6628 50  0000 L CNN
+F 2 "" H 1250 6500 50  0001 C CNN
+F 3 "" H 1250 6500 50  0001 C CNN
+	1    1250 6500
 	0    -1   -1   0
 $EndComp
 Wire Wire Line
-	1600 6500 1650 6500
+	1250 6500 1450 6500
 $Comp
 L Device:Q_NMOS_GSD Q?
@@
 Text Label 5400 1250 1    50   ~ 0
 SWDIO
+$Comp
+L Device:C C40
+U 1 1 5CD38C66
+P 1450 6200
+F 0 "C40" H 1565 6246 50  0000 L CNN
+F 1 "10uF" H 1565 6155 50  0000 L CNN
+F 2 "Capacitor_SMD:C_0603_1608Metric" H 1488 6050 50  0001 C CNN
+F 3 "~" H 1450 6200 50  0001 C CNN
+	1    1450 6200
+	1    0    0    -1
+$EndComp
+Connection ~ 1450 6500
+Wire Wire Line
+	1450 6500 1650 6500
+Wire Wire Line
+	1450 6350 1450 6500
+$Comp
+L power:GND #PWR0183
+U 1 1 5CD486FF
+P 1300 6000
+F 0 "#PWR0183" H 1300 5750 50  0001 C CNN
+F 1 "GND" H 1305 5827 50  0000 C CNN
+F 2 "" H 1300 6000 50  0001 C CNN
+F 3 "" H 1300 6000 50  0001 C CNN
+	1    1300 6000
+	0    1    1    0
+$EndComp
+Wire Wire Line
+	1300 6000 1450 6000
+Wire Wire Line
+	1450 6000 1450 6050
 $EndSCHEMATC
