File: pcb/badge/badge.kicad_pcb (KiCad board)
At the start: 2 copper layers, 80 x 57.1 mm, 69 parts, among them IC1 VS1053B, J1 AudioJack4, J3 Conn_01x08_Male, J4 USB_B_Micro, J5 Conn_01x08_Male, J6 Conn_01x04_Male, J7 PFC24/0.5mm, Q1 Si1308EDL, U1 AMS1117-1.8, U2 AMS1117-3.3, U3 E73-2G4M08S1C, U4 touch-slider-4pin, U5 touch-button, U6 touch-button, Y1 12.288M

Commit message: Add logo footprint
Parts:
- added svg2mod: G***, logo:aram-logo, B.Cu at (102.3, 104.2)
Changed lines of the file:
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@@
     (tracks 733)
     (zones 0)
-    (modules 69)
+    (modules 70)
     (nets 74)
   )
@@
     )
   )
+  (module logo:aram-logo (layer B.Cu)
+    (at 102.3 104.2 180)
+    (descr "Imported from Telegram Desktopram-logo.svg")
+    (tags svg2mod)
+    (attr smd)
+    (fp_text reference svg2mod (at 0 21.653108 180) (layer B.SilkS) hide
+      (effects (font (size 1.524 1.524) (thickness 0.3048)) (justify mirror))
+    )
+    (fp_text value G*** (at 0 -21.653108 180) (layer B.SilkS) hide
+      (effects (font (size 1.524 1.524) (thickness 0.3048)) (justify mirror))
+    )
+    (fp_poly (pts (xy -5.809042 -5.370484) (xy -6.627044 -4.401669) (xy -8.158921 -3.237623) (xy -10.577607 -2.119336)
+      (xy -11.979841 -1.506318) (xy -13.040926 -0.900554) (xy -14.065989 -0.009911) (xy -14.885068 0.939176)
+      (xy -15.441741 2.410396) (xy -15.42773 4.007969) (xy -14.789449 5.862331) (xy -13.594255 7.37463)
+      (xy -11.88408 8.506703) (xy -9.700851 9.220388) (xy -7.833707 9.369401) (xy -6.135312 9.005851)
+      (xy -4.559903 8.119942) (xy -3.24353 6.304094) (xy -3.283396 5.041207) (xy -4.147343 4.160425)
+      (xy -5.518839 3.77158) (xy -6.62072 4.199322) (xy -7.216552 6.213765) (xy -7.353423 7.317818)
+      (xy -8.136189 8.067767) (xy -9.083626 8.23129) (xy -10.051616 8.047954) (xy -10.957341 7.261952)
+      (xy -11.479615 6.088571) (xy -11.273631 4.029463) (xy -10.596285 2.443278) (xy -9.651481 0.951577)
+      (xy -8.534065 -0.295895) (xy -6.953758 -1.882196) (xy -5.740178 -3.531585) (xy -4.625941 -5.427196)
+      (xy -4.950321 -5.598367) (xy -5.809042 -5.370484)) (layer B.SilkS) (width 0.022927))
+    (fp_poly (pts (xy 5.07725 -5.70427) (xy 4.671926 -5.4434) (xy 5.796075 -3.53) (xy 6.96011 -1.943962)
+      (xy 8.176026 -0.715439) (xy 9.651995 0.862081) (xy 10.823299 2.845304) (xy 11.538524 5.101192)
+      (xy 11.178013 6.890779) (xy 10.051809 7.991539) (xy 9.112033 8.172954) (xy 7.422297 7.338145)
+      (xy 7.223528 6.088571) (xy 6.906983 4.444578) (xy 5.521097 3.690979) (xy 3.754123 4.333933)
+      (xy 3.218467 5.340582) (xy 3.542 6.902326) (xy 4.92865 8.30663) (xy 6.865174 9.175026)
+      (xy 8.230769 9.305353) (xy 9.696397 9.170055) (xy 11.76383 8.502265) (xy 13.404987 7.480027)
+      (xy 14.599688 6.12029) (xy 15.327756 4.440003) (xy 15.491073 3.130334) (xy 15.353273 1.944135)
+      (xy 14.840746 0.830327) (xy 14.013155 -0.168614) (xy 12.625807 -1.216144) (xy 10.549397 -2.195542)
+      (xy 9.039209 -2.833793) (xy 8.103634 -3.329637) (xy 6.781406 -4.310574) (xy 5.76635 -5.516889)
+      (xy 5.506181 -5.895365) (xy 5.07725 -5.704273) (xy 5.07725 -5.70427)) (layer B.SilkS) (width 0.022927))
+    (fp_poly (pts (xy -0.421301 -7.91618) (xy -0.530789 -7.281523) (xy -0.782175 -5.689947) (xy -1.264937 -2.655585)
+      (xy -1.846631 1.019667) (xy -2.244117 3.611324) (xy -2.49317 5.372342) (xy -2.629565 6.55568)
+      (xy -2.689077 7.414296) (xy -2.619487 9.119391) (xy -2.23512 10.43244) (xy -1.193641 11.494829)
+      (xy -0.197449 11.670378) (xy 0.741988 11.542196) (xy 1.809689 10.694056) (xy 2.43349 9.106714)
+      (xy 2.55992 7.216848) (xy 2.550262 6.354857) (xy 2.479867 5.436651) (xy 2.282621 3.970659)
+      (xy 1.892406 1.465311) (xy 1.243106 -2.570964) (xy 0.766473 -5.528021) (xy 0.495758 -7.211007)
+      (xy 0.371676 -7.986699) (xy -0.013382 -7.986699) (xy -0.421301 -7.91618)) (layer B.SilkS) (width 0.022927))
+    (fp_poly (pts (xy 3.306857 -10.917486) (xy 2.195203 -10.259566) (xy 1.786316 -9.632833) (xy 1.607796 -8.717153)
+      (xy 1.818484 -7.751992) (xy 2.923388 -6.670252) (xy 3.836143 -6.491729) (xy 4.748897 -6.670252)
+      (xy 5.853803 -7.751992) (xy 6.064492 -8.720079) (xy 5.853803 -9.688165) (xy 5.077575 -10.594335)
+      (xy 3.963035 -10.951698) (xy 3.306857 -10.917486)) (layer B.SilkS) (width 0.022927))
+    (fp_poly (pts (xy -4.478261 -10.917486) (xy -5.589914 -10.259566) (xy -5.998802 -9.632833) (xy -6.177323 -8.717153)
+      (xy -5.966634 -7.751992) (xy -4.861729 -6.670252) (xy -3.948975 -6.491729) (xy -3.03622 -6.670252)
+      (xy -1.931314 -7.751992) (xy -1.720626 -8.720079) (xy -1.931314 -9.688165) (xy -2.707544 -10.594335)
+      (xy -3.822083 -10.951698) (xy -4.478261 -10.917486)) (layer B.SilkS) (width 0.022927))
+    (fp_poly (pts (xy -0.529288 -14.471561) (xy -1.640941 -13.813644) (xy -2.049829 -13.18691) (xy -2.22835 -12.271228)
+      (xy -2.017662 -11.306067) (xy -0.912756 -10.224327) (xy -0.000001 -10.045804) (xy 0.912753 -10.224327)
+      (xy 2.017659 -11.306067) (xy 2.228348 -12.274154) (xy 2.017659 -13.24224) (xy 1.241429 -14.14841)
+      (xy 0.126891 -14.505773) (xy -0.529288 -14.471561)) (layer B.SilkS) (width 0.022927))
+    (fp_poly (pts (xy 2.193321 -16.928819) (xy -1.212901 -18.557734) (xy -3.657049 -18.222757) (xy -5.943171 -17.611369)
+      (xy -8.15181 -16.702031) (xy -10.066564 -15.627478) (xy -11.826144 -14.344682) (xy -13.415801 -12.873035)
+      (xy -14.820786 -11.231929) (xy -16.026348 -9.440755) (xy -17.017739 -7.518908) (xy -17.78021 -5.485778)
+      (xy -18.29901 -3.360759) (xy -18.529386 -1.733978) (xy -18.585929 0.024075) (xy -18.529386 1.782129)
+      (xy -18.29901 3.408911) (xy -17.765703 5.580366) (xy -16.980964 7.647307) (xy -15.962528 9.591609)
+      (xy -14.728131 11.39515) (xy -13.295508 13.039807) (xy -11.682393 14.507457) (xy -9.906524 15.779977)
+      (xy -7.985633 16.839245) (xy -5.937458 17.667136) (xy -3.779733 18.245529) (xy -1.9617 18.535488)
+      (xy -0.000001 18.605108) (xy 1.961698 18.535488) (xy 3.77973 18.245529) (xy 5.937455 17.667136)
+      (xy 7.985631 16.839245) (xy 9.906521 15.779977) (xy 11.682391 14.507457) (xy 13.295506 13.039807)
+      (xy 14.72813 11.39515) (xy 15.962527 9.591609) (xy 16.980963 7.647307) (xy 17.765701 5.580366)
+      (xy 18.299007 3.408911) (xy 18.529385 1.782129) (xy 18.585929 0.024075) (xy 18.529385 -1.733978)
+      (xy 18.299007 -3.360759) (xy 17.748507 -5.585106) (xy 16.925354 -7.720838) (xy 15.844331 -9.740337)
+      (xy 14.520219 -11.61599) (xy 12.9678 -13.32018) (xy 11.115389 -14.899864) (xy 9.103703 -16.209844)
+      (xy 6.947097 -17.243242) (xy 4.659929 -17.993177) (xy 2.256554 -18.452771) (xy 0.491002 -18.555155)
+      (xy -1.212901 -18.557734) (xy 2.193321 -16.928819) (xy 4.37544 -16.489864) (xy 6.447802 -15.788106)
+      (xy 8.423214 -14.818256) (xy 10.314483 -13.575025) (xy 11.956802 -12.114416) (xy 13.425203 -10.525323)
+      (xy 14.795608 -8.479784) (xy 15.849013 -6.333201) (xy 16.582258 -4.095213) (xy 16.992186 -1.77546)
+      (xy 17.075639 0.616421) (xy 16.880374 2.750896) (xy 16.438158 4.79309) (xy 15.74597 6.751543)
+      (xy 14.800795 8.634795) (xy 13.599612 10.451387) (xy 12.049534 12.186438) (xy 10.314483 13.736515)
+      (xy 8.417834 14.984269) (xy 6.445936 15.951158) (xy 4.365623 16.650825) (xy 2.143727 17.09691)
+      (xy -0.056416 17.201411) (xy -2.256558 17.09691) (xy -4.179093 16.728442) (xy -5.97833 16.176781)
+      (xy -7.691281 15.430579) (xy -9.324271 14.511192) (xy -10.75319 13.473672) (xy -12.161055 12.185133)
+      (xy -13.449595 10.777268) (xy -14.487117 9.348349) (xy -15.406507 7.715356) (xy -16.146494 6.026272)
+      (xy -16.687137 4.2872) (xy -17.032864 2.48042) (xy -17.188104 0.588215) (xy -17.101203 -1.799241)
+      (xy -16.689385 -4.114399) (xy -15.955959 -6.347183) (xy -14.904237 -8.487517) (xy -13.537526 -10.525323)
+      (xy -12.159821 -12.023141) (xy -10.662228 -13.400534) (xy -8.989745 -14.551688) (xy -7.251733 -15.484803)
+      (xy -5.439015 -16.203517) (xy -3.542413 -16.711469) (xy -1.552749 -17.012299) (xy 0.311043 -17.036557)
+      (xy 2.193321 -16.928819)) (layer B.SilkS) (width 0.022927))
+  )
   (gr_text SWD (at 52.43 87.33) (layer F.SilkS)

Commit message: Make logo smaller
Resize with `-f 0.5` parameter for svg2mod
Parts:
- ?: renamed from svg2mod; value G*** -> (none)
- moved ? 24.9 mm to (109.0, 80.2)
