File: pcb/badge/badge.kicad_pcb (KiCad board)
At the start: 2 copper layers, 80 x 57.1 mm, 71 parts, among them IC1 VS1053B, J1 AudioJack4, J3 Conn_01x08_Male, J4 USB_B_Micro, J5 Conn_01x08_Male, J6 Conn_01x04_Male, J7 PFC24/0.5mm, Q1 Si1308EDL, U1 AMS1117-1.8, U2 AMS1117-3.3, U3 E73-2G4M08S1C, U4 touch-slider-4pin, U5 touch-button, U6 touch-button, Y1 12.288M

Commit message: Fix reversed connector for EPD
Parts:
- J1: footprint audio:Jack_3.5mm_PJ320D_Horizontal -> connectors:Jack_3.5mm_PJ320D_Horizontal
- J7: footprint Connector_FFC-FPC:Hirose_FH12-24S-0.5SH_1x24-1MP_P0.50mm_Horizontal -> connectors:EPD-FPC-1x24-P0.50mm_Horizontal
- moved C33 34.3 mm to (108.6, 104.1)
- moved C32 29.2 mm to (108.4, 101.6)
- moved C31 23.9 mm to (108.4, 99.1)
- moved C26 22.1 mm to (114.8, 107.3), turned to 0 degrees
- moved Q1 22.0 mm to (108.5, 75.7)
- moved R10 21.9 mm to (108.4, 78.7)
- moved C30 18.8 mm to (108.6, 96.5)
- moved L1 15.0 mm to (100.3, 75.6), turned to 0 degrees
- moved C29 14.0 mm to (108.6, 94.0)
- moved D3 13.6 mm to (99.7, 87.6), turned to 0 degrees
- moved R11 12.8 mm to (108.6, 81.3)
- moved C24 9.85 mm to (99.5, 78.7), turned to 0 degrees
- moved D1 9.15 mm to (99.7, 91.4), turned to 180 degrees
- moved C28 9.00 mm to (108.6, 91.4)
- moved C34 6.50 mm to (108.6, 83.8)
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Routing:
- net +3V3: track 275.9 -> 238.2 mm
- net Net-(C33-Pad1): track 23.2 -> 5.68 mm
- net Net-(C31-Pad1): track 19.5 -> 5.55 mm
- net /SCLK: track 121.3 -> 110.8 mm
- net Net-(C25-Pad1): track 25.9 -> 15.6 mm
- net /MOSI: track 119.0 -> 109.0 mm
- net /Epaper/RESE: track 10.6 -> 20.2 mm
- net /Epaper/PREVGL: track 30.7 -> 22.1 mm
- net /DISPCS: track 74.8 -> 83.3 mm
- net /Epaper/GDR: track 10.7 -> 17.3 mm
- net Net-(C35-Pad1): track 15.4 -> 9.16 mm
- net Net-(C29-Pad1): track 15.8 -> 10.1 mm
- net /DISPBUSY: track 81.1 -> 76.3 mm
- net Net-(C34-Pad1): track 13.4 -> 11.1 mm
- net Net-(C25-Pad2): track 9.61 -> 11.4 mm
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
Commit message: feat(pcb): add 2 neopixels
Parts:
- added D6: WS2812B, LED_SMD:LED_WS2812B_PLCC4_5.0x5.0mm_P3.2mm, B.Cu at (70.5, 73.5)
- added D7: WS2812B, LED_SMD:LED_WS2812B_PLCC4_5.0x5.0mm_P3.2mm, B.Cu at (93.3, 73.4)
Connections:
- U3 pad 16: Net-(U3-Pad16) -> /NEOPIXEL
Routing:
- net /NEOPIXEL: track 0.00 -> 48.5 mm, vias 0 -> 1
- net Net-(D6-Pad2): track 0.00 -> 25.7 mm, vias 0 -> 2
- net +3V3: track 238.2 -> 257.0 mm, vias 0 -> 1

Commit message: cleanup(pcb): remove touch buttons / slider
Parts:
- removed U4: touch-slider-4pin, touch-buttons:TouchSlider-4_50x10mm
- removed U5, U6: touch-button, touch-buttons:TOUCH-CIRCLE
Connections:
- U3 pad 3: /TouchBTN2 -> Net-(U3-Pad3)
- U3 pad 4: /TouchBTN1 -> Net-(U3-Pad4)
Routing:
- net /TouchBTN2: track 73.5 -> 0.00 mm, vias 1 -> 0
- net Net-(U3-Pad10): track 51.0 -> 0.00 mm, vias 1 -> 0
- net Net-(U3-Pad9): track 49.2 -> 0.00 mm, vias 1 -> 0
- net Net-(U3-Pad7): track 36.6 -> 0.00 mm, vias 1 -> 0
- net Net-(U3-Pad8): track 34.7 -> 0.00 mm, vias 1 -> 0
- net /TouchBTN1: track 10.2 -> 0.00 mm, vias 1 -> 0

Commit message: feat(pcb): new board shape
Parts:
- moved ? 57.6 mm to (79.0, 129.4)
- moved svg2mod 16.4 mm to (78.6, 130.9)
Other:
- board size 80 x 57.1 mm -> 81.8 x 99.5 mm

Commit message: feat(pcb): create new footprint with board shape
based on Elad's design. The shape is automatically generated from
"board-shape.svg", along with the bottom silk screen and hints
where to place various components
Parts:
- removed ?: , logo:aram-logo
- added D8: WS2812B, LED_SMD:LED_WS2812B_PLCC4_5.0x5.0mm_P3.2mm, B.Cu at (107.0, 62.3)
- added D9: WS2812B, LED_SMD:LED_WS2812B_PLCC4_5.0x5.0mm_P3.2mm, B.Cu at (104.6, 54.2)
- added svg2mod: G***, logo:board-shape, F.Cu at (78.5, 92.5)
- moved J1 80.3 mm to (116.4, 118.6), turned to 90 degrees
- moved R3 69.6 mm to (106.3, 128.3), turned to 180 degrees
- moved R4 65.4 mm to (106.3, 125.7), turned to 180 degrees
- moved C21 64.0 mm to (100.5, 128.3), turned to 180 degrees
- moved R2 61.4 mm to (106.3, 123.2), turned to 180 degrees
- moved C22 59.4 mm to (100.5, 125.7), turned to 180 degrees
- moved C20 54.9 mm to (100.5, 123.2), turned to 180 degrees
- moved J4 48.9 mm to (76.5, 45.8), turned to 180 degrees
- moved D7 43.0 mm to (54.9, 54.1)
- moved R13 34.6 mm to (47.2, 113.3), turned to 180 degrees
- moved D6 21.3 mm to (52.5, 62.2)
Routing:
- net +3V3: track 257.0 -> 359.5 mm, vias 1 -> 0
- net /SheetMP3/RIGHT: track 69.7 -> 0.00 mm, vias 2 -> 0
- net Net-(D7-Pad2): track 0.00 -> 60.0 mm
- net /SheetMP3/GBUF: track 58.3 -> 0.00 mm, vias 2 -> 0
- net /SheetMP3/LEFT: track 48.9 -> 0.00 mm, vias 2 -> 0
- net GNDA: track 70.2 -> 38.0 mm
- net Net-(D5-Pad2): track 33.5 -> 2.44 mm
- net Net-(D6-Pad2): track 25.7 -> 3.90 mm, vias 2 -> 0
- net +5V: track 26.6 -> 7.02 mm
- net Net-(J4-Pad6): track 12.9 -> 0.00 mm
- net /D-: track 13.9 -> 3.87 mm
- net /D+: track 12.7 -> 4.49 mm
- net Net-(D8-Pad2): track 0.00 -> 6.84 mm
- net Net-(C22-Pad1): track 4.29 -> 0.00 mm
- net Net-(C21-Pad1): track 4.29 -> 0.00 mm
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Other:
- board size 81.8 x 99.5 mm -> 85 x 99.6 mm

Commit message: feat(pcb): Add 3 Cherry MX buttons
Parts:
- added SW1: SW_Push, Button_Switch_Keyboard:SW_Cherry_MX1A_1.00u_PCB, B.Cu at (54.7, 119.4)
- added SW2: SW_Push, Button_Switch_Keyboard:SW_Cherry_MX1A_1.00u_PCB, B.Cu at (77.3, 123.9)
- added SW3: SW_Push, Button_Switch_Keyboard:SW_Cherry_MX1A_1.00u_PCB, B.Cu at (99.7, 119.4)
- moved svg2mod 71.1 mm to (80.0, 59.8)
- moved C22 10.2 mm to (96.1, 134.9)
- moved R4 10.2 mm to (101.9, 134.9)
- moved C20 10.2 mm to (96.1, 132.4)
- moved C21 10.2 mm to (96.1, 137.4)
- moved R2 10.2 mm to (101.9, 132.4)
- moved R3 10.2 mm to (101.9, 137.4)
- moved C3 1.61 mm to (98.5, 116.4)
Routing:
- net GND: track 99.5 -> 88.6 mm

Commit message: feat(pcb): add standard ARM-JTAG connector
Parts:
- J6: value Conn_01x04_Male -> Conn_ARM_JTAG_SWD_10; footprint Connector_PinHeader_2.54mm:PinHeader_1x04_P2.54mm_Vertical -> Connector_PinHeader_1.27mm:PinHeader_2x05_P1.27mm_Vertical_SMD; moved to B.Cu
- moved J6 25.8 mm to (79.9, 66.8), turned to 90 degrees
Connections:
- J6 pad 3: /SWDCLK -> GND
- J6 pad 4: GND -> /SWDCLK
Routing:
- net /SWDCLK: track 15.8 -> 53.8 mm
- net /SWDIO: track 16.5 -> 52.1 mm
- net +5V: track 7.02 -> 19.4 mm
- net GND: track 88.6 -> 91.8 mm
- net Net-(D7-Pad2): track 60.0 -> 62.3 mm

Commit message: feat(pcb): reposition audio jack, display connector
Parts:
- moved C11 25.4 mm to (72.9, 114.3), turned to 90 degrees
- moved U1 24.4 mm to (81.7, 116.8)
- moved C3 23.4 mm to (75.2, 118.4), turned to 90 degrees
- moved C5 23.2 mm to (75.2, 114.3), turned to 90 degrees
- moved C21 23.1 mm to (100.6, 114.8)
- moved R3 22.8 mm to (104.4, 114.8)
- moved C22 22.6 mm to (100.6, 112.8)
- moved R4 22.3 mm to (104.4, 112.8)
- moved C20 22.1 mm to (100.6, 110.7)
- moved R2 21.8 mm to (104.4, 110.7)
- moved J1 11.6 mm to (114.0, 107.3), turned to 180 degrees
- moved C26 9.33 mm to (108.0, 101.0), turned to 180 degrees
- moved C31 5.75 mm to (107.8, 93.3)
- moved R11 5.75 mm to (107.9, 75.6)
- moved C27 5.75 mm to (108.0, 83.2)
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Routing:
- net /D-: track 3.87 -> 81.2 mm, vias 0 -> 2
- net /D+: track 4.49 -> 77.8 mm, vias 0 -> 2
- net Net-(SW3-Pad1): track 0.00 -> 59.5 mm, vias 0 -> 1
- net +5V: track 19.4 -> 75.4 mm, vias 0 -> 2
- net Net-(SW2-Pad1): track 0.00 -> 36.6 mm, vias 0 -> 1
- net /SheetMP3/GBUF: track 0.00 -> 36.6 mm, vias 0 -> 2
- net /SheetMP3/LEFT: track 0.00 -> 33.0 mm, vias 0 -> 2
- net +3V3: track 359.5 -> 326.5 mm, vias 0 -> 5
- net /SheetMP3/RIGHT: track 0.00 -> 31.0 mm, vias 0 -> 2
- net Net-(SW1-Pad1): track 0.00 -> 23.7 mm, vias 0 -> 1
- net GNDA: track 38.0 -> 53.9 mm, vias 0 -> 2
- net Net-(J4-Pad6): track 0.00 -> 12.9 mm
- net /MOSI: track 109.0 -> 120.6 mm
- net /SCLK: track 110.8 -> 118.9 mm, vias 3 -> 2
- net /Epaper/PREVGL: track 22.1 -> 15.5 mm
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Other:
- board text removed: "CLK"
- board text removed: "IO"
- board text removed: "SWD"
