File: pcb/badge/badge.kicad_pcb (KiCad board)
At the start: 2 copper layers, 85 x 99.6 mm, 76 parts, among them IC1 VS1053B, J1 AudioJack4, J2 SAO_CONN, J4 USB_B_Micro, J6 Conn_ARM_JTAG_SWD_10, J7 PFC24/0.5mm, Q1 Si1308EDL, SW1 SW_Push, SW2 SW_Push, SW3 SW_Push, U1 AMS1117-1.8, U2 AMS1117-3.3, U3 E73-2G4M08S1C, U4 TPS610986DSET, Y1 12.288M

Commit message: fix(pcb): move BLE module to edge of board
we need to reroute everything again :q
Parts:
- moved U4 23.1 mm to (76.8, 78.1)
- moved U3 8.82 mm to (43.2, 95.9)
- moved R13 3.14 mm to (49.5, 111.1), turned to 0 degrees
- moved D5 2.09 mm to (45.2, 111.1)
Routing:
- net /DISPCS: track 82.8 -> 0.00 mm, vias 2 -> 0
- net /D-: track 81.2 -> 1.31 mm, vias 2 -> 0
- net /DISPDC: track 78.2 -> 0.00 mm, vias 2 -> 0
- net /DISPRST: track 77.7 -> 1.01 mm, vias 2 -> 0
- net /DISPBUSY: track 74.1 -> 0.24 mm, vias 2 -> 0
- net /D+: track 78.2 -> 4.57 mm, vias 2 -> 1
- net Net-(SW3-Pad1): track 59.5 -> 0.00 mm, vias 1 -> 0
- net /SWDCLK: track 54.0 -> 1.51 mm
- net /SWDIO: track 52.3 -> 0.00 mm
- net /SNDDREQ: track 56.4 -> 4.32 mm, vias 2 -> 1
- net /NEOPIXEL: track 45.8 -> 0.00 mm, vias 1 -> 0
- net /MOSI: track 103.5 -> 58.0 mm, vias 3 -> 2
- net /MISO: track 43.2 -> 0.00 mm, vias 2 -> 0
- net /SNDxDCS: track 57.8 -> 23.0 mm, vias 4 -> 2
- net /SNDRESET: track 31.3 -> 0.00 mm, vias 2 -> 0
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
Commit message: PCB routing
Parts:
- added BZ1: Buzzer, Connector_PinHeader_2.00mm:PinHeader_1x02_P2.00mm_Vertical, F.Cu at (46.6, 69.2)
- added C36: 1uF, Capacitor_SMD:C_0603_1608Metric, F.Cu at (82.4, 83.3)
- added C37: 100nF, Capacitor_SMD:C_0603_1608Metric, F.Cu at (73.7, 83.2)
- added L2: 4.7uH, Inductor_SMD:L_1210_3225Metric, F.Cu at (85.5, 78.7)
- added Q2: Si1308EDL, Package_TO_SOT_SMD:SOT-323_SC-70, F.Cu at (45.3, 76.7)
- added R14: 400R, Resistor_SMD:R_0603_1608Metric, F.Cu at (78.3, 83.2)
- added SW4: SW_SPDT, Button_Switch_THT:SW_CuK_OS102011MA1QN1_SPDT_Angled, F.Cu at (39.5, 110.2)
- added U5: GD25Q16C, Package_SO:SOIC-8_3.9x4.9mm_P1.27mm, F.Cu at (44.3, 82.3)
- moved C12 36.5 mm to (91.7, 82.2)
- moved C4 15.3 mm to (66.9, 86.7)
- moved C6 12.8 mm to (70.5, 79.9)
- moved U3 0.89 mm to (43.2, 95.0)
- renumbered svg2mod to SHAPE
Connections:
- BT1 pad 2: Net-(BT1-Pad2) -> GND
- C16 pad 1: +3V3 -> /V_BAT
- C6 pad 1: +3V3 -> GND
- C6 pad 2: GND -> +3V3
- U2 pad 2: +3V3 -> Net-(C36-Pad2)
- U3 pad 10: Net-(U3-Pad10) -> /V_BAT
- U3 pad 28: (no net) -> Net-(U3-Pad28)
- U3 pad 30: (no net) -> /VIBRATOR
- U3 pad 32: (no net) -> /FLASH_SO
- U3 pad 34: (no net) -> Net-(U3-Pad34)
- U3 pad 36: (no net) -> Net-(U3-Pad36)
- U3 pad 38: (no net) -> Net-(U3-Pad38)
- U3 pad 40: (no net) -> Net-(U3-Pad40)
- U3 pad 42: (no net) -> Net-(U3-Pad42)
- U4 pad 1: Net-(U4-Pad1) -> +3V3
- U4 pad 4: Net-(U4-Pad4) -> +3V3
- U4 pad 6: Net-(U4-Pad6) -> GND
Routing:
- net /V_BAT: track 0.00 -> 103.7 mm, vias 0 -> 1
- net Net-(BT1-Pad1): track 0.00 -> 99.8 mm, vias 0 -> 1
- net Net-(C36-Pad2): track 0.00 -> 89.2 mm, vias 0 -> 5
- net /DISPRST: track 1.01 -> 82.0 mm, vias 0 -> 2
- net /SDA: track 0.00 -> 77.5 mm, vias 0 -> 4
- net /SCL: track 0.00 -> 76.0 mm, vias 0 -> 2
- net /DISPBUSY: track 0.24 -> 71.6 mm, vias 0 -> 2
- net +3V3: track 330.8 -> 400.4 mm
- net /SWDCLK: track 1.51 -> 70.7 mm, vias 1 -> 3
- net Net-(SW3-Pad1): track 0.00 -> 64.6 mm, vias 0 -> 1
- net /MOSI: track 58.0 -> 120.9 mm, vias 2 -> 3
- net /SWDIO: track 0.00 -> 59.1 mm, vias 1 -> 4
- net /D-: track 1.31 -> 58.5 mm
- net /SNDDREQ: track 4.32 -> 60.7 mm, vias 1 -> 2
- net /D+: track 4.57 -> 57.0 mm
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Other:
- rule trace_min: 0.2 -> 0.15
- board text added: "+"

Commit message: feat(pcb): complete layout
Parts:
- moved Q1 8.75 mm to (114.5, 75.6)
- moved R10 6.46 mm to (114.2, 72.6)
- turned C37 to 180 degrees
- turned Q2 to 90 degrees
Routing:
- net /DISPCS: track 0.00 -> 76.8 mm, vias 0 -> 2
- net /DISPDC: track 1.19 -> 74.8 mm, vias 0 -> 2
- net /SNDxDCS: track 0.00 -> 69.8 mm, vias 0 -> 2
- net GND: track 66.4 -> 120.3 mm, vias 14 -> 23
- net /SNDDREQ: track 60.7 -> 72.5 mm
- net /MOSI: track 120.9 -> 112.2 mm
- net /DISPRST: track 82.0 -> 74.7 mm
- net /SWDCLK: track 70.7 -> 76.8 mm, vias 3 -> 4
- net Net-(C25-Pad1): track 17.7 -> 22.4 mm
- net /VIBRATOR: track 21.5 -> 18.2 mm
- net /SNDCS: track 61.5 -> 58.5 mm
- net Net-(L2-Pad2): track 25.5 -> 23.2 mm
- net +3V3: track 400.4 -> 398.1 mm
- net GNDA: track 56.9 -> 54.8 mm
- net /Epaper/GDR: track 18.5 -> 16.5 mm
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
Commit message: feat(pcb): add texts to switch, indicate SAO VCC pin
Other:
- board text added: "BAT"
- board text added: "Power"
- board text added: "USB"
Changed lines of the file:
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@@
   (general
     (thickness 1.6)
-    (drawings 3)
+    (drawings 7)
     (tracks 1122)
     (zones 0)
@@
     (34 B.Paste user)
     (35 F.Paste user)
-    (36 B.SilkS user hide)
+    (36 B.SilkS user)
     (37 F.SilkS user)
     (38 B.Mask user)
     (39 F.Mask user)
-    (40 Dwgs.User user hide)
+    (40 Dwgs.User user)
     (41 Cmts.User user)
     (42 Eco1.User user)
@@
     )
   )
+  (gr_text Power (at 43.688 112.268 270) (layer B.SilkS)
+    (effects (font (size 1.5 1.5) (thickness 0.3)) (justify mirror))
+  )
+  (gr_text BAT (at 42.164 105.156) (layer B.SilkS)
+    (effects (font (size 1.5 1.5) (thickness 0.3)) (justify mirror))
+  )
+  (gr_text USB (at 41.656 119.888) (layer B.SilkS)
+    (effects (font (size 1.5 1.5) (thickness 0.3)) (justify mirror))
+  )
+  (gr_circle (center 84.31784 57.25668) (end 84.66784 57.25668) (layer F.SilkS) (width 0.5))
   (gr_text + (at 48.26 68.961) (layer F.SilkS)
     (effects (font (size 1 1) (thickness 0.2)))

Commit message: fix(pcb): change step-up resistor to 390R
400R is not a common value, 390 is.
Parts:
- R14: value 400R -> 390R
Changed lines of the file:
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@@
       (effects (font (size 1 1) (thickness 0.15)))
     )
-    (fp_text value 400R (at 0 1.43) (layer F.Fab)
+    (fp_text value 390R (at 0 1.43) (layer F.Fab)
       (effects (font (size 1 1) (thickness 0.15)))
     )

Commit message: feat(pcb): add battery reverse polarity protection
Parts:
- added U6: PMPB15XP,115, PMPB15XP_115:MOSFET_PMPB55ENEAX, F.Cu at (94.0, 74.9)
Connections:
- SW4 pad 1: Net-(BT1-Pad1) -> Net-(SW4-Pad1)
Routing:
- net Net-(SW4-Pad1): track 0.00 -> 82.7 mm, vias 0 -> 1
- net Net-(BT1-Pad1): track 99.8 -> 26.0 mm, vias 1 -> 0
- net GND: track 120.3 -> 120.9 mm

Commit message: feat(pcb): add LIS2DH12TR accelerometer
Parts:
- added C38: 10uF, Capacitor_SMD:C_0603_1608Metric, F.Cu at (96.5, 54.0)
- added C39: 100nF, Capacitor_SMD:C_0603_1608Metric, F.Cu at (96.5, 52.1)
- added U7: LIS2DH12TR, Package_LGA:LGA-12_2x2mm_P0.5mm, F.Cu at (92.0, 53.3)
Routing:
- net +3V3: track 398.1 -> 416.1 mm
- net /SCL: track 77.3 -> 88.4 mm
- net /SDA: track 79.3 -> 86.1 mm
- net GND: track 120.9 -> 125.8 mm
