File: pcb/badge/MP3.sch (KiCad schematic (older format))
At the start: 39 parts

Commit message: Fix names in MP3 sheet
Add programming connector
Parts:
- removed C? (x2): 33pF, Capacitor_SMD:C_0603_1608Metric, symbol Device:C
- removed C? (x2): 10nF, Capacitor_SMD:C_0603_1608Metric, symbol Device:C
- removed C?: 47nF, Capacitor_SMD:C_0603_1608Metric, symbol Device:C
- removed C?: 1uF, Capacitor_SMD:C_0603_1608Metric, symbol Device:C
- removed C? (x14): 100nF, Capacitor_SMD:C_0603_1608Metric, symbol Device:C
- removed C? (x2): 10uF, Capacitor_SMD:C_0603_1608Metric, symbol Device:CP1
- removed C?: 100uF, Capacitor_Tantalum_SMD:CP_EIA-3216-18_Kemet-A, symbol Device:CP1
- removed IC?: VS1053B, Package_QFP:LQFP-48_7x7mm_P0.5mm, symbol COM-08892:COM-08892
- removed J?: AudioJack4_Ground, audio:Jack_3.5mm_PJ320D_Horizontal, symbol Connector:AudioJack4_Ground
- removed J?: Conn_01x08_Male, Connector_PinHeader_2.54mm:PinHeader_1x08_P2.54mm_Vertical, symbol Connector:Conn_01x08_Male
- removed J?: Conn_01x04_Male, Connector_PinSocket_2.54mm:PinSocket_1x04_P2.54mm_Vertical, symbol Connector:Conn_01x04_Male
- removed R?: 1M, Resistor_SMD:R_0603_1608Metric, symbol Device:R
- removed R? (x4): 100k, Resistor_SMD:R_0603_1608Metric, symbol Device:R
- removed R? (x3): 20R, Resistor_SMD:R_0603_1608Metric, symbol Device:R
- removed R?: 0, Jumper:SolderJumper-2_P1.3mm_Bridged2Bar_RoundedPad1.0x1.5mm, symbol Device:R
- removed U?: AMS1117-1.8, Package_TO_SOT_SMD:SOT-223-3_TabPin2, symbol Regulator_Linear:AMS1117-1.8
- removed U?: AMS1117-3.3, Package_TO_SOT_SMD:SOT-223-3_TabPin2, symbol Regulator_Linear:AMS1117-3.3
- removed Y?: 12.288M, Crystal:Crystal_SMD_3225-4Pin_3.2x2.5mm, symbol Device:Crystal
- added C1, C2: 33pF, Capacitor_SMD:C_0603_1608Metric, symbol Device:C
- added C10, C13, C14, C15, C17, C18, C19, C3, C4, C5, C6, C7, C8, C9: 100nF, Capacitor_SMD:C_0603_1608Metric, symbol Device:C
- added C11, C16: 10uF, Capacitor_SMD:C_0603_1608Metric, symbol Device:CP1
- added C12: 100uF, Capacitor_Tantalum_SMD:CP_EIA-3216-18_Kemet-A, symbol Device:CP1
- added C20, C21: 10nF, Capacitor_SMD:C_0603_1608Metric, symbol Device:C
- added C22: 47nF, Capacitor_SMD:C_0603_1608Metric, symbol Device:C
- added C23: 1uF, Capacitor_SMD:C_0603_1608Metric, symbol Device:C
- added IC1: VS1053B, Package_QFP:LQFP-48_7x7mm_P0.5mm, symbol COM-08892:COM-08892
- added J1: AudioJack4_Ground, audio:Jack_3.5mm_PJ320D_Horizontal, symbol Connector:AudioJack4_Ground
- added J2: Conn_01x04_Male, Connector_PinSocket_2.54mm:PinSocket_1x04_P2.54mm_Vertical, symbol Connector:Conn_01x04_Male
- added J3: Conn_01x08_Male, Connector_PinHeader_2.54mm:PinHeader_1x08_P2.54mm_Vertical, symbol Connector:Conn_01x08_Male
- added R1: 1M, Resistor_SMD:R_0603_1608Metric, symbol Device:R
- added R2, R3, R4: 20R, Resistor_SMD:R_0603_1608Metric, symbol Device:R
- added R5, R6, R8, R9: 100k, Resistor_SMD:R_0603_1608Metric, symbol Device:R
- added R7: 0, Jumper:SolderJumper-2_P1.3mm_Bridged2Bar_RoundedPad1.0x1.5mm, symbol Device:R
- added U1: AMS1117-1.8, Package_TO_SOT_SMD:SOT-223-3_TabPin2, symbol Regulator_Linear:AMS1117-1.8
- added U2: AMS1117-3.3, Package_TO_SOT_SMD:SOT-223-3_TabPin2, symbol Regulator_Linear:AMS1117-3.3
- added Y1: 12.288M, Crystal:Crystal_SMD_3225-4Pin_3.2x2.5mm, symbol Device:Crystal

Commit message: Fix ERC problems
Connections:
- no-connect marks 0 -> 7
Changed lines of the file:
@@
 Text HLabel 6500 7250 2    50   Input ~ 0
 xCS
+NoConn ~ 6150 1200
+NoConn ~ 6650 1400
+NoConn ~ 8350 1800
+NoConn ~ 10150 3400
+NoConn ~ 8550 4600
+NoConn ~ 7750 2600
+NoConn ~ 7750 2500
 $EndSCHEMATC

Commit message: Routing the CPU
Parts:
- removed J1: AudioJack4_Ground, audio:Jack_3.5mm_PJ320D_Horizontal, symbol Connector:AudioJack4_Ground
- removed J2: Conn_01x04_Male, Connector_PinSocket_2.54mm:PinSocket_1x04_P2.54mm_Vertical, symbol Connector:Conn_01x04_Male
- added J1: AudioJack4, audio:Jack_3.5mm_PJ320D_Horizontal, symbol Connector:AudioJack4
Connections:
- wire segments 157 -> 153
- no-connect marks 7 -> 6
Changed lines of the file:
@@
 	8800 5750 8500 5750
 Connection ~ 8800 5750
-$Comp
-L Connector:AudioJack4_Ground J1
-U 1 1 5BF87719
-P 6550 1200
-F 0 "J1" V 6470 1405 50  0000 L CNN
-F 1 "AudioJack4_Ground" V 6561 1405 50  0000 L CNN
-F 2 "audio:Jack_3.5mm_PJ320D_Horizontal" H 6550 1200 50  0001 C CNN
-F 3 "~" H 6550 1200 50  0001 C CNN
-	1    6550 1200
-	0    1    1    0
-$EndComp
 Text Label 6350 1700 1    50   ~ 0
 LEFT
@@
 	3250 6650 3800 6650
 $Comp
-L Connector:Conn_01x04_Male J2
-U 1 1 5C241429
-P 1200 1600
-F 0 "J2" H 1306 1878 50  0000 C CNN
-F 1 "Conn_01x04_Male" H 1306 1787 50  0000 C CNN
-F 2 "Connector_PinSocket_2.54mm:PinSocket_1x04_P2.54mm_Vertical" H 1200 1600 50  0001 C CNN
-F 3 "~" H 1200 1600 50  0001 C CNN
-	1    1200 1600
-	1    0    0    -1
-$EndComp
-$Comp
-L power:GND #PWR0137
-U 1 1 5C241497
-P 1600 1800
-F 0 "#PWR0137" H 1600 1550 50  0001 C CNN
-F 1 "GND" V 1605 1672 50  0000 R CNN
-F 2 "" H 1600 1800 50  0001 C CNN
-F 3 "" H 1600 1800 50  0001 C CNN
-	1    1600 1800
-	0    -1   -1   0
-$EndComp
-$Comp
-L power:GND #PWR0138
-U 1 1 5C241556
-P 1600 1500
-F 0 "#PWR0138" H 1600 1250 50  0001 C CNN
-F 1 "GND" V 1605 1372 50  0000 R CNN
-F 2 "" H 1600 1500 50  0001 C CNN
-F 3 "" H 1600 1500 50  0001 C CNN
-	1    1600 1500
-	0    -1   -1   0
-$EndComp
-$Comp
-L power:+3V3 #PWR0139
-U 1 1 5C2415A9
-P 1600 1600
-F 0 "#PWR0139" H 1600 1450 50  0001 C CNN
-F 1 "+3V3" V 1615 1728 50  0000 L CNN
-F 2 "" H 1600 1600 50  0001 C CNN
-F 3 "" H 1600 1600 50  0001 C CNN
-	1    1600 1600
-	0    1    1    0
-$EndComp
-$Comp
-L power:+5V #PWR0140
-U 1 1 5C241BBA
-P 1600 1700
-F 0 "#PWR0140" H 1600 1550 50  0001 C CNN
-F 1 "+5V" V 1615 1828 50  0000 L CNN
-F 2 "" H 1600 1700 50  0001 C CNN
-F 3 "" H 1600 1700 50  0001 C CNN
-	1    1600 1700
-	0    1    1    0
-$EndComp
-Wire Wire Line
-	1400 1500 1600 1500
-Wire Wire Line
-	1600 1600 1400 1600
-Wire Wire Line
-	1400 1700 1600 1700
-Wire Wire Line
-	1400 1800 1600 1800
-$Comp
 L Device:R R7
 U 1 1 5C26550C
@@
 Text HLabel 6500 7250 2    50   Input ~ 0
 xCS
-NoConn ~ 6150 1200
 NoConn ~ 6650 1400
 NoConn ~ 8350 1800
@@
 NoConn ~ 7750 2600
 NoConn ~ 7750 2500
+$Comp
+L Connector:AudioJack4 J1
+U 1 1 5C2EE96B
+P 6550 1200
+F 0 "J1" V 6459 1388 50  0000 L CNN
+F 1 "AudioJack4" V 6550 1388 50  0000 L CNN
+F 2 "audio:Jack_3.5mm_PJ320D_Horizontal" H 6550 1200 50  0001 C CNN
+F 3 "~" H 6550 1200 50  0001 C CNN
+	1    6550 1200
+	0    1    1    0
+$EndComp
 $EndSCHEMATC

Commit message: Fix reversed connector for EPD
Parts:
- J1: footprint audio:Jack_3.5mm_PJ320D_Horizontal -> connectors:Jack_3.5mm_PJ320D_Horizontal
Changed lines of the file:
@@
 F 0 "J1" V 6459 1388 50  0000 L CNN
 F 1 "AudioJack4" V 6550 1388 50  0000 L CNN
-F 2 "audio:Jack_3.5mm_PJ320D_Horizontal" H 6550 1200 50  0001 C CNN
+F 2 "connectors:Jack_3.5mm_PJ320D_Horizontal" H 6550 1200 50  0001 C CNN
 F 3 "~" H 6550 1200 50  0001 C CNN
 	1    6550 1200

Commit message: cleanup(PCB): remove display/sound headers from schematic
Parts:
- removed J3: Conn_01x08_Male, Connector_PinHeader_2.54mm:PinHeader_1x08_P2.54mm_Vertical, symbol Connector:Conn_01x08_Male
Connections:
- wire segments 153 -> 145
Changed lines of the file:
@@
 F 3 "" H 9450 4800 50  0001 C CNN
 	1    9450 4800
-	-1   0    0    1
+	0    1    1    0
 $EndComp
 Wire Wire Line
@@
 Text Label 6550 1700 1    50   ~ 0
 GBUF
-$Comp
-L Connector:Conn_01x08_Male J3
-U 1 1 5C0E7589
-P 5800 6850
-F 0 "J3" H 5906 7328 50  0000 C CNN
-F 1 "Conn_01x08_Male" H 5906 7237 50  0000 C CNN
-F 2 "Connector_PinHeader_2.54mm:PinHeader_1x08_P2.54mm_Vertical" H 5800 6850 50  0001 C CNN
-F 3 "~" H 5800 6850 50  0001 C CNN
-	1    5800 6850
-	1    0    0    -1
-$EndComp
-$Comp
-L power:GND #PWR0146
-U 1 1 5C0E8288
-P 6400 6550
-F 0 "#PWR0146" H 6400 6300 50  0001 C CNN
-F 1 "GND" V 6405 6422 50  0000 R CNN
-F 2 "" H 6400 6550 50  0001 C CNN
-F 3 "" H 6400 6550 50  0001 C CNN
-	1    6400 6550
-	0    -1   -1   0
-$EndComp
-Wire Wire Line
-	6000 6550 6400 6550
-Wire Wire Line
-	6000 6650 6450 6650
-Wire Wire Line
-	6000 6750 6450 6750
-Wire Wire Line
-	6000 6850 6400 6850
-Wire Wire Line
-	6000 7050 6500 7050
-Wire Wire Line
-	6000 7150 6500 7150
-Wire Wire Line
-	6000 7250 6500 7250
-Wire Wire Line
-	6000 6950 6450 6950
-Text Label 6150 6650 0    50   ~ 0
-MOSI
-Text Label 6050 6750 0    50   ~ 0
-MISO
-Text Label 6100 6850 0    50   ~ 0
-SCLK
-Text Label 6100 6950 0    50   ~ 0
-XRESET
-Text Label 6050 7050 0    50   ~ 0
-DREQ
-Text Label 6100 7150 0    50   ~ 0
-xDCS
-Text Label 6150 7250 0    50   ~ 0
-xCS
-Wire Wire Line
-	7750 2700 7300 2700
-Text Label 7350 2700 0    50   ~ 0
-XRESET
+Wire Wire Line
+	7750 2700 7450 2700
 Wire Wire Line
 	10150 3100 10500 3100
-Text Label 10200 3100 0    50   ~ 0
-MISO
-Wire Wire Line
-	10150 3200 10550 3200
-Text Label 10350 3200 0    50   ~ 0
-MOSI
-Text Label 10350 3300 0    50   ~ 0
-SCLK
-Wire Wire Line
-	10150 3300 10600 3300
-Wire Wire Line
-	7750 3200 7350 3200
-Text Label 7500 3200 0    50   ~ 0
-DREQ
+Wire Wire Line
+	10150 3200 10500 3200
+Wire Wire Line
+	10150 3300 10500 3300
+Wire Wire Line
+	7750 3200 7450 3200
 Wire Wire Line
 	8350 4600 8350 4800
-Text Label 8350 4750 1    50   ~ 0
-xDCS
-Wire Wire Line
-	9350 4600 9350 4900
-Text Label 9350 4750 1    50   ~ 0
-xCS
+Wire Wire Line
+	9350 4600 9350 4850
 $Comp
 L power:GND #PWR0147
@@
 Wire Wire Line
 	10900 2550 10800 2550
-Text HLabel 6450 6650 2    50   Input ~ 0
+Text HLabel 10500 3200 2    50   Input ~ 0
 MOSI
-Text HLabel 6450 6750 2    50   Output ~ 0
+Text HLabel 10500 3100 2    50   Output ~ 0
 MISO
-Text HLabel 6400 6850 2    50   Input ~ 0
+Text HLabel 10500 3300 2    50   Input ~ 0
 SCLK
-Text HLabel 6450 6950 2    50   Input ~ 0
+Text HLabel 7450 2700 0    50   Input ~ 0
 XRESET
-Text HLabel 6500 7050 2    50   Output ~ 0
+Text HLabel 7450 3200 0    50   Output ~ 0
 DREQ
-Text HLabel 6500 7150 2    50   Input ~ 0
+Text HLabel 8350 4800 0    50   Input ~ 0
 xDCS
-Text HLabel 6500 7250 2    50   Input ~ 0
+Text HLabel 9350 4850 3    50   Input ~ 0
 xCS
 NoConn ~ 6650 1400

Commit message: Add Flash memory + connect battery and step-up IC
Parts:
- removed C12: 100uF, Capacitor_Tantalum_SMD:CP_EIA-3216-18_Kemet-A, symbol Device:CP1
- removed C16: 10uF, Capacitor_SMD:C_0603_1608Metric, symbol Device:CP1
- removed C4, C6: 100nF, Capacitor_SMD:C_0603_1608Metric, symbol Device:C
- removed U2: AMS1117-3.3, Package_TO_SOT_SMD:SOT-223-3_TabPin2, symbol Regulator_Linear:AMS1117-3.3
Changed lines of the file:
@@
 Connection ~ 2700 5250
-$Comp
-L Regulator_Linear:AMS1117-3.3 U2
-U 1 1 5C21D4A4
-P 2150 6350
-F 0 "U2" H 2150 6592 50  0000 C CNN
-F 1 "AMS1117-3.3" H 2150 6501 50  0000 C CNN
-F 2 "Package_TO_SOT_SMD:SOT-223-3_TabPin2" H 2150 6550 50  0001 C CNN
-F 3 "http://www.advanced-monolithic.com/pdf/ds1117.pdf" H 2250 6100 50  0001 C CNN
-	1    2150 6350
-	1    0    0    -1
-$EndComp
-Wire Wire Line
-	2450 6350 2750 6350
-Wire Wire Line
-	2150 6650 2150 6850
-Wire Wire Line
-	1850 6350 1500 6350
-$Comp
-L power:GND #PWR0134
-U 1 1 5C22386B
-P 2150 6850
-F 0 "#PWR0134" H 2150 6600 50  0001 C CNN
-F 1 "GND" H 2155 6677 50  0000 C CNN
-F 2 "" H 2150 6850 50  0001 C CNN
-F 3 "" H 2150 6850 50  0001 C CNN
-	1    2150 6850
-	1    0    0    -1
-$EndComp
-$Comp
-L power:+3V3 #PWR0135
-U 1 1 5C223877
-P 3950 6350
-F 0 "#PWR0135" H 3950 6200 50  0001 C CNN
-F 1 "+3V3" V 3965 6478 50  0000 L CNN
-F 2 "" H 3950 6350 50  0001 C CNN
-F 3 "" H 3950 6350 50  0001 C CNN
-	1    3950 6350
-	1    0    0    -1
-$EndComp
-$Comp
-L Device:C C4
-U 1 1 5C22387D
-P 1500 6500
-F 0 "C4" H 1615 6546 50  0000 L CNN
-F 1 "100nF" H 1615 6455 50  0000 L CNN
-F 2 "Capacitor_SMD:C_0603_1608Metric" H 1538 6350 50  0001 C CNN
-F 3 "~" H 1500 6500 50  0001 C CNN
-	1    1500 6500
-	1    0    0    -1
-$EndComp
-Connection ~ 1500 6350
-Wire Wire Line
-	1500 6350 1350 6350
-$Comp
-L Device:C C6
-U 1 1 5C223885
-P 2750 6500
-F 0 "C6" H 2865 6546 50  0000 L CNN
-F 1 "100nF" H 2865 6455 50  0000 L CNN
-F 2 "Capacitor_SMD:C_0603_1608Metric" H 2788 6350 50  0001 C CNN
-F 3 "~" H 2750 6500 50  0001 C CNN
-	1    2750 6500
-	1    0    0    -1
-$EndComp
-$Comp
-L Device:CP1 C16
-U 1 1 5C22388D
-P 3800 6500
-F 0 "C16" H 3915 6546 50  0000 L CNN
-F 1 "10uF" H 3915 6455 50  0000 L CNN
-F 2 "Capacitor_SMD:C_0603_1608Metric" H 3800 6500 50  0001 C CNN
-F 3 "~" H 3800 6500 50  0001 C CNN
-	1    3800 6500
-	1    0    0    -1
-$EndComp
-Connection ~ 3800 6350
-Wire Wire Line
-	3800 6350 3950 6350
-Wire Wire Line
-	1500 6650 2150 6650
-Connection ~ 2150 6650
-Wire Wire Line
-	2150 6650 2750 6650
-$Comp
-L power:+5V #PWR0136
-U 1 1 5C22B0EC
-P 1350 6350
-F 0 "#PWR0136" H 1350 6200 50  0001 C CNN
-F 1 "+5V" H 1365 6523 50  0000 C CNN
-F 2 "" H 1350 6350 50  0001 C CNN
-F 3 "" H 1350 6350 50  0001 C CNN
-	1    1350 6350
-	1    0    0    -1
-$EndComp
-Wire Wire Line
-	2750 6350 3250 6350
-Connection ~ 2750 6350
-Wire Wire Line
-	2750 6650 3250 6650
-Connection ~ 2750 6650
-$Comp
-L Device:CP1 C12
-U 1 1 5C240494
-P 3250 6500
-F 0 "C12" H 3365 6546 50  0000 L CNN
-F 1 "100uF" H 3365 6455 50  0000 L CNN
-F 2 "Capacitor_Tantalum_SMD:CP_EIA-3216-18_Kemet-A" H 3250 6500 50  0001 C CNN
-F 3 "~" H 3250 6500 50  0001 C CNN
-	1    3250 6500
-	1    0    0    -1
-$EndComp
-Connection ~ 3250 6350
-Wire Wire Line
-	3250 6350 3800 6350
-Connection ~ 3250 6650
-Wire Wire Line
-	3250 6650 3800 6650
 $Comp
 L Device:R R7
