File: pcb/badge/power.sch (KiCad schematic (older format))
At the start: 12 parts, among them SW4 SW_SPDT, U2 AMS1117-3.3, U4 TPS610986DSET

Commit message: feat(pcb): add battery reverse polarity protection
Parts:
- added U6: PMPB15XP,115, PMPB15XP_115:MOSFET_PMPB55ENEAX, symbol PMPB15XP_115:PMPB15XP,115
Connections:
- net GND: now also U6.3 (GATE)
- net at BT1.1 (+): now also U6.1 (DRAIN-1), U6.2 (DRAIN), U6.5 (DRAIN-3), U6.6 (DRAIN-2), U6.7 (DRAIN-4); no longer SW4.1 (A)
- new net: SW4.1 (A), U6.4 (SOURCE), U6.8 (SOURCE-1)
Other:
- moved on the sheet: BT1
Changed lines of the file:
@@
 L Device:Battery_Cell BT1
 U 1 1 5C4AE687
-P 4750 4350
-F 0 "BT1" H 4868 4446 50  0000 L CNN
-F 1 "Battery_Cell" H 4868 4355 50  0000 L CNN
-F 2 "AA_battery_clip:BK-53_MPD_AAClip" V 4750 4410 50  0001 C CNN
-F 3 "~" V 4750 4410 50  0001 C CNN
-	1    4750 4350
+P 3650 4850
+F 0 "BT1" H 3768 4946 50  0000 L CNN
+F 1 "Battery_Cell" H 3768 4855 50  0000 L CNN
+F 2 "AA_battery_clip:BK-53_MPD_AAClip" V 3650 4910 50  0001 C CNN
+F 3 "~" V 3650 4910 50  0001 C CNN
+	1    3650 4850
 	0    1    1    0
 $EndComp
@@
 L power:GND #PWR0168
 U 1 1 5C4AE6F4
-P 4650 4350
-F 0 "#PWR0168" H 4650 4100 50  0001 C CNN
-F 1 "GND" V 4655 4222 50  0000 R CNN
-F 2 "" H 4650 4350 50  0001 C CNN
-F 3 "" H 4650 4350 50  0001 C CNN
-	1    4650 4350
+P 3550 4850
+F 0 "#PWR0168" H 3550 4600 50  0001 C CNN
+F 1 "GND" V 3555 4722 50  0000 R CNN
+F 2 "" H 3550 4850 50  0001 C CNN
+F 3 "" H 3550 4850 50  0001 C CNN
+	1    3550 4850
 	0    1    1    0
 $EndComp
@@
 Connection ~ 6750 3100
 Wire Wire Line
-	5250 3700 5250 4350
+	5250 3700 5250 4250
 Wire Wire Line
 	4850 3500 5150 3500
-Wire Wire Line
-	4950 4350 5250 4350
 Wire Wire Line
 	5150 3500 5150 3350
@@
 Wire Wire Line
 	6100 3600 6300 3600
+$Comp
+L PMPB15XP_115:PMPB15XP,115 U6
+U 1 1 5C4C77B2
+P 5350 5050
+F 0 "U6" H 4700 5600 50  0000 L CNN
+F 1 "PMPB15XP,115" H 4700 4700 50  0000 L CNN
+F 2 "PMPB15XP_115:MOSFET_PMPB55ENEAX" H 5350 5050 50  0001 L BNN
+F 3 "PMPB15XP,115" H 5350 5050 50  0001 L BNN
+F 4 "UDFN-6 Nexperia USA" H 5350 5050 50  0001 L BNN "Field4"
+F 5 "Nexperia USA" H 5350 5050 50  0001 L BNN "Field5"
+F 6 "None" H 5350 5050 50  0001 L BNN "Field6"
+F 7 "Unavailable" H 5350 5050 50  0001 L BNN "Field7"
+F 8 "Trans MOSFET P-CH 12V 8.2A 6-Pin DFN-MD EP T/R" H 5350 5050 50  0001 L BNN "Field8"
+	1    5350 5050
+	1    0    0    -1
+$EndComp
+Wire Wire Line
+	5150 4350 5150 4250
+Wire Wire Line
+	5150 4250 5250 4250
+Connection ~ 5250 4250
+Wire Wire Line
+	5250 4250 5250 4350
+Wire Wire Line
+	4450 4650 4450 4750
+Connection ~ 4450 4750
+Wire Wire Line
+	4450 4750 4450 4850
+Connection ~ 4450 4850
+Wire Wire Line
+	4450 4850 4450 4950
+Connection ~ 4450 4950
+Wire Wire Line
+	4450 4950 4450 5050
+Wire Wire Line
+	3850 4850 4450 4850
+$Comp
+L power:GND #PWR?
+U 1 1 5C4C9F8B
+P 4300 5300
+AR Path="/5C1D48B0/5C4C9F8B" Ref="#PWR?"  Part="1"
+AR Path="/5C4C9F8B" Ref="#PWR?"  Part="1"
+AR Path="/5C4AA0D1/5C4C9F8B" Ref="#PWR0176"  Part="1"
+F 0 "#PWR0176" H 4300 5050 50  0001 C CNN
+F 1 "GND" H 4305 5127 50  0000 C CNN
+F 2 "" H 4300 5300 50  0001 C CNN
+F 3 "" H 4300 5300 50  0001 C CNN
+	1    4300 5300
+	1    0    0    -1
+$EndComp
+Wire Wire Line
+	4450 5250 4300 5250
+Wire Wire Line
+	4300 5250 4300 5300
 $EndSCHEMATC
