File: pcb/badge/Epaper.sch (KiCad schematic (older format))
At the start: 20 parts

Commit message: Fix ERC problems
Parts:
- gave numbers to parts that had none: 20
Changed lines of the file:
@@
 $EndDescr
 $Comp
-L power:GND #PWR?
+L power:GND #PWR0152
 U 1 1 5C21C39F
 P 3900 2450
-F 0 "#PWR?" H 3900 2200 50  0001 C CNN
+F 0 "#PWR0152" H 3900 2200 50  0001 C CNN
 F 1 "GND" V 3905 2322 50  0000 R CNN
 F 2 "" H 3900 2450 50  0001 C CNN
@@
 	3650 2450 3900 2450
 $Comp
-L Device:D_Schottky D?
+L Device:D_Schottky D1
 U 1 1 5C21C3F6
 P 3500 2450
-F 0 "D?" H 3500 2234 50  0000 C CNN
+F 0 "D1" H 3500 2234 50  0000 C CNN
 F 1 "MBR0530" H 3500 2325 50  0000 C CNN
 F 2 "" H 3500 2450 50  0001 C CNN
@@
 	3100 2800 3450 2800
 $Comp
-L Device:D_Schottky D?
+L Device:D_Schottky D3
 U 1 1 5C21C48B
 P 3600 2800
-F 0 "D?" H 3600 3016 50  0000 C CNN
+F 0 "D3" H 3600 3016 50  0000 C CNN
 F 1 "MBR0530" H 3600 2925 50  0000 C CNN
 F 2 "" H 3600 2800 50  0001 C CNN
@@
 	3100 2650 3100 2800
 $Comp
-L Device:C C?
+L Device:C C24
 U 1 1 5C21C5D9
 P 2200 4050
-F 0 "C?" H 2315 4096 50  0000 L CNN
+F 0 "C24" H 2315 4096 50  0000 L CNN
 F 1 "4.7uF" H 2315 4005 50  0000 L CNN
 F 2 "" H 2238 3900 50  0001 C CNN
@@
 	2950 3600 3400 3600
 $Comp
-L Device:D_Schottky D?
+L Device:D_Schottky D2
 U 1 1 5C21C85D
 P 3550 3600
-F 0 "D?" H 3550 3384 50  0000 C CNN
+F 0 "D2" H 3550 3384 50  0000 C CNN
 F 1 "MBR0530" H 3550 3475 50  0000 C CNN
 F 2 "" H 3550 3600 50  0001 C CNN
@@
 	2950 3600 2650 3600
 $Comp
-L Device:L_Core_Iron L?
+L Device:L_Core_Iron L1
 U 1 1 5C21CAD1
 P 2500 3600
-F 0 "L?" V 2725 3600 50  0000 C CNN
+F 0 "L1" V 2725 3600 50  0000 C CNN
 F 1 "68uH" V 2634 3600 50  0000 C CNN
 F 2 "" H 2500 3600 50  0001 C CNN
@@
 $EndComp
 $Comp
-L power:GND #PWR?
+L power:GND #PWR0153
 U 1 1 5C21D11C
 P 2200 4350
-F 0 "#PWR?" H 2200 4100 50  0001 C CNN
+F 0 "#PWR0153" H 2200 4100 50  0001 C CNN
 F 1 "GND" H 2205 4177 50  0000 C CNN
 F 2 "" H 2200 4350 50  0001 C CNN
@@
 	2950 3600 2950 3250
 $Comp
-L power:+3.3V #PWR?
+L power:+3.3V #PWR0154
 U 1 1 5C21D74B
 P 1900 3600
-F 0 "#PWR?" H 1900 3450 50  0001 C CNN
+F 0 "#PWR0154" H 1900 3450 50  0001 C CNN
 F 1 "+3.3V" V 1915 3728 50  0000 L CNN
 F 2 "" H 1900 3600 50  0001 C CNN
@@
 	2350 4750 2350 5450
 $Comp
-L Device:Q_NMOS_GSD Q?
+L Device:Q_NMOS_GSD Q1
 U 1 1 5C21E5CE
 P 2850 4750
-F 0 "Q?" H 3055 4796 50  0000 L CNN
+F 0 "Q1" H 3055 4796 50  0000 L CNN
 F 1 "Si1308EDL" H 3055 4705 50  0000 L CNN
 F 2 "" H 3050 4850 50  0001 C CNN
@@
 $EndComp
 $Comp
-L Device:R R?
+L Device:R R10
 U 1 1 5C21EC08
 P 2350 5600
-F 0 "R?" H 2420 5646 50  0000 L CNN
+F 0 "R10" H 2420 5646 50  0000 L CNN
 F 1 "10K" H 2420 5555 50  0000 L CNN
 F 2 "" V 2280 5600 50  0001 C CNN
@@
 $EndComp
 $Comp
-L Device:R R?
+L Device:R R11
 U 1 1 5C21EC36
 P 2950 5600
-F 0 "R?" H 3020 5646 50  0000 L CNN
+F 0 "R11" H 3020 5646 50  0000 L CNN
 F 1 "3R" H 3020 5555 50  0000 L CNN
 F 2 "" V 2880 5600 50  0001 C CNN
@@
 Connection ~ 2950 5900
 $Comp
-L power:GND #PWR?
+L power:GND #PWR0155
 U 1 1 5C21F181
 P 2950 6000
-F 0 "#PWR?" H 2950 5750 50  0001 C CNN
+F 0 "#PWR0155" H 2950 5750 50  0001 C CNN
 F 1 "GND" H 2955 5827 50  0000 C CNN
 F 2 "" H 2950 6000 50  0001 C CNN
@@
 RESE
 $Comp
-L Connector_Generic:Conn_01x24 J?
+L Connector_Generic:Conn_01x24 J7
 U 1 1 5C21FA6D
 P 8100 3550
-F 0 "J?" H 8180 3542 50  0000 L CNN
+F 0 "J7" H 8180 3542 50  0000 L CNN
 F 1 "PFC24/0.5mm" H 8180 3451 50  0000 L CNN
 F 2 "" H 8100 3550 50  0001 C CNN
@@
 BS
 $Comp
-L power:+3.3V #PWR?
+L power:+3.3V #PWR0156
 U 1 1 5C22A863
 P 7100 3850
-F 0 "#PWR?" H 7100 3700 50  0001 C CNN
+F 0 "#PWR0156" H 7100 3700 50  0001 C CNN
 F 1 "+3.3V" V 7115 3978 50  0000 L CNN
 F 2 "" H 7100 3850 50  0001 C CNN
@@
 	6950 3750 6650 3750
 $Comp
-L Device:C C?
+L Device:C C26
 U 1 1 5C22B69E
 P 6500 3750
-F 0 "C?" V 6450 3600 50  0000 C CNN
+F 0 "C26" V 6450 3600 50  0000 C CNN
 F 1 "100nF" V 6450 3900 50  0000 C CNN
 F 2 "" H 6538 3600 50  0001 C CNN
@@
 $EndComp
 $Comp
-L power:+3.3V #PWR?
+L power:+3.3V #PWR0157
 U 1 1 5C22B722
 P 7350 3950
-F 0 "#PWR?" H 7350 3800 50  0001 C CNN
+F 0 "#PWR0157" H 7350 3800 50  0001 C CNN
 F 1 "+3.3V" V 7365 4078 50  0000 L CNN
 F 2 "" H 7350 3950 50  0001 C CNN
@@
 $EndComp
 $Comp
-L power:GND #PWR?
+L power:GND #PWR0158
 U 1 1 5C22B75A
 P 7350 4050
-F 0 "#PWR?" H 7350 3800 50  0001 C CNN
+F 0 "#PWR0158" H 7350 3800 50  0001 C CNN
 F 1 "GND" V 7355 3922 50  0000 R CNN
 F 2 "" H 7350 4050 50  0001 C CNN
@@
 	6950 4150 7900 4150
 $Comp
-L Device:C C?
+L Device:C C27
 U 1 1 5C22E6B3
 P 6500 3950
-F 0 "C?" V 6450 3800 50  0000 C CNN
+F 0 "C27" V 6450 3800 50  0000 C CNN
 F 1 "1uF" V 6450 4100 50  0000 C CNN
 F 2 "" H 6538 3800 50  0001 C CNN
@@
 	6000 4550 5850 4550
 $Comp
-L power:GND #PWR?
+L power:GND #PWR0159
 U 1 1 5C23BD6D
 P 5850 4550
-F 0 "#PWR?" H 5850 4300 50  0001 C CNN
+F 0 "#PWR0159" H 5850 4300 50  0001 C CNN
 F 1 "GND" V 5855 4422 50  0000 R CNN
 F 2 "" H 5850 4550 50  0001 C CNN
@@
 	6350 2800 6350 2950
 $Comp
-L power:GND #PWR?
+L power:GND #PWR0160
 U 1 1 5C272CFF
 P 6200 2800
-F 0 "#PWR?" H 6200 2550 50  0001 C CNN
+F 0 "#PWR0160" H 6200 2550 50  0001 C CNN
 F 1 "GND" V 6205 2672 50  0000 R CNN
 F 2 "" H 6200 2800 50  0001 C CNN
@@
 $EndComp
 $Comp
-L Device:C C?
+L Device:C C28
 U 1 1 5C273A0A
 P 6500 4150
-F 0 "C?" V 6450 4000 50  0000 C CNN
+F 0 "C28" V 6450 4000 50  0000 C CNN
 F 1 "1uF" V 6450 4300 50  0000 C CNN
 F 2 "" H 6538 4000 50  0001 C CNN
@@
 $EndComp
 $Comp
-L Device:C C?
+L Device:C C29
 U 1 1 5C273A3C
 P 6500 4350
-F 0 "C?" V 6450 4200 50  0000 C CNN
+F 0 "C29" V 6450 4200 50  0000 C CNN
 F 1 "1uF" V 6450 4500 50  0000 C CNN
 F 2 "" H 6538 4200 50  0001 C CNN
@@
 $EndComp
 $Comp
-L Device:C C?
+L Device:C C30
 U 1 1 5C273A84
 P 6500 4550
-F 0 "C?" V 6450 4400 50  0000 C CNN
+F 0 "C30" V 6450 4400 50  0000 C CNN
 F 1 "1uF" V 6450 4700 50  0000 C CNN
 F 2 "" H 6538 4400 50  0001 C CNN
@@
 $EndComp
 $Comp
-L Device:C C?
+L Device:C C31
 U 1 1 5C273ADA
 P 6500 4750
-F 0 "C?" V 6450 4600 50  0000 C CNN
+F 0 "C31" V 6450 4600 50  0000 C CNN
 F 1 "1uF" V 6450 4900 50  0000 C CNN
 F 2 "" H 6538 4600 50  0001 C CNN
@@
 $EndComp
 $Comp
-L Device:C C?
+L Device:C C32
 U 1 1 5C273B12
 P 6500 4950
-F 0 "C?" V 6450 4800 50  0000 C CNN
+F 0 "C32" V 6450 4800 50  0000 C CNN
 F 1 "1uF" V 6450 5100 50  0000 C CNN
 F 2 "" H 6538 4800 50  0001 C CNN
@@
 $EndComp
 $Comp
-L Device:C C?
+L Device:C C33
 U 1 1 5C273B50
 P 6500 5150
-F 0 "C?" V 6450 5000 50  0000 C CNN
+F 0 "C33" V 6450 5000 50  0000 C CNN
 F 1 "1uF" V 6450 5300 50  0000 C CNN
 F 2 "" H 6538 5000 50  0001 C CNN
@@
 $EndComp
 $Comp
-L Device:C C?
+L Device:C C35
 U 1 1 5C273BCC
 P 6700 2950
-F 0 "C?" V 6650 2800 50  0000 C CNN
+F 0 "C35" V 6650 2800 50  0000 C CNN
 F 1 "1uF" V 6650 3100 50  0000 C CNN
 F 2 "" H 6738 2800 50  0001 C CNN
@@
 $EndComp
 $Comp
-L Device:C C?
+L Device:C C34
 U 1 1 5C273C24
 P 6700 2650
-F 0 "C?" V 6650 2500 50  0000 C CNN
+F 0 "C34" V 6650 2500 50  0000 C CNN
 F 1 "1uF" V 6650 2800 50  0000 C CNN
 F 2 "" H 6738 2500 50  0001 C CNN
@@
 $EndComp
 $Comp
-L Device:C C?
+L Device:C C25
 U 1 1 5C274212
 P 2950 3100
-F 0 "C?" V 2900 2950 50  0000 C CNN
+F 0 "C25" V 2900 2950 50  0000 C CNN
 F 1 "100nF" V 2900 3250 50  0000 C CNN
 F 2 "" H 2988 2950 50  0001 C CNN
@@
 BUSY
 $Comp
-L power:GND #PWR?
+L power:GND #PWR0161
 U 1 1 5C27CD98
 P 7350 3150
-F 0 "#PWR?" H 7350 2900 50  0001 C CNN
+F 0 "#PWR0161" H 7350 2900 50  0001 C CNN
 F 1 "GND" V 7355 3022 50  0000 R CNN
 F 2 "" H 7350 3150 50  0001 C CNN

Commit message: Add touch button symbols + footprints
Parts:
- C24, C25, C26, C27, C28, C29, C30, C31, C32, C33, C34, C35: footprint (none) -> Capacitor_SMD:C_0603_1608Metric
- D1, D2, D3: footprint (none) -> Diode_SMD:D_SOD-123
- J7: footprint (none) -> Connector_FFC-FPC:Hirose_FH12-24S-0.5SH_1x24-1MP_P0.50mm_Horizontal
- L1: footprint (none) -> Inductor_SMD:L_1210_3225Metric
- Q1: footprint (none) -> Package_TO_SOT_SMD:SOT-323_SC-70
- R10, R11: footprint (none) -> Resistor_SMD:R_0603_1608Metric
Changed lines of the file:
@@
 F 0 "D1" H 3500 2234 50  0000 C CNN
 F 1 "MBR0530" H 3500 2325 50  0000 C CNN
-F 2 "" H 3500 2450 50  0001 C CNN
+F 2 "Diode_SMD:D_SOD-123" H 3500 2450 50  0001 C CNN
 F 3 "~" H 3500 2450 50  0001 C CNN
 	1    3500 2450
@@
 F 0 "D3" H 3600 3016 50  0000 C CNN
 F 1 "MBR0530" H 3600 2925 50  0000 C CNN
-F 2 "" H 3600 2800 50  0001 C CNN
+F 2 "Diode_SMD:D_SOD-123" H 3600 2800 50  0001 C CNN
 F 3 "~" H 3600 2800 50  0001 C CNN
 	1    3600 2800
@@
 F 0 "C24" H 2315 4096 50  0000 L CNN
 F 1 "4.7uF" H 2315 4005 50  0000 L CNN
-F 2 "" H 2238 3900 50  0001 C CNN
+F 2 "Capacitor_SMD:C_0603_1608Metric" H 2238 3900 50  0001 C CNN
 F 3 "~" H 2200 4050 50  0001 C CNN
 	1    2200 4050
@@
 F 0 "D2" H 3550 3384 50  0000 C CNN
 F 1 "MBR0530" H 3550 3475 50  0000 C CNN
-F 2 "" H 3550 3600 50  0001 C CNN
+F 2 "Diode_SMD:D_SOD-123" H 3550 3600 50  0001 C CNN
 F 3 "~" H 3550 3600 50  0001 C CNN
 	1    3550 3600
@@
 F 0 "L1" V 2725 3600 50  0000 C CNN
 F 1 "68uH" V 2634 3600 50  0000 C CNN
-F 2 "" H 2500 3600 50  0001 C CNN
+F 2 "Inductor_SMD:L_1210_3225Metric" H 2500 3600 50  0001 C CNN
 F 3 "~" H 2500 3600 50  0001 C CNN
 	1    2500 3600
@@
 F 0 "Q1" H 3055 4796 50  0000 L CNN
 F 1 "Si1308EDL" H 3055 4705 50  0000 L CNN
-F 2 "" H 3050 4850 50  0001 C CNN
+F 2 "Package_TO_SOT_SMD:SOT-323_SC-70" H 3050 4850 50  0001 C CNN
 F 3 "~" H 2850 4750 50  0001 C CNN
 	1    2850 4750
@@
 F 0 "R10" H 2420 5646 50  0000 L CNN
 F 1 "10K" H 2420 5555 50  0000 L CNN
-F 2 "" V 2280 5600 50  0001 C CNN
+F 2 "Resistor_SMD:R_0603_1608Metric" V 2280 5600 50  0001 C CNN
 F 3 "~" H 2350 5600 50  0001 C CNN
 	1    2350 5600
@@
 F 0 "R11" H 3020 5646 50  0000 L CNN
 F 1 "3R" H 3020 5555 50  0000 L CNN
-F 2 "" V 2880 5600 50  0001 C CNN
+F 2 "Resistor_SMD:R_0603_1608Metric" V 2880 5600 50  0001 C CNN
 F 3 "~" H 2950 5600 50  0001 C CNN
 	1    2950 5600
@@
 F 0 "J7" H 8180 3542 50  0000 L CNN
 F 1 "PFC24/0.5mm" H 8180 3451 50  0000 L CNN
-F 2 "" H 8100 3550 50  0001 C CNN
+F 2 "Connector_FFC-FPC:Hirose_FH12-24S-0.5SH_1x24-1MP_P0.50mm_Horizontal" H 8100 3550 50  0001 C CNN
 F 3 "~" H 8100 3550 50  0001 C CNN
 	1    8100 3550
@@
 F 0 "C26" V 6450 3600 50  0000 C CNN
 F 1 "100nF" V 6450 3900 50  0000 C CNN
-F 2 "" H 6538 3600 50  0001 C CNN
+F 2 "Capacitor_SMD:C_0603_1608Metric" H 6538 3600 50  0001 C CNN
 F 3 "~" H 6500 3750 50  0001 C CNN
 	1    6500 3750
@@
 F 0 "C27" V 6450 3800 50  0000 C CNN
 F 1 "1uF" V 6450 4100 50  0000 C CNN
-F 2 "" H 6538 3800 50  0001 C CNN
+F 2 "Capacitor_SMD:C_0603_1608Metric" H 6538 3800 50  0001 C CNN
 F 3 "~" H 6500 3950 50  0001 C CNN
 	1    6500 3950
@@
 F 0 "C28" V 6450 4000 50  0000 C CNN
 F 1 "1uF" V 6450 4300 50  0000 C CNN
-F 2 "" H 6538 4000 50  0001 C CNN
+F 2 "Capacitor_SMD:C_0603_1608Metric" H 6538 4000 50  0001 C CNN
 F 3 "~" H 6500 4150 50  0001 C CNN
 	1    6500 4150
@@
 F 0 "C29" V 6450 4200 50  0000 C CNN
 F 1 "1uF" V 6450 4500 50  0000 C CNN
-F 2 "" H 6538 4200 50  0001 C CNN
+F 2 "Capacitor_SMD:C_0603_1608Metric" H 6538 4200 50  0001 C CNN
 F 3 "~" H 6500 4350 50  0001 C CNN
 	1    6500 4350
@@
 F 0 "C30" V 6450 4400 50  0000 C CNN
 F 1 "1uF" V 6450 4700 50  0000 C CNN
-F 2 "" H 6538 4400 50  0001 C CNN
+F 2 "Capacitor_SMD:C_0603_1608Metric" H 6538 4400 50  0001 C CNN
 F 3 "~" H 6500 4550 50  0001 C CNN
 	1    6500 4550
@@
 F 0 "C31" V 6450 4600 50  0000 C CNN
 F 1 "1uF" V 6450 4900 50  0000 C CNN
-F 2 "" H 6538 4600 50  0001 C CNN
+F 2 "Capacitor_SMD:C_0603_1608Metric" H 6538 4600 50  0001 C CNN
 F 3 "~" H 6500 4750 50  0001 C CNN
 	1    6500 4750
@@
 F 0 "C32" V 6450 4800 50  0000 C CNN
 F 1 "1uF" V 6450 5100 50  0000 C CNN
-F 2 "" H 6538 4800 50  0001 C CNN
+F 2 "Capacitor_SMD:C_0603_1608Metric" H 6538 4800 50  0001 C CNN
 F 3 "~" H 6500 4950 50  0001 C CNN
 	1    6500 4950
@@
 F 0 "C33" V 6450 5000 50  0000 C CNN
 F 1 "1uF" V 6450 5300 50  0000 C CNN
-F 2 "" H 6538 5000 50  0001 C CNN
+F 2 "Capacitor_SMD:C_0603_1608Metric" H 6538 5000 50  0001 C CNN
 F 3 "~" H 6500 5150 50  0001 C CNN
 	1    6500 5150
@@
 F 0 "C35" V 6650 2800 50  0000 C CNN
 F 1 "1uF" V 6650 3100 50  0000 C CNN
-F 2 "" H 6738 2800 50  0001 C CNN
+F 2 "Capacitor_SMD:C_0603_1608Metric" H 6738 2800 50  0001 C CNN
 F 3 "~" H 6700 2950 50  0001 C CNN
 	1    6700 2950
@@
 F 0 "C34" V 6650 2500 50  0000 C CNN
 F 1 "1uF" V 6650 2800 50  0000 C CNN
-F 2 "" H 6738 2500 50  0001 C CNN
+F 2 "Capacitor_SMD:C_0603_1608Metric" H 6738 2500 50  0001 C CNN
 F 3 "~" H 6700 2650 50  0001 C CNN
 	1    6700 2650
@@
 F 0 "C25" V 2900 2950 50  0000 C CNN
 F 1 "100nF" V 2900 3250 50  0000 C CNN
-F 2 "" H 2988 2950 50  0001 C CNN
+F 2 "Capacitor_SMD:C_0603_1608Metric" H 2988 2950 50  0001 C CNN
 F 3 "~" H 2950 3100 50  0001 C CNN
 	1    2950 3100

Commit message: Fix reversed connector for EPD
Parts:
- J7: footprint Connector_FFC-FPC:Hirose_FH12-24S-0.5SH_1x24-1MP_P0.50mm_Horizontal -> connectors:EPD-FPC-1x24-P0.50mm_Horizontal
Changed lines of the file:
@@
 F 0 "J7" H 8180 3542 50  0000 L CNN
 F 1 "PFC24/0.5mm" H 8180 3451 50  0000 L CNN
-F 2 "Connector_FFC-FPC:Hirose_FH12-24S-0.5SH_1x24-1MP_P0.50mm_Horizontal" H 8100 3550 50  0001 C CNN
+F 2 "connectors:EPD-FPC-1x24-P0.50mm_Horizontal" H 8100 3550 50  0001 C CNN
 F 3 "~" H 8100 3550 50  0001 C CNN
 	1    8100 3550

Commit message: fix(pcb): update R11 value to 0.47R
This is due to switching our EPaper display panel to GDEW029T5,
which requires a smaller resistor value than the original Waveshare panel
Parts:
- R11: value 3R -> 0.47R
Changed lines of the file:
@@
 P 2950 5600
 F 0 "R11" H 3020 5646 50  0000 L CNN
-F 1 "3R" H 3020 5555 50  0000 L CNN
+F 1 "0.47R" H 3020 5555 50  0000 L CNN
 F 2 "Resistor_SMD:R_0603_1608Metric" V 2880 5600 50  0001 C CNN
 F 3 "~" H 2950 5600 50  0001 C CNN
