File: pcb/tiny-sao/tiny-sao.kicad_pcb (KiCad board)
At the start: 2 copper layers, 20 x 20 mm, 3 parts, among them J1 Conn_02x02_Counter_Clockwise, SW1 SW_Push, U1 ATtiny45-20SU

Commit message: feat(pcb): add indication LED to tiny-sao
Parts:
- added D1: LED, LED_SMD:LED_0603_1608Metric, F.Cu at (135.1, 93.0)
- added R1: R, Resistor_SMD:R_0603_1608Metric, F.Cu at (136.9, 96.0)
Routing:
- net Net-(D1-Pad1): track 0.00 -> 5.15 mm, vias 0 -> 2
- net Net-(D1-Pad2): track 0.00 -> 2.70 mm
- net VCC: track 14.1 -> 14.7 mm
Changed lines of the file:
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@@
     (thickness 1.6)
     (drawings 2)
-    (tracks 31)
+    (tracks 42)
     (zones 0)
-    (modules 3)
-    (nets 9)
+    (modules 5)
+    (nets 10)
   )
   (page A4)
@@
     (solder_mask_min_width 0.25)
     (aux_axis_origin 0 0)
-    (visible_elements FFFFFF7F)
+    (visible_elements 7FFFFFFF)
     (pcbplotparams
       (layerselection 0x010fc_ffffffff)
-      (usegerberextensions false)
+      (usegerberextensions true)
       (usegerberattributes false)
       (usegerberadvancedattributes false)
@@
       (outputformat 1)
       (mirror false)
-      (drillshape 1)
+      (drillshape 0)
       (scaleselection 1)
-      (outputdirectory ""))
+      (outputdirectory "gerber"))
   )
   (net 0 "")
@@
   (net 6 "Net-(U1-Pad2)")
   (net 7 "Net-(U1-Pad3)")
-  (net 8 "Net-(U1-Pad6)")
+  (net 8 "Net-(D1-Pad1)")
+  (net 9 "Net-(D1-Pad2)")
   (net_class Default "This is the default net class."
     (clearance 0.2)
@@
     (add_net /SDA)
     (add_net GND)
+    (add_net "Net-(D1-Pad1)")
+    (add_net "Net-(D1-Pad2)")
     (add_net "Net-(SW1-Pad1)")
     (add_net "Net-(U1-Pad2)")
     (add_net "Net-(U1-Pad3)")
-    (add_net "Net-(U1-Pad6)")
     (add_net VCC)
   )
@@
     (fp_line (start 2.99974 -1.09982) (end 2.99974 1.09982) (layer F.SilkS) (width 0.127))
     (fp_line (start -2.99974 -1.09982) (end -2.99974 1.09982) (layer F.SilkS) (width 0.127))
-    (pad 2 smd rect (at 3.1496 0 135) (size 2.2987 1.59766) (layers F.Cu F.Paste F.Mask)
+    (pad 2 smd rect (at 3.149601 0 135) (size 2.2987 1.59766) (layers F.Cu F.Paste F.Mask)
       (net 2 GND))
-    (pad 1 smd rect (at -3.1496 0 135) (size 2.2987 1.59766) (layers F.Cu F.Paste F.Mask)
+    (pad 1 smd rect (at -3.149601 0 135) (size 2.2987 1.59766) (layers F.Cu F.Paste F.Mask)
       (net 5 "Net-(SW1-Pad1)"))
     (model ${KISYS3DMOD}/Button_Switch_SMD.3dshapes/SW_SPST_CK_RS282G05A3.wrl
@@
       (net 4 /SDA))
     (pad 6 smd rect (at 3.65 0.635) (size 1.7 0.65) (layers F.Cu F.Paste F.Mask)
-      (net 8 "Net-(U1-Pad6)"))
+      (net 8 "Net-(D1-Pad1)"))
     (pad 7 smd rect (at 3.65 -0.635) (size 1.7 0.65) (layers F.Cu F.Paste F.Mask)
       (net 3 /SCL))
@@
     )
   )
-  (gr_text CTF (at 134.62 92.71) (layer F.SilkS)
+  (module LED_SMD:LED_0603_1608Metric (layer F.Cu)
+    (at 135.128 92.964 315)
+    (descr "LED SMD 0603 (1608 Metric), square (rectangular) end terminal, IPC_7351 nominal, (Body size source: http://www.tortai-tech.com/upload/download/2011102023233369053.pdf), generated with kicad-footprint-generator")
+    (tags diode)
+    (attr smd)
+    (fp_text reference D1 (at 0 -1.43 315) (layer F.SilkS) hide
+      (effects (font (size 1 1) (thickness 0.15)))
+    )
+    (fp_text value LED (at 0 1.43 315) (layer F.Fab)
+      (effects (font (size 1 1) (thickness 0.15)))
+    )
+    (fp_line (start 0.8 -0.4) (end -0.5 -0.4) (layer F.Fab) (width 0.1))
+    (fp_line (start -0.5 -0.4) (end -0.8 -0.1) (layer F.Fab) (width 0.1))
+    (fp_line (start -0.8 -0.1) (end -0.8 0.4) (layer F.Fab) (width 0.1))
+    (fp_line (start -0.8 0.4) (end 0.8 0.4) (layer F.Fab) (width 0.1))
+    (fp_line (start 0.8 0.4) (end 0.8 -0.4) (layer F.Fab) (width 0.1))
+    (fp_line (start 0.8 -0.735) (end -1.485 -0.735) (layer F.SilkS) (width 0.12))
+    (fp_line (start -1.485 -0.735) (end -1.485 0.735) (layer F.SilkS) (width 0.12))
+    (fp_line (start -1.485 0.735) (end 0.8 0.735) (layer F.SilkS) (width 0.12))
+    (fp_line (start -1.48 0.73) (end -1.48 -0.73) (layer F.CrtYd) (width 0.05))
+    (fp_line (start -1.48 -0.73) (end 1.48 -0.73) (layer F.CrtYd) (width 0.05))
+    (fp_line (start 1.48 -0.73) (end 1.48 0.73) (layer F.CrtYd) (width 0.05))
+    (fp_line (start 1.48 0.73) (end -1.48 0.73) (layer F.CrtYd) (width 0.05))
+    (fp_text user %R (at 0 0 315) (layer F.Fab)
+      (effects (font (size 0.4 0.4) (thickness 0.06)))
+    )
+    (pad 1 smd roundrect (at -0.787501 0 315) (size 0.875 0.95) (layers F.Cu F.Paste F.Mask) (roundrect_rratio 0.25)
+      (net 8 "Net-(D1-Pad1)"))
+    (pad 2 smd roundrect (at 0.787501 0 315) (size 0.875 0.95) (layers F.Cu F.Paste F.Mask) (roundrect_rratio 0.25)
+      (net 9 "Net-(D1-Pad2)"))
+    (model ${KISYS3DMOD}/LED_SMD.3dshapes/LED_0603_1608Metric.wrl
+      (at (xyz 0 0 0))
+      (scale (xyz 1 1 1))
+      (rotate (xyz 0 0 0))
+    )
+  )
+  (module Resistor_SMD:R_0603_1608Metric (layer F.Cu)
+    (at 136.906 96.0375 45)
+    (descr "Resistor SMD 0603 (1608 Metric), square (rectangular) end terminal, IPC_7351 nominal, (Body size source: http://www.tortai-tech.com/upload/download/2011102023233369053.pdf), generated with kicad-footprint-generator")
+    (tags resistor)
+    (attr smd)
+    (fp_text reference R1 (at 0 -1.43 45) (layer F.SilkS) hide
+      (effects (font (size 1 1) (thickness 0.15)))
+    )
+    (fp_text value R (at 0 1.43 45) (layer F.Fab)
+      (effects (font (size 1 1) (thickness 0.15)))
+    )
+    (fp_line (start -0.8 0.4) (end -0.8 -0.4) (layer F.Fab) (width 0.1))
+    (fp_line (start -0.8 -0.4) (end 0.8 -0.4) (layer F.Fab) (width 0.1))
+    (fp_line (start 0.8 -0.4) (end 0.8 0.4) (layer F.Fab) (width 0.1))
+    (fp_line (start 0.8 0.4) (end -0.8 0.4) (layer F.Fab) (width 0.1))
+    (fp_line (start -0.162779 -0.51) (end 0.162779 -0.51) (layer F.SilkS) (width 0.12))
+    (fp_line (start -0.162779 0.51) (end 0.162779 0.51) (layer F.SilkS) (width 0.12))
+    (fp_line (start -1.48 0.73) (end -1.48 -0.73) (layer F.CrtYd) (width 0.05))
+    (fp_line (start -1.48 -0.73) (end 1.48 -0.73) (layer F.CrtYd) (width 0.05))
+    (fp_line (start 1.48 -0.73) (end 1.48 0.73) (layer F.CrtYd) (width 0.05))
+    (fp_line (start 1.48 0.73) (end -1.48 0.73) (layer F.CrtYd) (width 0.05))
+    (fp_text user %R (at 0 0 45) (layer F.Fab)
+      (effects (font (size 0.4 0.4) (thickness 0.06)))
+    )
+    (pad 1 smd roundrect (at -0.7875 0 45) (size 0.875 0.95) (layers F.Cu F.Paste F.Mask) (roundrect_rratio 0.25)
+      (net 1 VCC))
+    (pad 2 smd roundrect (at 0.7875 0 45) (size 0.875 0.95) (layers F.Cu F.Paste F.Mask) (roundrect_rratio 0.25)
+      (net 9 "Net-(D1-Pad2)"))
+    (model ${KISYS3DMOD}/Resistor_SMD.3dshapes/R_0603_1608Metric.wrl
+      (at (xyz 0 0 0))
+      (scale (xyz 1 1 1))
+      (rotate (xyz 0 0 0))
+    )
+  )
+  (gr_text CTF (at 129.921 89.916) (layer F.SilkS)
     (effects (font (size 1.5 1.5) (thickness 0.3)))
   )
@@
   (segment (start 131.429 92.329) (end 135.854002 96.754002) (width 0.25) (layer F.Cu) (net 1) (status 10))
   (segment (start 130.904 92.329) (end 131.429 92.329) (width 0.25) (layer F.Cu) (net 1) (status 30))
+  (segment (start 136.013657 96.594347) (end 135.854002 96.754002) (width 0.25) (layer F.Cu) (net 1))
+  (segment (start 136.349153 96.594347) (end 136.013657 96.594347) (width 0.25) (layer F.Cu) (net 1))
   (segment (start 127.488601 99.498601) (end 127.488601 102.609001) (width 0.25) (layer F.Cu) (net 2))
   (segment (start 124.129 96.139) (end 127.488601 99.498601) (width 0.25) (layer F.Cu) (net 2) (status 10))
@@
   (segment (start 123.079 92.329) (end 122.428999 92.979001) (width 0.25) (layer F.Cu) (net 5))
   (segment (start 123.604 92.329) (end 123.079 92.329) (width 0.25) (layer F.Cu) (net 5))
+  (segment (start 134.571153 92.407153) (end 133.633306 93.345) (width 0.25) (layer F.Cu) (net 8))
+  (via (at 133.633306 93.345) (size 0.8) (drill 0.4) (layers F.Cu B.Cu) (net 8))
+  (segment (start 133.633306 93.345) (end 133.633306 93.950694) (width 0.25) (layer B.Cu) (net 8))
+  (via (at 132.588 94.996) (size 0.8) (drill 0.4) (layers F.Cu B.Cu) (net 8))
+  (segment (start 133.633306 93.950694) (end 132.588 94.996) (width 0.25) (layer B.Cu) (net 8))
+  (segment (start 131.031 94.996) (end 130.904 94.869) (width 0.25) (layer F.Cu) (net 8))
+  (segment (start 132.588 94.996) (end 131.031 94.996) (width 0.25) (layer F.Cu) (net 8))
+  (segment (start 137.462847 95.298847) (end 137.462847 95.480653) (width 0.25) (layer F.Cu) (net 9))
+  (segment (start 135.684847 93.520847) (end 137.462847 95.298847) (width 0.25) (layer F.Cu) (net 9))
   (zone (net 2) (net_name GND) (layer F.Cu) (hatch edge 0.508)
     (connect_pads (clearance 0.508))
