File: pcb/tiny-sao/tiny-sao.sch (KiCad schematic (older format))
At the start: 3 parts, among them J1 Conn_02x02_Counter_Clockwise, SW1 SW_Push, U1 ATtiny45-20SU

Commit message: feat(pcb): add indication LED to tiny-sao
Parts:
- added D1: LED, LED_SMD:LED_0603_1608Metric, symbol Device:LED
- added R1: R, Resistor_SMD:R_0603_1608Metric, symbol Device:R
Connections:
- wire segments 6 -> 10
Changed lines of the file:
@@
 EESchema Schematic File Version 4
+LIBS:tiny-sao-cache
 EELAYER 26 0
 EELAYER END
@@
 Text Label 5850 3450 0    50   ~ 0
 SCL
+$Comp
+L Device:LED D1
+U 1 1 5C4FBC5C
+P 6750 3100
+F 0 "D1" V 6788 2983 50  0000 R CNN
+F 1 "LED" V 6697 2983 50  0000 R CNN
+F 2 "LED_SMD:LED_0603_1608Metric" H 6750 3100 50  0001 C CNN
+F 3 "~" H 6750 3100 50  0001 C CNN
+	1    6750 3100
+	0    -1   -1   0
+$EndComp
+$Comp
+L Device:R R1
+U 1 1 5C4FBE85
+P 6750 2650
+F 0 "R1" H 6820 2696 50  0000 L CNN
+F 1 "R" H 6820 2605 50  0000 L CNN
+F 2 "Resistor_SMD:R_0603_1608Metric" V 6680 2650 50  0001 C CNN
+F 3 "~" H 6750 2650 50  0001 C CNN
+	1    6750 2650
+	1    0    0    -1
+$EndComp
+Wire Wire Line
+	6750 2800 6750 2950
+Wire Wire Line
+	6750 3250 6750 3350
+Wire Wire Line
+	5750 3350 6750 3350
+$Comp
+L power:VCC #PWR0106
+U 1 1 5C4FC051
+P 6600 2500
+F 0 "#PWR0106" H 6600 2350 50  0001 C CNN
+F 1 "VCC" H 6617 2673 50  0000 C CNN
+F 2 "" H 6600 2500 50  0001 C CNN
+F 3 "" H 6600 2500 50  0001 C CNN
+	1    6600 2500
+	0    -1   -1   0
+$EndComp
+Wire Wire Line
+	6750 2500 6600 2500
 $EndSCHEMATC
