File: pcbv2/badge2.sch (KiCad schematic (older format))
At the start: 25 parts, among them J1 Conn_02x04_Counter_Clockwise, J2 SAO_CONN, J3 USB_C_Receptacle_USB2.0, J6 Conn_ARM_JTAG_SWD_10, Q2 Si1308EDL, SW1 SW_Push, SW2 SW_Push, SW3 SW_Push, U3 E73-2G4M08S1C, U5 GD25Q16C, U7 LIS2DH12TR

Commit message: feat(pcbv2): remove 2 neopixels
We only want two in the new design
Parts:
- removed D8, D9: WS2812B, LED_SMD:LED_WS2812B_PLCC4_5.0x5.0mm_P3.2mm, symbol LED:WS2812B
Connections:
- wire segments 133 -> 127
Changed lines of the file:
@@
 	4350 6200 3900 6200
-$Comp
-L LED:WS2812B D8
-U 1 1 5C3CF153
-P 4650 6650
-F 0 "D8" V 4604 6991 50  0000 L CNN
-F 1 "WS2812B" V 4695 6991 50  0000 L CNN
-F 2 "LED_SMD:LED_WS2812B_PLCC4_5.0x5.0mm_P3.2mm" H 4700 6350 50  0001 L TNN
-F 3 "https://cdn-shop.adafruit.com/datasheets/WS2812B.pdf" H 4750 6275 50  0001 L TNN
-	1    4650 6650
-	0    1    1    0
-$EndComp
-$Comp
-L LED:WS2812B D9
-U 1 1 5C3CF19D
-P 4650 7350
-F 0 "D9" V 4604 7691 50  0000 L CNN
-F 1 "WS2812B" V 4695 7691 50  0000 L CNN
-F 2 "LED_SMD:LED_WS2812B_PLCC4_5.0x5.0mm_P3.2mm" H 4700 7050 50  0001 L TNN
-F 3 "https://cdn-shop.adafruit.com/datasheets/WS2812B.pdf" H 4750 6975 50  0001 L TNN
-	1    4650 7350
-	0    1    1    0
-$EndComp
-Wire Wire Line
-	4950 6150 4950 6650
-Connection ~ 4950 6150
-Wire Wire Line
-	4950 7350 4950 6650
-Connection ~ 4950 6650
-Wire Wire Line
-	4350 6200 4350 6650
-Connection ~ 4350 6200
-Wire Wire Line
-	4350 6650 4350 7350
-Connection ~ 4350 6650
-Wire Wire Line
-	4650 6950 4650 7050
-Wire Wire Line
-	4650 6350 4650 6150
 $Comp
 L Switch:SW_Push SW1

Commit message: feat(pcbv2): replace keyboard buttons with 6x6 buttons
Now we have 4 buttons: top/left/right/down instead of the 3 keyboard buttons we used to have
Parts:
- added BTN4: RIGHT, Button_Switch_SMD:SW_Push_1P1T_NO_6x6mm_H9.5mm, symbol Switch:SW_Push
- BTN1: renamed from SW1; value SW_Push -> TOP; footprint Button_Switch_Keyboard:SW_Cherry_MX1A_1.00u_PCB -> Button_Switch_SMD:SW_Push_1P1T_NO_6x6mm_H9.5mm
- BTN2: renamed from SW2; value SW_Push -> LEFT; footprint Button_Switch_Keyboard:SW_Cherry_MX1A_1.00u_PCB -> Button_Switch_SMD:SW_Push_1P1T_NO_6x6mm_H9.5mm
- BTN3: renamed from SW3; value SW_Push -> DOWN; footprint Button_Switch_Keyboard:SW_Cherry_MX1A_1.00u_PCB -> Button_Switch_SMD:SW_Push_1P1T_NO_6x6mm_H9.5mm
Connections:
- wire segments 127 -> 131
Changed lines of the file:
@@
 Wire Wire Line
 	4350 6200 3900 6200
-$Comp
-L Switch:SW_Push SW1
-U 1 1 5C3D29EC
-P 6800 2650
-F 0 "SW1" H 6800 2935 50  0000 C CNN
-F 1 "SW_Push" H 6800 2844 50  0000 C CNN
-F 2 "Button_Switch_Keyboard:SW_Cherry_MX1A_1.00u_PCB" H 6800 2850 50  0001 C CNN
-F 3 "" H 6800 2850 50  0001 C CNN
-	1    6800 2650
-	1    0    0    -1
-$EndComp
-$Comp
-L Switch:SW_Push SW2
-U 1 1 5C3D2AC9
-P 6800 3050
-F 0 "SW2" H 6800 3335 50  0000 C CNN
-F 1 "SW_Push" H 6800 3244 50  0000 C CNN
-F 2 "Button_Switch_Keyboard:SW_Cherry_MX1A_1.00u_PCB" H 6800 3250 50  0001 C CNN
-F 3 "" H 6800 3250 50  0001 C CNN
-	1    6800 3050
-	1    0    0    -1
-$EndComp
-$Comp
-L Switch:SW_Push SW3
-U 1 1 5C3D2B3F
-P 6800 3450
-F 0 "SW3" H 6800 3735 50  0000 C CNN
-F 1 "SW_Push" H 6800 3644 50  0000 C CNN
-F 2 "Button_Switch_Keyboard:SW_Cherry_MX1A_1.00u_PCB" H 6800 3650 50  0001 C CNN
-F 3 "" H 6800 3650 50  0001 C CNN
-	1    6800 3450
-	1    0    0    -1
-$EndComp
 Wire Wire Line
 	6350 2850 5800 2850
@@
 F1 "lipo.sch" 50
 $EndSheet
+Wire Wire Line
+	5800 3300 6500 3300
+Wire Wire Line
+	6500 3300 6500 3850
+Wire Wire Line
+	6500 3850 6600 3850
+Wire Wire Line
+	7000 3850 7000 3450
+Connection ~ 7000 3450
+$Comp
+L Switch:SW_Push BTN3
+U 1 1 5C3D2B3F
+P 6800 3450
+F 0 "BTN3" H 6800 3735 50  0000 C CNN
+F 1 "DOWN" H 6800 3644 50  0000 C CNN
+F 2 "Button_Switch_SMD:SW_Push_1P1T_NO_6x6mm_H9.5mm" H 6800 3650 50  0001 C CNN
+F 3 "" H 6800 3650 50  0001 C CNN
+	1    6800 3450
+	1    0    0    -1
+$EndComp
+$Comp
+L Switch:SW_Push BTN2
+U 1 1 5C3D2AC9
+P 6800 3050
+F 0 "BTN2" H 6800 3335 50  0000 C CNN
+F 1 "LEFT" H 6800 3244 50  0000 C CNN
+F 2 "Button_Switch_SMD:SW_Push_1P1T_NO_6x6mm_H9.5mm" H 6800 3250 50  0001 C CNN
+F 3 "" H 6800 3250 50  0001 C CNN
+	1    6800 3050
+	1    0    0    -1
+$EndComp
+$Comp
+L Switch:SW_Push BTN1
+U 1 1 5C3D29EC
+P 6800 2650
+F 0 "BTN1" H 6800 2935 50  0000 C CNN
+F 1 "TOP" H 6800 2844 50  0000 C CNN
+F 2 "Button_Switch_SMD:SW_Push_1P1T_NO_6x6mm_H9.5mm" H 6800 2850 50  0001 C CNN
+F 3 "" H 6800 2850 50  0001 C CNN
+	1    6800 2650
+	1    0    0    -1
+$EndComp
+$Comp
+L Switch:SW_Push BTN4
+U 1 1 5DA11288
+P 6800 3850
+F 0 "BTN4" H 6800 4135 50  0000 C CNN
+F 1 "RIGHT" H 6800 4044 50  0000 C CNN
+F 2 "Button_Switch_SMD:SW_Push_1P1T_NO_6x6mm_H9.5mm" H 6800 4050 50  0001 C CNN
+F 3 "" H 6800 4050 50  0001 C CNN
+	1    6800 3850
+	1    0    0    -1
+$EndComp
 $EndSCHEMATC

Commit message: feat(pcbv2): add action button
Parts:
- added BTN5: ACTION, Button_Switch_SMD:SW_Push_1P1T_NO_6x6mm_H9.5mm, symbol Switch:SW_Push
Connections:
- wire segments 131 -> 134
Other:
- moved on the sheet: D4, R12
Changed lines of the file:
@@
 L Device:LED D4
 U 1 1 5C21B86B
-P 1800 4450
-F 0 "D4" H 1792 4195 50  0000 C CNN
-F 1 "LED" H 1792 4286 50  0000 C CNN
-F 2 "LED_SMD:LED_0603_1608Metric" H 1800 4450 50  0001 C CNN
-F 3 "~" H 1800 4450 50  0001 C CNN
-	1    1800 4450
+P 1350 5150
+F 0 "D4" H 1342 4895 50  0000 C CNN
+F 1 "LED" H 1342 4986 50  0000 C CNN
+F 2 "LED_SMD:LED_0603_1608Metric" H 1350 5150 50  0001 C CNN
+F 3 "~" H 1350 5150 50  0001 C CNN
+	1    1350 5150
 	-1   0    0    1
 $EndComp
@@
 L power:+3.3V #PWR0139
 U 1 1 5C21C876
-P 1150 4250
-F 0 "#PWR0139" H 1150 4100 50  0001 C CNN
-F 1 "+3.3V" H 1165 4423 50  0000 C CNN
-F 2 "" H 1150 4250 50  0001 C CNN
-F 3 "" H 1150 4250 50  0001 C CNN
-	1    1150 4250
+P 700 4950
+F 0 "#PWR0139" H 700 4800 50  0001 C CNN
+F 1 "+3.3V" H 715 5123 50  0000 C CNN
+F 2 "" H 700 4950 50  0001 C CNN
+F 3 "" H 700 4950 50  0001 C CNN
+	1    700  4950
 	1    0    0    -1
 $EndComp
@@
 L Device:R R12
 U 1 1 5C21C8AD
-P 1400 4450
-F 0 "R12" V 1193 4450 50  0000 C CNN
-F 1 "470R" V 1284 4450 50  0000 C CNN
-F 2 "Resistor_SMD:R_0603_1608Metric" V 1330 4450 50  0001 C CNN
-F 3 "~" H 1400 4450 50  0001 C CNN
-	1    1400 4450
+P 950 5150
+F 0 "R12" V 743 5150 50  0000 C CNN
+F 1 "470R" V 834 5150 50  0000 C CNN
+F 2 "Resistor_SMD:R_0603_1608Metric" V 880 5150 50  0001 C CNN
+F 3 "~" H 950 5150 50  0001 C CNN
+	1    950  5150
 	0    1    1    0
 $EndComp
@@
 L power:GND #PWR0140
 U 1 1 5C21E734
-P 2200 4450
-F 0 "#PWR0140" H 2200 4200 50  0001 C CNN
-F 1 "GND" H 2205 4277 50  0000 C CNN
-F 2 "" H 2200 4450 50  0001 C CNN
-F 3 "" H 2200 4450 50  0001 C CNN
-	1    2200 4450
+P 1750 5150
+F 0 "#PWR0140" H 1750 4900 50  0001 C CNN
+F 1 "GND" H 1755 4977 50  0000 C CNN
+F 2 "" H 1750 5150 50  0001 C CNN
+F 3 "" H 1750 5150 50  0001 C CNN
+	1    1750 5150
 	0    -1   -1   0
 $EndComp
 Wire Wire Line
-	2200 4450 1950 4450
-Wire Wire Line
-	1650 4450 1550 4450
-Wire Wire Line
-	1250 4450 1150 4450
-Wire Wire Line
-	1150 4450 1150 4250
+	1750 5150 1500 5150
+Wire Wire Line
+	1200 5150 1100 5150
+Wire Wire Line
+	800  5150 700  5150
+Wire Wire Line
+	700  5150 700  4950
 Text Label 4650 4750 1    50   ~ 0
 NEOPIXEL
@@
 	1    0    0    -1
 $EndComp
+$Comp
+L Switch:SW_Push BTN5
+U 1 1 5DA74DB7
+P 2100 4250
+F 0 "BTN5" H 2100 4535 50  0000 C CNN
+F 1 "ACTION" H 2100 4444 50  0000 C CNN
+F 2 "Button_Switch_SMD:SW_Push_1P1T_NO_6x6mm_H9.5mm" H 2100 4450 50  0001 C CNN
+F 3 "" H 2100 4450 50  0001 C CNN
+	1    2100 4250
+	0    -1   -1   0
+$EndComp
+Wire Wire Line
+	2400 4050 2100 4050
+$Comp
+L power:GND #PWR?
+U 1 1 5DA89890
+P 1950 4600
+F 0 "#PWR?" H 1950 4350 50  0001 C CNN
+F 1 "GND" V 1955 4472 50  0000 R CNN
+F 2 "" H 1950 4600 50  0001 C CNN
+F 3 "" H 1950 4600 50  0001 C CNN
+	1    1950 4600
+	0    1    1    0
+$EndComp
+Wire Wire Line
+	2100 4450 2100 4600
+Wire Wire Line
+	2100 4600 1950 4600
 $EndSCHEMATC

Commit message: refactor(pcbv2): move accelerometer to own sheet
Parts:
- removed C38: 10uF, Capacitor_SMD:C_0603_1608Metric, symbol Device:C
- removed C39: 100nF, Capacitor_SMD:C_0603_1608Metric, symbol Device:C
- removed U7: LIS2DH12TR, Package_LGA:LGA-12_2x2mm_P0.5mm, symbol LIS2DH12TR:LIS2DH12TR
Connections:
- wire segments 134 -> 115
- no-connect marks 6 -> 4
Other:
- moved on the sheet: J2

Commit message: feat(pcbv2): add FM module connector
Parts:
- added J4: Conn_01x08_Female, Connector_PinSocket_2.54mm:PinSocket_1x08_P2.54mm_Horizontal, symbol Connector:Conn_01x08_Female
Connections:
- net labels added: FM_~RST
- wire segments 115 -> 121
- no-connect marks 4 -> 7
Changed lines of the file:
@@
 Text Label 8900 4750 0    50   ~ 0
 SDA
+$Comp
+L Connector:Conn_01x08_Female J4
+U 1 1 5DAFBF97
+P 7800 5500
+F 0 "J4" H 7828 5476 50  0000 L CNN
+F 1 "Conn_01x08_Female" H 7828 5385 50  0000 L CNN
+F 2 "Connector_PinSocket_2.54mm:PinSocket_1x08_P2.54mm_Horizontal" H 7800 5500 50  0001 C CNN
+F 3 "~" H 7800 5500 50  0001 C CNN
+	1    7800 5500
+	1    0    0    -1
+$EndComp
+$Comp
+L power:GND #PWR?
+U 1 1 5DB0509B
+P 7350 5300
+F 0 "#PWR?" H 7350 5050 50  0001 C CNN
+F 1 "GND" V 7355 5172 50  0000 R CNN
+F 2 "" H 7350 5300 50  0001 C CNN
+F 3 "" H 7350 5300 50  0001 C CNN
+	1    7350 5300
+	0    1    1    0
+$EndComp
+Wire Wire Line
+	7600 5300 7350 5300
+$Comp
+L power:+3.3V #PWR?
+U 1 1 5DB09B35
+P 7400 5200
+F 0 "#PWR?" H 7400 5050 50  0001 C CNN
+F 1 "+3.3V" H 7415 5373 50  0000 C CNN
+F 2 "" H 7400 5200 50  0001 C CNN
+F 3 "" H 7400 5200 50  0001 C CNN
+	1    7400 5200
+	1    0    0    -1
+$EndComp
+Wire Wire Line
+	7600 5200 7400 5200
+Text Label 7500 5400 2    50   ~ 0
+SDA
+Wire Wire Line
+	7600 5400 7350 5400
+Text Label 7350 5500 0    50   ~ 0
+SCL
+Wire Wire Line
+	7600 5500 7350 5500
+Wire Wire Line
+	5250 2050 5250 1700
+Text Label 5250 2000 1    50   ~ 0
+FM_~RST
+Text Label 7550 5700 2    50   ~ 0
+FM_~RST
+Wire Wire Line
+	7600 5700 7350 5700
+NoConn ~ 7600 5600
+NoConn ~ 7600 5800
+NoConn ~ 7600 5900
 $EndSCHEMATC

Commit message: feat(pcbv2): add reset button
Parts:
- added BTN6: RESET, Button_Switch_SMD:SW_SPST_PTS810, symbol Switch:SW_Push
Connections:
- wire segments 121 -> 123
Changed lines of the file:
@@
 $EndComp
 $Comp
-L power:GND #PWR?
+L power:GND #PWR0120
 U 1 1 5DB0509B
 P 7350 5300
-F 0 "#PWR?" H 7350 5050 50  0001 C CNN
+F 0 "#PWR0120" H 7350 5050 50  0001 C CNN
 F 1 "GND" V 7355 5172 50  0000 R CNN
 F 2 "" H 7350 5300 50  0001 C CNN
@@
 	7600 5300 7350 5300
 $Comp
-L power:+3.3V #PWR?
+L power:+3.3V #PWR0121
 U 1 1 5DB09B35
 P 7400 5200
-F 0 "#PWR?" H 7400 5050 50  0001 C CNN
+F 0 "#PWR0121" H 7400 5050 50  0001 C CNN
 F 1 "+3.3V" H 7415 5373 50  0000 C CNN
 F 2 "" H 7400 5200 50  0001 C CNN
@@
 NoConn ~ 7600 5800
 NoConn ~ 7600 5900
+$Comp
+L Switch:SW_Push BTN6
+U 1 1 5DB3D78E
+P 2000 2700
+F 0 "BTN6" H 2000 2985 50  0000 C CNN
+F 1 "RESET" H 2000 2894 50  0000 C CNN
+F 2 "Button_Switch_SMD:SW_SPST_PTS810" H 2000 2900 50  0001 C CNN
+F 3 "" H 2000 2900 50  0001 C CNN
+	1    2000 2700
+	1    0    0    -1
+$EndComp
+Wire Wire Line
+	2200 2700 2400 2700
+$Comp
+L power:GND #PWR0122
+U 1 1 5DB476F4
+P 1600 2700
+F 0 "#PWR0122" H 1600 2450 50  0001 C CNN
+F 1 "GND" V 1605 2572 50  0000 R CNN
+F 2 "" H 1600 2700 50  0001 C CNN
+F 3 "" H 1600 2700 50  0001 C CNN
+	1    1600 2700
+	1    0    0    -1
+$EndComp
+Wire Wire Line
+	1800 2700 1600 2700
 $EndSCHEMATC

Commit message: cleanup(pcbv2): remove Cortex-M connector
Parts:
- removed J6: Conn_ARM_JTAG_SWD_10, Connector_PinHeader_1.27mm:PinHeader_2x05_P1.27mm_Vertical_SMD, symbol badge2-rescue:Conn_ARM_JTAG_SWD_10-Connector
- J1: value Conn_02x04_Counter_Clockwise -> SOICbite
Connections:
- wire segments 123 -> 119
Changed lines of the file:
@@
 SCLK
-Wire Wire Line
-	8300 1450 8650 1450
-Text Label 8350 1450 0    50   ~ 0
-SWDIO
-Text Label 8350 1350 0    50   ~ 0
-SWDCLK
-$Comp
-L power:+3.3V #PWR0148
-U 1 1 5C1C8FC9
-P 7800 750
-F 0 "#PWR0148" H 7800 600 50  0001 C CNN
-F 1 "+3.3V" H 7815 923 50  0000 C CNN
-F 2 "" H 7800 750 50  0001 C CNN
-F 3 "" H 7800 750 50  0001 C CNN
-	1    7800 750
-	1    0    0    -1
-$EndComp
 Wire Wire Line
 	2400 3750 2000 3750
@@
 Text Label 2050 3750 0    50   ~ 0
 SWDCLK
-$Comp
-L power:GND #PWR0149
-U 1 1 5C1CA857
-P 7800 2250
-F 0 "#PWR0149" H 7800 2000 50  0001 C CNN
-F 1 "GND" H 7805 2077 50  0000 C CNN
-F 2 "" H 7800 2250 50  0001 C CNN
-F 3 "" H 7800 2250 50  0001 C CNN
-	1    7800 2250
-	1    0    0    -1
-$EndComp
 Text Label 8700 2150 0    50   ~ 0
 MOSI
@@
 Wire Wire Line
 	8700 2150 9100 2150
-Wire Wire Line
-	8300 1350 8650 1350
 $Comp
 L power:GND #PWR0162
@@
 Wire Wire Line
 	7000 3050 7000 3450
-$Comp
-L badge2-rescue:Conn_ARM_JTAG_SWD_10-Connector J6
-U 1 1 5C3F1CD3
-P 7800 1450
-F 0 "J6" V 7250 1500 50  0000 R CNN
-F 1 "Conn_ARM_JTAG_SWD_10" V 7350 1850 50  0000 R CNN
-F 2 "Connector_PinHeader_1.27mm:PinHeader_2x05_P1.27mm_Vertical_SMD" H 7850 900 50  0001 L TNN
-F 3 "http://infocenter.arm.com/help/topic/com.arm.doc.faqs/attached/13634/cortex_debug_connectors.pdf" V 7450 200 50  0001 C CNN
-	1    7800 1450
-	1    0    0    -1
-$EndComp
-Wire Wire Line
-	7800 2050 7800 2250
-Wire Wire Line
-	7800 750  7800 850
 $Comp
 L Connector_Generic:Conn_02x03_Odd_Even J2
@@
 P 4600 900
 F 0 "J1" H 4650 1217 50  0000 C CNN
-F 1 "Conn_02x04_Counter_Clockwise" H 4650 1126 50  0000 C CNN
+F 1 "SOICbite" H 4650 1126 50  0000 C CNN
 F 2 "SOICbite:SOIC_clipProgSmall" H 4600 900 50  0001 C CNN
 F 3 "~" H 4600 900 50  0001 C CNN

Commit message: feat(pcbv2): replace flash memory
Upgrade flash to 128MBit (16MByte):
GD25Q16C → W25Q128JVS

The new flash chip has a different package (SOIC-8  208-mil), so the PCB was updated with the new footprint
Parts:
- U5: value GD25Q16C -> W25Q128JVSIQ; footprint Package_SO:SOIC-8_3.9x4.9mm_P1.27mm -> Package_SO:SOIC-8_5.23x5.23mm_P1.27mm; symbol Memory_Flash:AT25SF081-SSHD-X -> Memory_Flash:W25Q32JVSS; LCSC Part (none) -> C97521
Connections:
- net labels added: FLASH_CLK, FLASH_CS, FLASH_DI, FLASH_DO, FLASH_IO2, FLASH_IO3
- net labels removed: FLASH_SO
Other:
- moved on the sheet: U5
Changed lines of the file:
@@
 Text Label 5850 2700 0    50   ~ 0
 V_BAT
-$Comp
-L Memory_Flash:AT25SF081-SSHD-X U5
-U 1 1 5C51FC1A
-P 3400 5100
-F 0 "U5" H 4041 5146 50  0000 L CNN
-F 1 "GD25Q16C" H 4041 5055 50  0000 L CNN
-F 2 "Package_SO:SOIC-8_3.9x4.9mm_P1.27mm" H 3400 4500 50  0001 C CNN
-F 3 "https://www.adestotech.com/wp-content/uploads/DS-AT25SF081_045.pdf" H 3400 5100 50  0001 C CNN
-	1    3400 5100
-	0    1    1    0
-$EndComp
-$Comp
-L power:GND #PWR?
-U 1 1 5C51FD2C
-P 2850 5100
-AR Path="/5C1D48B0/5C51FD2C" Ref="#PWR?"  Part="1"
-AR Path="/5C51FD2C" Ref="#PWR0171"  Part="1"
-F 0 "#PWR0171" H 2850 4850 50  0001 C CNN
-F 1 "GND" H 2855 4927 50  0000 C CNN
-F 2 "" H 2850 5100 50  0001 C CNN
-F 3 "" H 2850 5100 50  0001 C CNN
-	1    2850 5100
-	0    1    1    0
-$EndComp
-Wire Wire Line
-	2900 5100 2850 5100
-$Comp
-L power:+3.3V #PWR0172
-U 1 1 5C522E76
-P 4000 5100
-F 0 "#PWR0172" H 4000 4950 50  0001 C CNN
-F 1 "+3.3V" H 4015 5273 50  0000 C CNN
-F 2 "" H 4000 5100 50  0001 C CNN
-F 3 "" H 4000 5100 50  0001 C CNN
-	1    4000 5100
-	0    1    1    0
-$EndComp
-Wire Wire Line
-	4000 5100 3900 5100
-Wire Wire Line
-	3150 4350 3150 4500
-Wire Wire Line
-	3150 4500 3200 4500
-Wire Wire Line
-	3300 4350 3300 4500
-Wire Wire Line
-	3450 4350 3450 4500
-Wire Wire Line
-	3450 4500 3400 4500
-Wire Wire Line
-	3500 4500 3500 4400
-Wire Wire Line
-	3500 4400 3600 4400
-Wire Wire Line
-	3600 4400 3600 4350
-Wire Wire Line
-	3750 4350 3750 4500
-Wire Wire Line
-	3750 4500 3600 4500
-Wire Wire Line
-	3600 5700 3600 6050
-Text Label 3600 6050 1    50   ~ 0
-FLASH_SO
 Wire Wire Line
 	3900 4350 3900 4800
-Text Label 3900 4750 1    50   ~ 0
-FLASH_SO
 $Comp
 L Device:Buzzer BZ1
@@
 Wire Wire Line
 	1800 2700 1600 2700
+$Comp
+L Memory_Flash:W25Q32JVSS U5
+U 1 1 5C51FC1A
+P 3000 5700
+F 0 "U5" H 3350 5300 50  0000 L CNN
+F 1 "W25Q128JVSIQ" H 2400 5350 50  0000 L CNN
+F 2 "Package_SO:SOIC-8_5.23x5.23mm_P1.27mm" H 3000 5100 50  0001 C CNN
+F 3 "https://datasheet.lcsc.com/szlcsc/Winbond-Elec-W25Q128JVSIQTR_C97521.pdf" H 3000 5700 50  0001 C CNN
+F 4 "C97521" H 3000 5700 50  0001 C CNN "LCSC Part"
+	1    3000 5700
+	-1   0    0    1
+$EndComp
+$Comp
+L power:GND #PWR?
+U 1 1 5C51FD2C
+P 3000 5200
+AR Path="/5C1D48B0/5C51FD2C" Ref="#PWR?"  Part="1"
+AR Path="/5C51FD2C" Ref="#PWR0171"  Part="1"
+F 0 "#PWR0171" H 3000 4950 50  0001 C CNN
+F 1 "GND" H 3005 5027 50  0000 C CNN
+F 2 "" H 3000 5200 50  0001 C CNN
+F 3 "" H 3000 5200 50  0001 C CNN
+	1    3000 5200
+	0    1    1    0
+$EndComp
+Wire Wire Line
+	3000 5200 3000 5300
+$Comp
+L power:+3.3V #PWR0172
+U 1 1 5C522E76
+P 3000 6200
+F 0 "#PWR0172" H 3000 6050 50  0001 C CNN
+F 1 "+3.3V" H 3015 6373 50  0000 C CNN
+F 2 "" H 3000 6200 50  0001 C CNN
+F 3 "" H 3000 6200 50  0001 C CNN
+	1    3000 6200
+	-1   0    0    1
+$EndComp
+Wire Wire Line
+	3000 6200 3000 6100
+Wire Wire Line
+	2500 5800 2100 5800
+Text Label 2100 5800 0    50   ~ 0
+FLASH_DO
+Wire Wire Line
+	3750 4350 3750 4800
+Text Label 3600 4800 1    50   ~ 0
+FLASH_CLK
+Text Label 3950 5600 2    50   ~ 0
+FLASH_CLK
+Wire Wire Line
+	3500 5600 3950 5600
+Wire Wire Line
+	3600 4350 3600 4800
+Text Label 3450 4800 1    50   ~ 0
+FLASH_CS
+Text Label 3950 5800 2    50   ~ 0
+FLASH_CS
+Wire Wire Line
+	3950 5800 3500 5800
+Wire Wire Line
+	3450 4350 3450 4800
+Wire Wire Line
+	3150 4350 3150 4800
+Text Label 3150 4800 1    50   ~ 0
+FLASH_IO3
+Text Label 2100 5500 0    50   ~ 0
+FLASH_IO3
+Wire Wire Line
+	2500 5500 2100 5500
+Wire Wire Line
+	2500 5600 2100 5600
+Text Label 2100 5600 0    50   ~ 0
+FLASH_IO2
+Text Label 3300 4800 1    50   ~ 0
+FLASH_IO2
+Wire Wire Line
+	3300 4350 3300 4800
+Text Label 3900 4800 1    50   ~ 0
+FLASH_DO
+Text Label 3750 4800 1    50   ~ 0
+FLASH_DI
+Text Label 2100 5900 0    50   ~ 0
+FLASH_DI
+Wire Wire Line
+	2100 5900 2500 5900
 $EndSCHEMATC
