File: pcbv2/badge2.sch (KiCad schematic (older format))
At the start: 23 parts, among them J1 SOICbite, J2 SAO_CONN, J3 USB_C_Receptacle_USB2.0, J4 Conn_01x08_Female, Q2 Si1308EDL, U3 E73-2G4M08S1C, U5 W25Q128JVSIQ

Commit message: fix(pcbv2): reconnect VUSB pin
also add decoupling cap on VUSB, as recommended in nRF reference design
Parts:
- added C3: 4.7uF, Capacitor_SMD:C_0603_1608Metric, symbol Device:C
Connections:
- wire segments 119 -> 125
Other:
- moved on the sheet: BTN6
Changed lines of the file:
@@
 L Switch:SW_Push BTN6
 U 1 1 5DB3D78E
-P 2000 2700
-F 0 "BTN6" H 2000 2985 50  0000 C CNN
-F 1 "RESET" H 2000 2894 50  0000 C CNN
-F 2 "Button_Switch_SMD:SW_SPST_PTS810" H 2000 2900 50  0001 C CNN
-F 3 "" H 2000 2900 50  0001 C CNN
-	1    2000 2700
+P 1900 2600
+F 0 "BTN6" H 1900 2885 50  0000 C CNN
+F 1 "RESET" H 1900 2794 50  0000 C CNN
+F 2 "Button_Switch_SMD:SW_SPST_PTS810" H 1900 2800 50  0001 C CNN
+F 3 "" H 1900 2800 50  0001 C CNN
+	1    1900 2600
 	1    0    0    -1
 $EndComp
-Wire Wire Line
-	2200 2700 2400 2700
 $Comp
 L power:GND #PWR0122
@@
 F 3 "" H 1600 2700 50  0001 C CNN
 	1    1600 2700
-	1    0    0    -1
+	0    1    1    0
 $EndComp
 Wire Wire Line
-	1800 2700 1600 2700
+	1700 2600 1600 2600
 $Comp
 L Memory_Flash:W25Q32JVSS U5
@@
 Wire Wire Line
 	2100 5900 2500 5900
+Text Label 2150 2850 0    50   ~ 0
+VBUS
+$Comp
+L Device:C C3
+U 1 1 5DA9540D
+P 1850 2850
+F 0 "C3" H 1965 2896 50  0000 L CNN
+F 1 "4.7uF" H 1965 2805 50  0000 L CNN
+F 2 "Capacitor_SMD:C_0603_1608Metric" H 1888 2700 50  0001 C CNN
+F 3 "~" H 1850 2850 50  0001 C CNN
+	1    1850 2850
+	0    1    1    0
+$EndComp
+Wire Wire Line
+	2200 2700 2400 2700
+Wire Wire Line
+	2100 2600 2200 2600
+Wire Wire Line
+	2200 2600 2200 2700
+Wire Wire Line
+	2000 2850 2400 2850
+Wire Wire Line
+	1700 2850 1600 2850
+Wire Wire Line
+	1600 2850 1600 2700
+Connection ~ 1600 2700
+Wire Wire Line
+	1600 2700 1600 2600
 $EndSCHEMATC

Commit message: feat(pcbv2): replace SAO footprint with the official one
also add a 3D model
Parts:
- J2: footprint Connector_PinSocket_2.54mm:PinSocket_2x03_P2.54mm_Vertical -> badge:Badgelife-SAOv169-BADGE-2x3; symbol Connector_Generic:Conn_02x03_Odd_Even -> badgelife_shitty_addon_v169bis:Badgelife_sao_connector_v169bis; Digikey Part (none) -> SFH11-NBPC-D03-ST-BK-ND
Changed lines of the file:
@@
 Wire Wire Line
 	7000 3050 7000 3450
-$Comp
-L Connector_Generic:Conn_02x03_Odd_Even J2
-U 1 1 5C4210C2
-P 7650 4650
-F 0 "J2" H 7700 4867 50  0000 C CNN
-F 1 "SAO_CONN" H 7700 4950 50  0000 C CNN
-F 2 "Connector_PinSocket_2.54mm:PinSocket_2x03_P2.54mm_Vertical" H 7650 4650 50  0001 C CNN
-F 3 "~" H 7650 4650 50  0001 C CNN
-	1    7650 4650
-	1    0    0    -1
-$EndComp
-$Comp
-L power:+3.3V #PWR0166
-U 1 1 5C4211E2
-P 7150 4550
-F 0 "#PWR0166" H 7150 4400 50  0001 C CNN
-F 1 "+3.3V" H 7165 4723 50  0000 C CNN
-F 2 "" H 7150 4550 50  0001 C CNN
-F 3 "" H 7150 4550 50  0001 C CNN
-	1    7150 4550
-	0    -1   -1   0
-$EndComp
-Wire Wire Line
-	7450 4550 7150 4550
-$Comp
-L power:GND #PWR0167
-U 1 1 5C42404A
-P 8150 4550
-F 0 "#PWR0167" H 8150 4300 50  0001 C CNN
-F 1 "GND" V 8155 4422 50  0000 R CNN
-F 2 "" H 8150 4550 50  0001 C CNN
-F 3 "" H 8150 4550 50  0001 C CNN
-	1    8150 4550
-	0    -1   -1   0
-$EndComp
-Wire Wire Line
-	7450 4650 7200 4650
-Text Label 7350 4650 2    50   ~ 0
+Text Label 8600 4500 2    50   ~ 0
 SDA
-Wire Wire Line
-	7950 4650 8200 4650
-Text Label 8050 4650 0    50   ~ 0
+Text Label 6700 4500 0    50   ~ 0
 SCL
 Wire Wire Line
@@
 	1750 1000 2050 1000
 Wire Wire Line
-	8150 4550 7950 4550
-Wire Wire Line
 	4950 4350 4950 4700
 Wire Wire Line
@@
 Text Label 4950 2000 1    50   ~ 0
 SAO_GPIO2
-Wire Wire Line
-	7000 4750 7450 4750
-Text Label 7000 4750 0    50   ~ 0
+Text Label 8600 4700 2    50   ~ 0
 SAO_GPIO1
-Text Label 8050 4750 0    50   ~ 0
+Text Label 6700 4700 0    50   ~ 0
 SAO_GPIO2
-Wire Wire Line
-	7950 4750 8450 4750
 Text Label 4800 4400 3    50   ~ 0
 SAO_GPIO1
@@
 Wire Wire Line
 	1600 2700 1600 2600
+$Comp
+L badgelife_shitty_addon_v169bis:Badgelife_sao_connector_v169bis J2
+U 1 1 5C4210C2
+P 7650 4500
+F 0 "J2" V 7229 4497 50  0000 C CNN
+F 1 "SAO_CONN" V 7300 4500 50  0000 C CNN
+F 2 "badge:Badgelife-SAOv169-BADGE-2x3" H 7650 4500 50  0001 C CNN
+F 3 "" H 7650 4500 50  0001 C CNN
+F 4 "SFH11-NBPC-D03-ST-BK-ND" H 7650 4500 50  0001 C CNN "Digikey Part"
+	1    7650 4500
+	0    1    1    0
+$EndComp
+$Comp
+L power:GND #PWR0167
+U 1 1 5C42404A
+P 7000 4300
+F 0 "#PWR0167" H 7000 4050 50  0001 C CNN
+F 1 "GND" V 7005 4172 50  0000 R CNN
+F 2 "" H 7000 4300 50  0001 C CNN
+F 3 "" H 7000 4300 50  0001 C CNN
+	1    7000 4300
+	0    1    1    0
+$EndComp
+$Comp
+L power:+3.3V #PWR0166
+U 1 1 5C4211E2
+P 8400 4300
+F 0 "#PWR0166" H 8400 4150 50  0001 C CNN
+F 1 "+3.3V" H 8415 4473 50  0000 C CNN
+F 2 "" H 8400 4300 50  0001 C CNN
+F 3 "" H 8400 4300 50  0001 C CNN
+	1    8400 4300
+	0    1    1    0
+$EndComp
+Wire Wire Line
+	8200 4700 8600 4700
+Wire Wire Line
+	8200 4500 8600 4500
+Wire Wire Line
+	7100 4700 6700 4700
+Wire Wire Line
+	7100 4500 6700 4500
+Wire Wire Line
+	7000 4300 7100 4300
+Wire Wire Line
+	8200 4300 8400 4300
 $EndSCHEMATC

Commit message: feat(pcbv2): add LCSC part# for USB Type C connector
Parts:
- J3: LCSC Part (none) -> C388659
Changed lines of the file:
@@
 F 2 "Connector_USB:USB_C_Receptacle_Amphenol_12401548E4-2A" H 1150 1450 50  0001 C CNN
 F 3 "https://www.usb.org/sites/default/files/documents/usb_type-c.zip" H 1150 1450 50  0001 C CNN
+F 4 "C388659" H 1000 1450 50  0001 C CNN "LCSC Part"
 	1    1000 1450
 	1    0    0    -1

Commit message: feat(pcbv2): add part numbers to schematics
mostly LCSC / Digikey. Some components still missing, will
add them soon.
Parts:
- J1: No Assembly (none) -> True
Changed lines of the file:
@@
 F 2 "SOICbite:SOIC_clipProgSmall" H 4600 900 50  0001 C CNN
 F 3 "~" H 4600 900 50  0001 C CNN
+F 4 "True" H 4600 900 50  0001 C CNN "No Assembly"
 	1    4600 900
 	1    0    0    -1

Commit message: feat(pcbv2): add BOM part numbers
most parts there there, still missing a few
Parts:
- C3: LCSC Part (none) -> C19666; Vendor (none) -> CL10A475KO8NNNC
- C40: LCSC Part (none) -> C19702; Vendor (none) -> CL10A106KP8NNNC
- D4, D5: value LED -> LED Green; LCSC Part (none) -> C72043
- D6: LCSC Part (none) -> C114585
- J4: value Conn_01x08_Female -> Conn_01x08_Female Through Hole Right Angle; LCSC Part (none) -> C225516; Vendor (none) -> A2541HWR-8P
- Q2: Digikey Part (none) -> SI1308EDL-T1-GE3CT-ND; LCSC Part (none) -> C150506
- R1: LCSC Part (none) -> C23186; Vendor (none) -> 0603WAF5101T5E
- R12: value 470R -> 4.7K
- R13: value 470R -> 4.7K; LCSC Part (none) -> C23162; Vendor (none) -> 0603WAF4701T5E
- U3: LCSC Part (none) -> C356849
Changed lines of the file:
@@
 F 2 "EBYTE:E73-2G4M08S1C" H 4600 3300 50  0001 C CNN
 F 3 "" H 4600 3300 50  0001 C CNN
+F 4 "C356849" H 4700 3250 50  0001 C CNN "LCSC Part"
 	1    4700 3250
 	1    0    0    -1
@@
 P 6100 4200
 F 0 "D5" V 6045 4278 50  0000 L CNN
-F 1 "LED" V 6136 4278 50  0000 L CNN
+F 1 "LED Green" V 6136 4278 50  0000 L CNN
 F 2 "LED_SMD:LED_0603_1608Metric" H 6100 4200 50  0001 C CNN
 F 3 "~" H 6100 4200 50  0001 C CNN
+F 4 "C72043" V 6100 4200 50  0001 C CNN "LCSC Part"
 	1    6100 4200
 	0    1    1    0
@@
 P 6100 4650
 F 0 "R13" H 6170 4696 50  0000 L CNN
-F 1 "470R" H 6170 4605 50  0000 L CNN
+F 1 "4.7K" H 6170 4605 50  0000 L CNN
 F 2 "Resistor_SMD:R_0603_1608Metric" V 6030 4650 50  0001 C CNN
 F 3 "~" H 6100 4650 50  0001 C CNN
+F 4 "C23162" H 6100 4650 50  0001 C CNN "LCSC Part"
+F 5 "0603WAF4701T5E" H 6100 4650 50  0001 C CNN "Vendor"
 	1    6100 4650
 	1    0    0    -1
@@
 P 1350 5150
 F 0 "D4" H 1342 4895 50  0000 C CNN
-F 1 "LED" H 1342 4986 50  0000 C CNN
+F 1 "LED Green" H 1342 4986 50  0000 C CNN
 F 2 "LED_SMD:LED_0603_1608Metric" H 1350 5150 50  0001 C CNN
 F 3 "~" H 1350 5150 50  0001 C CNN
+F 4 "C72043" H 1350 5150 50  0001 C CNN "LCSC Part"
 	1    1350 5150
 	-1   0    0    1
@@
 P 950 5150
 F 0 "R12" V 743 5150 50  0000 C CNN
-F 1 "470R" V 834 5150 50  0000 C CNN
+F 1 "4.7K" V 834 5150 50  0000 C CNN
 F 2 "Resistor_SMD:R_0603_1608Metric" V 880 5150 50  0001 C CNN
 F 3 "~" H 950 5150 50  0001 C CNN
@@
 F 2 "LED_SMD:LED_WS2812B_PLCC4_5.0x5.0mm_P3.2mm" H 4700 4900 50  0001 L TNN
 F 3 "https://cdn-shop.adafruit.com/datasheets/WS2812B.pdf" H 4750 4825 50  0001 L TNN
+F 4 "C114585" V 4650 5200 50  0001 C CNN "LCSC Part"
 	1    4650 5200
 	0    1    1    0
@@
 F 2 "Package_TO_SOT_SMD:SOT-323_SC-70" H 1500 7000 50  0001 C CNN
 F 3 "~" H 1300 6900 50  0001 C CNN
+F 4 "C150506" H 1300 6900 50  0001 C CNN "LCSC Part"
+F 5 "SI1308EDL-T1-GE3CT-ND" H 1300 6900 50  0001 C CNN "Digikey Part"
 	1    1300 6900
 	1    0    0    -1
@@
 F 2 "Capacitor_SMD:C_0603_1608Metric" H 1488 6050 50  0001 C CNN
 F 3 "~" H 1450 6200 50  0001 C CNN
+F 4 "C19702" H 1450 6200 50  0001 C CNN "LCSC Part"
+F 5 "CL10A106KP8NNNC" H 1450 6200 50  0001 C CNN "Vendor"
 	1    1450 6200
 	1    0    0    -1
@@
 F 2 "Resistor_SMD:R_0603_1608Metric" V 2130 1000 50  0001 C CNN
 F 3 "~" H 2200 1000 50  0001 C CNN
+F 4 "C23186" V 2200 1000 50  0001 C CNN "LCSC Part"
+F 5 "0603WAF5101T5E" V 2200 1000 50  0001 C CNN "Vendor"
 	1    2200 1000
 	0    1    1    0
@@
 P 7800 5500
 F 0 "J4" H 7828 5476 50  0000 L CNN
-F 1 "Conn_01x08_Female" H 7828 5385 50  0000 L CNN
+F 1 "Conn_01x08_Female Through Hole Right Angle" H 7828 5385 50  0000 L CNN
 F 2 "Connector_PinSocket_2.54mm:PinSocket_1x08_P2.54mm_Horizontal" H 7800 5500 50  0001 C CNN
 F 3 "~" H 7800 5500 50  0001 C CNN
+F 4 "C225516" H 7800 5500 50  0001 C CNN "LCSC Part"
+F 5 "A2541HWR-8P" H 7800 5500 50  0001 C CNN "Vendor"
 	1    7800 5500
 	1    0    0    -1
@@
 F 2 "Capacitor_SMD:C_0603_1608Metric" H 1888 2700 50  0001 C CNN
 F 3 "~" H 1850 2850 50  0001 C CNN
+F 4 "C19666" H 1850 2850 50  0001 C CNN "LCSC Part"
+F 5 "CL10A475KO8NNNC" H 1850 2850 50  0001 C CNN "Vendor"
 	1    1850 2850
 	0    1    1    0

Commit message: feat(pcbv2): add missing parts to BOM
Parts:
- BTN1, BTN2, BTN3, BTN4: LCSC Part (none) -> C406163; Vendor (none) -> TC-1102T-C
- BTN5: LCSC Part (none) -> C319406; Vendor (none) -> 1TS005A-2400-5001
- BTN6: Digikey Part (none) -> CKN10502CT-ND; LCSC Part (none) -> C221897; Vendor (none) -> PTS810SJS250SMTRLFS
- BZ1: Digikey Part (none) -> 1597-1244-ND; Vendor (none) -> Seeed Studio 316040001
Changed lines of the file:
@@
 F 2 "Connector_PinHeader_2.00mm:PinHeader_1x02_P2.00mm_Vertical" V 1725 6700 50  0001 C CNN
 F 3 "~" V 1725 6700 50  0001 C CNN
+F 4 "1597-1244-ND" H 1750 6600 50  0001 C CNN "Digikey Part"
+F 5 "Seeed Studio 316040001" H 1750 6600 50  0001 C CNN "Vendor"
 	1    1750 6600
 	1    0    0    -1
@@
 F 2 "Button_Switch_SMD:SW_Push_1P1T_NO_6x6mm_H9.5mm" H 6800 3650 50  0001 C CNN
 F 3 "" H 6800 3650 50  0001 C CNN
+F 4 "C406163" H 6800 3450 50  0001 C CNN "LCSC Part"
+F 5 "TC-1102T-C" H 6800 3450 50  0001 C CNN "Vendor"
 	1    6800 3450
 	1    0    0    -1
@@
 F 2 "Button_Switch_SMD:SW_Push_1P1T_NO_6x6mm_H9.5mm" H 6800 3250 50  0001 C CNN
 F 3 "" H 6800 3250 50  0001 C CNN
+F 4 "C406163" H 6800 3050 50  0001 C CNN "LCSC Part"
+F 5 "TC-1102T-C" H 6800 3050 50  0001 C CNN "Vendor"
 	1    6800 3050
 	1    0    0    -1
@@
 F 2 "Button_Switch_SMD:SW_Push_1P1T_NO_6x6mm_H9.5mm" H 6800 2850 50  0001 C CNN
 F 3 "" H 6800 2850 50  0001 C CNN
+F 4 "C406163" H 6800 2650 50  0001 C CNN "LCSC Part"
+F 5 "TC-1102T-C" H 6800 2650 50  0001 C CNN "Vendor"
 	1    6800 2650
 	1    0    0    -1
@@
 F 2 "Button_Switch_SMD:SW_Push_1P1T_NO_6x6mm_H9.5mm" H 6800 4050 50  0001 C CNN
 F 3 "" H 6800 4050 50  0001 C CNN
+F 4 "C406163" H 6800 3850 50  0001 C CNN "LCSC Part"
+F 5 "TC-1102T-C" H 6800 3850 50  0001 C CNN "Vendor"
 	1    6800 3850
 	1    0    0    -1
@@
 F 2 "Button_Switch_SMD:SW_Push_1P1T_NO_6x6mm_H9.5mm" H 2100 4450 50  0001 C CNN
 F 3 "" H 2100 4450 50  0001 C CNN
+F 4 "C319406" H 2100 4250 50  0001 C CNN "LCSC Part"
+F 5 "1TS005A-2400-5001" H 2100 4250 50  0001 C CNN "Vendor"
 	1    2100 4250
 	0    -1   -1   0
@@
 F 2 "Button_Switch_SMD:SW_SPST_PTS810" H 1900 2800 50  0001 C CNN
 F 3 "" H 1900 2800 50  0001 C CNN
+F 4 "C221897" H 1900 2600 50  0001 C CNN "LCSC Part"
+F 5 "PTS810SJS250SMTRLFS" H 1900 2600 50  0001 C CNN "Vendor"
+F 6 "CKN10502CT-ND" H 1900 2600 50  0001 C CNN "Digikey Part"
 	1    1900 2600
 	1    0    0    -1

Commit message: Added battery holders BOM data
Parts:
- U5: symbol Memory_Flash:W25Q32JVSS -> badge2-rescue:W25Q32JVSS-Memory_Flash
Changed lines of the file:
@@
 EESchema Schematic File Version 4
 LIBS:badge2-cache
-EELAYER 30 0
+EELAYER 26 0
 EELAYER END
 $Descr A4 11693 8268
@@
 	1700 2600 1600 2600
 $Comp
-L Memory_Flash:W25Q32JVSS U5
+L badge2-rescue:W25Q32JVSS-Memory_Flash U5
 U 1 1 5C51FC1A
 P 3000 5700

Commit message: fix(pcbv2): broken schematic symbols
Parts:
- U5: symbol badge2-rescue:W25Q32JVSS-Memory_Flash -> Memory_Flash:W25Q32JVSS
Changed lines of the file:
@@
 EESchema Schematic File Version 4
 LIBS:badge2-cache
-EELAYER 26 0
+EELAYER 30 0
 EELAYER END
 $Descr A4 11693 8268
@@
 	1700 2600 1600 2600
 $Comp
-L badge2-rescue:W25Q32JVSS-Memory_Flash U5
+L Memory_Flash:W25Q32JVSS U5
 U 1 1 5C51FC1A
 P 3000 5700
