File: pcbv2/badge2.sch (KiCad schematic (older format))
At the start: 24 parts, among them J1 SOICbite, J2 SAO_CONN, J3 USB_C_Receptacle_USB2.0, J4 Conn_01x08_Female Through Hol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, Q2 Si1308EDL, U3 E73-2G4M08S1C, U5 W25Q128JVSIQ

Commit message: feat(pcbv2): connect remaining pins of FM module
also remove unused MISO pin
Connections:
- net labels added: FM_GPIO1, FM_GPIO2, FM_~SEN
- net labels removed: MISO
- wire segments 125 -> 130
- no-connect marks 12 -> 11
Changed lines of the file:
@@
 L power:GND #PWR0101
 U 1 1 5C1F19F6
-P 4500 1600
-F 0 "#PWR0101" H 4500 1350 50  0001 C CNN
-F 1 "GND" H 4505 1427 50  0000 C CNN
-F 2 "" H 4500 1600 50  0001 C CNN
-F 3 "" H 4500 1600 50  0001 C CNN
-	1    4500 1600
-	0    -1   -1   0
+P 4500 1500
+F 0 "#PWR0101" H 4500 1250 50  0001 C CNN
+F 1 "GND" H 4505 1327 50  0000 C CNN
+F 2 "" H 4500 1500 50  0001 C CNN
+F 3 "" H 4500 1500 50  0001 C CNN
+	1    4500 1500
+	0    1    1    0
 $EndComp
 $Comp
@@
 L power:+3.3V #PWR0104
 U 1 1 5C1F1A95
-P 4650 1900
-F 0 "#PWR0104" H 4650 1750 50  0001 C CNN
-F 1 "+3.3V" H 4650 2050 50  0000 C CNN
-F 2 "" H 4650 1900 50  0001 C CNN
-F 3 "" H 4650 1900 50  0001 C CNN
-	1    4650 1900
+P 4650 1700
+F 0 "#PWR0104" H 4650 1550 50  0001 C CNN
+F 1 "+3.3V" H 4650 1850 50  0000 C CNN
+F 2 "" H 4650 1700 50  0001 C CNN
+F 3 "" H 4650 1700 50  0001 C CNN
+	1    4650 1700
 	1    0    0    -1
 $EndComp
@@
 Wire Wire Line
 	2400 3000 2250 3000
-Text Label 2300 3000 0    50   ~ 0
+Text Label 2250 3000 0    50   ~ 0
 D-
 Wire Wire Line
@@
 D+
 Wire Wire Line
-	4800 2050 4800 1700
-Wire Wire Line
 	5100 2050 5100 1700
 Wire Wire Line
 	5800 3900 6100 3900
-Text Label 5850 3900 0    50   ~ 0
+Text Label 6100 3900 2    50   ~ 0
 MOSI
-Text Label 4800 2000 1    50   ~ 0
-MISO
-Text Label 5100 2000 1    50   ~ 0
+Text Label 5100 1700 3    50   ~ 0
 SCLK
 Wire Wire Line
@@
 Wire Wire Line
 	2400 3600 2000 3600
-Text Label 2100 3600 0    50   ~ 0
+Text Label 2000 3600 0    50   ~ 0
 SWDIO
-Text Label 2050 3750 0    50   ~ 0
+Text Label 2000 3750 0    50   ~ 0
 SWDCLK
 Text Label 8700 2150 0    50   ~ 0
@@
 $EndComp
 Wire Wire Line
-	4650 1900 4650 2050
-Wire Wire Line
-	4500 1600 4500 2050
+	4650 1700 4650 2050
+Wire Wire Line
+	4500 1500 4500 2050
 Wire Wire Line
 	4350 1900 4350 2050
@@
 Wire Wire Line
 	5800 3750 6100 3750
-Text Label 5900 3600 0    50   ~ 0
+Text Label 6100 3600 2    50   ~ 0
 SCL
-Text Label 5900 3750 0    50   ~ 0
+Text Label 6100 3750 2    50   ~ 0
 SDA
 Wire Wire Line
 	5800 2700 6100 2700
-Text Label 5850 2700 0    50   ~ 0
+Text Label 6100 2700 2    50   ~ 0
 V_BAT
 Wire Wire Line
@@
 Wire Wire Line
 	1100 6900 800  6900
-Text Label 850  6900 0    50   ~ 0
+Text Label 800  6900 0    50   ~ 0
 VIBRATOR
 Wire Wire Line
@@
 Wire Wire Line
 	4900 1100 5250 1100
-Text Label 4950 900  0    50   ~ 0
+Text Label 5250 900  2    50   ~ 0
 SWDCLK
 Wire Wire Line
@@
 Wire Wire Line
 	5100 4350 5100 4700
-Text Label 4950 4350 3    50   ~ 0
+Text Label 4950 4700 1    50   ~ 0
 DISPDC
-Text Label 5100 4400 3    50   ~ 0
+Text Label 5100 4700 1    50   ~ 0
 DISPCS
 Wire Wire Line
@@
 Text Label 4350 4700 1    50   ~ 0
 DISPBUSY
-Text Label 4500 4650 1    50   ~ 0
+Text Label 4500 4700 1    50   ~ 0
 DISPRST
 Wire Wire Line
-	4950 2050 4950 1650
-Text Label 4950 2000 1    50   ~ 0
+	4950 2050 4950 1600
+Text Label 4950 1600 3    50   ~ 0
 SAO_GPIO2
 Text Label 8600 4700 2    50   ~ 0
@@
 Text Label 6700 4700 0    50   ~ 0
 SAO_GPIO2
-Text Label 4800 4400 3    50   ~ 0
+Text Label 4800 4800 1    50   ~ 0
 SAO_GPIO1
 Wire Wire Line
@@
 L power:GND #PWR0120
 U 1 1 5DB0509B
-P 7350 5300
-F 0 "#PWR0120" H 7350 5050 50  0001 C CNN
-F 1 "GND" V 7355 5172 50  0000 R CNN
-F 2 "" H 7350 5300 50  0001 C CNN
-F 3 "" H 7350 5300 50  0001 C CNN
-	1    7350 5300
-	0    1    1    0
-$EndComp
-Wire Wire Line
-	7600 5300 7350 5300
+P 7250 5300
+F 0 "#PWR0120" H 7250 5050 50  0001 C CNN
+F 1 "GND" V 7255 5172 50  0000 R CNN
+F 2 "" H 7250 5300 50  0001 C CNN
+F 3 "" H 7250 5300 50  0001 C CNN
+	1    7250 5300
+	0    1    1    0
+$EndComp
+Wire Wire Line
+	7600 5300 7250 5300
 $Comp
 L power:+3.3V #PWR0121
@@
 Wire Wire Line
 	7600 5200 7400 5200
-Text Label 7500 5400 2    50   ~ 0
+Text Label 7250 5400 0    50   ~ 0
 SDA
 Wire Wire Line
-	7600 5400 7350 5400
-Text Label 7350 5500 0    50   ~ 0
+	7600 5400 7250 5400
+Text Label 7250 5500 0    50   ~ 0
 SCL
 Wire Wire Line
-	7600 5500 7350 5500
+	7600 5500 7250 5500
 Wire Wire Line
 	5250 2050 5250 1700
-Text Label 5250 2000 1    50   ~ 0
+Text Label 7250 5700 0    50   ~ 0
 FM_~RST
-Text Label 7550 5700 2    50   ~ 0
-FM_~RST
-Wire Wire Line
-	7600 5700 7350 5700
-NoConn ~ 7600 5600
-NoConn ~ 7600 5800
-NoConn ~ 7600 5900
 $Comp
 L Switch:SW_Push BTN6
@@
 NoConn ~ 4400 900
 NoConn ~ 4650 6150
+Wire Wire Line
+	7250 5700 7600 5700
+Text Label 7250 5600 0    50   ~ 0
+FM_~SEN
+Wire Wire Line
+	7250 5600 7600 5600
+Text Label 7250 5800 0    50   ~ 0
+FM_GPIO1
+Text Label 7250 5900 0    50   ~ 0
+FM_GPIO2
+Wire Wire Line
+	7600 5900 7250 5900
+Wire Wire Line
+	7600 5800 7250 5800
+Text Label 4200 4800 1    50   ~ 0
+FM_~SEN
+Wire Wire Line
+	4200 4350 4200 4800
+Text Label 2000 3300 0    50   ~ 0
+FM_GPIO1
+Wire Wire Line
+	2400 3300 2000 3300
+Text Label 2000 3450 0    50   ~ 0
+FM_GPIO2
+Wire Wire Line
+	2400 3450 2000 3450
+NoConn ~ 2400 3900
+Text Label 5250 1700 3    50   ~ 0
+FM_~RST
+NoConn ~ 4800 2050
 $EndSCHEMATC

Commit message: fix(pcbv2): remove AMS1117-3.3 regulator
We already have RT9013-33GB that does the same.
This also fixes an issue where the power switch would not be able to cut USB/LiPo power.
Also move LiPo circuit into power schematic.
Changed lines of the file:
@@
 $Descr A4 11693 8268
 encoding utf-8
-Sheet 1 5
+Sheet 1 4
 Title ""
 Date ""
@@
 Wire Wire Line
 	4800 4350 4800 4800
-$Sheet
-S 9100 3100 950  350
-U 5D9D2F80
-F0 "LiPo" 50
-F1 "lipo.sch" 50
-$EndSheet
 Wire Wire Line
 	5800 3300 6500 3300

Commit message: fix(pcbv2): add pull-down resistor to vibration motor
This ensures the vibration motor doesn't randomally go start before the MCU configures the respective GPIO to output

The new resistor is R9
Parts:
- added R9: 10K, Resistor_SMD:R_0603_1608Metric, symbol Device:R
Connections:
- net GND: now also R9.2
- net VIBRATOR: now also R9.1
Changed lines of the file:
@@
 L power:GND #PWR0175
 U 1 1 5C567B60
-P 1400 7100
-F 0 "#PWR0175" H 1400 6850 50  0001 C CNN
-F 1 "GND" H 1405 6927 50  0000 C CNN
-F 2 "" H 1400 7100 50  0001 C CNN
-F 3 "" H 1400 7100 50  0001 C CNN
-	1    1400 7100
-	1    0    0    -1
-$EndComp
-Wire Wire Line
-	1100 6900 800  6900
-Text Label 800  6900 0    50   ~ 0
+P 1400 7350
+F 0 "#PWR0175" H 1400 7100 50  0001 C CNN
+F 1 "GND" H 1405 7177 50  0000 C CNN
+F 2 "" H 1400 7350 50  0001 C CNN
+F 3 "" H 1400 7350 50  0001 C CNN
+	1    1400 7350
+	1    0    0    -1
+$EndComp
+Wire Wire Line
+	1100 6900 950  6900
+Text Label 550  6900 0    50   ~ 0
 VIBRATOR
 Wire Wire Line
@@
 FM_~RST
 NoConn ~ 4800 2050
+$Comp
+L Device:R R9
+U 1 1 5DBF2958
+P 950 7150
+F 0 "R9" H 1020 7196 50  0000 L CNN
+F 1 "10K" H 1020 7105 50  0000 L CNN
+F 2 "Resistor_SMD:R_0603_1608Metric" V 880 7150 50  0001 C CNN
+F 3 "~" H 950 7150 50  0001 C CNN
+F 4 "C25804" H 950 7150 50  0001 C CNN "LCSC Part"
+F 5 "0603WAF1002T5E" H 950 7150 50  0001 C CNN "Vendor"
+	1    950  7150
+	1    0    0    -1
+$EndComp
+Wire Wire Line
+	950  7300 1400 7300
+Wire Wire Line
+	1400 7300 1400 7350
+Wire Wire Line
+	1400 7100 1400 7300
+Connection ~ 1400 7300
+Wire Wire Line
+	950  7000 950  6900
+Connection ~ 950  6900
+Wire Wire Line
+	950  6900 550  6900
 $EndSCHEMATC

Commit message: fix(pcbv2): change green LED resistors to 390ohm
4.7k caused them to be too dim
Parts:
- R12: value 4.7K -> 390R; LCSC Part (none) -> C23151; Vendor (none) -> 0603WAF3900T5E
- R13: value 4.7K -> 390R; LCSC Part C23162 -> C23151; Vendor 0603WAF4701T5E -> 0603WAF3900T5E
Changed lines of the file:
@@
 EESchema Schematic File Version 4
-LIBS:badge2-cache
 EELAYER 30 0
 EELAYER END
@@
 P 6100 4650
 F 0 "R13" H 6170 4696 50  0000 L CNN
-F 1 "4.7K" H 6170 4605 50  0000 L CNN
+F 1 "390R" H 6170 4605 50  0000 L CNN
 F 2 "Resistor_SMD:R_0603_1608Metric" V 6030 4650 50  0001 C CNN
 F 3 "~" H 6100 4650 50  0001 C CNN
-F 4 "C23162" H 6100 4650 50  0001 C CNN "LCSC Part"
-F 5 "0603WAF4701T5E" H 6100 4650 50  0001 C CNN "Vendor"
+F 4 "C23151" H 6100 4650 50  0001 C CNN "LCSC Part"
+F 5 "0603WAF3900T5E" H 6100 4650 50  0001 C CNN "Vendor"
 	1    6100 4650
 	1    0    0    -1
@@
 P 950 5150
 F 0 "R12" V 743 5150 50  0000 C CNN
-F 1 "4.7K" V 834 5150 50  0000 C CNN
+F 1 "390R" V 834 5150 50  0000 C CNN
 F 2 "Resistor_SMD:R_0603_1608Metric" V 880 5150 50  0001 C CNN
 F 3 "~" H 950 5150 50  0001 C CNN
+F 4 "C23151" V 950 5150 50  0001 C CNN "LCSC Part"
+F 5 "0603WAF3900T5E" V 950 5150 50  0001 C CNN "Vendor"
 	1    950  5150
 	0    1    1    0

Commit message: feat(pcbv2): add I2C pullup resistors
R6/R7, 10k ohm
Parts:
- added R6, R7: 10K, Resistor_SMD:R_0603_1608Metric, symbol Device:R
Connections:
- net +3V3: now also R6.2, R7.2
- net SCL: now also R6.1
- net SDA: now also R7.1
Other:
- note added: "I²C Pullups"
Changed lines of the file:
@@
 Wire Wire Line
 	950  6900 550  6900
+$Comp
+L Device:R R6
+U 1 1 5E0E6DE0
+P 6400 900
+AR Path="/5E0E6DE0" Ref="R6"  Part="1"
+F 0 "R6" V 6500 900 50  0000 L CNN
+F 1 "10K" V 6400 850 50  0000 L CNN
+F 2 "Resistor_SMD:R_0603_1608Metric" V 6330 900 50  0001 C CNN
+F 3 "~" H 6400 900 50  0001 C CNN
+F 4 "C25804" H 6400 900 50  0001 C CNN "LCSC Part"
+F 5 "0603WAF1002T5E" H 6400 900 50  0001 C CNN "Vendor"
+	1    6400 900
+	0    -1   -1   0
+$EndComp
+$Comp
+L Device:R R7
+U 1 1 5E0ECD1B
+P 6400 1100
+AR Path="/5E0ECD1B" Ref="R7"  Part="1"
+F 0 "R7" V 6500 1100 50  0000 L CNN
+F 1 "10K" V 6400 1050 50  0000 L CNN
+F 2 "Resistor_SMD:R_0603_1608Metric" V 6330 1100 50  0001 C CNN
+F 3 "~" H 6400 1100 50  0001 C CNN
+F 4 "C25804" H 6400 1100 50  0001 C CNN "LCSC Part"
+F 5 "0603WAF1002T5E" H 6400 1100 50  0001 C CNN "Vendor"
+	1    6400 1100
+	0    -1   -1   0
+$EndComp
+Text Label 6050 900  0    50   ~ 0
+SCL
+Text Label 6050 1100 0    50   ~ 0
+SDA
+Wire Wire Line
+	6250 900  6050 900
+Wire Wire Line
+	6050 1100 6250 1100
+$Comp
+L power:+3.3V #PWR02
+U 1 1 5E1052E7
+P 6700 1000
+F 0 "#PWR02" H 6700 850 50  0001 C CNN
+F 1 "+3.3V" H 6715 1173 50  0000 C CNN
+F 2 "" H 6700 1000 50  0001 C CNN
+F 3 "" H 6700 1000 50  0001 C CNN
+	1    6700 1000
+	0    1    1    0
+$EndComp
+Wire Wire Line
+	6550 900  6550 1000
+Wire Wire Line
+	6550 1000 6700 1000
+Wire Wire Line
+	6550 1000 6550 1100
+Connection ~ 6550 1000
+Text Notes 6200 700  0    50   ~ 0
+I²C Pullups
+Wire Notes Line
+	5900 550  7000 550
+Wire Notes Line
+	7000 550  7000 1200
+Wire Notes Line
+	7000 1200 5900 1200
+Wire Notes Line
+	5900 1200 5900 550
 $EndSCHEMATC

Commit message: Created a smaller hole diameter footprint for the buzzer, based on AWG 32 and 7 windes (like it says here - https://media.digikey.com/pdf/Data%20Sheets/Seeed%20Technology/1020-15-003-001_Spec.pdf). Hole size calculations were according to this - http://www.pcblibraries.com/downloads/temp/ANSI_Wire_Gauge_Charts_8646019.pdf
Parts:
- BZ1: footprint Connector_PinHeader_2.00mm:PinHeader_1x02_P2.00mm_Vertical -> buzzer:buzzer_footprint
- U5: symbol Memory_Flash:W25Q32JVSS -> badge2-rescue:W25Q32JVSS-Memory_Flash
Changed lines of the file:
@@
 F 0 "BZ1" H 1903 6629 50  0000 L CNN
 F 1 "Buzzer" H 1903 6538 50  0000 L CNN
-F 2 "Connector_PinHeader_2.00mm:PinHeader_1x02_P2.00mm_Vertical" V 1725 6700 50  0001 C CNN
+F 2 "buzzer:buzzer_footprint" V 1725 6700 50  0001 C CNN
 F 3 "~" V 1725 6700 50  0001 C CNN
 F 4 "1597-1244-ND" H 1750 6600 50  0001 C CNN "Digikey Part"
@@
 	1700 2600 1600 2600
 $Comp
-L Memory_Flash:W25Q32JVSS U5
+L badge2-rescue:W25Q32JVSS-Memory_Flash U5
 U 1 1 5C51FC1A
 P 3000 5700
@@
 U 1 1 5E0E6DE0
 P 6400 900
-AR Path="/5E0E6DE0" Ref="R6"  Part="1"
 F 0 "R6" V 6500 900 50  0000 L CNN
 F 1 "10K" V 6400 850 50  0000 L CNN
@@
 U 1 1 5E0ECD1B
 P 6400 1100
-AR Path="/5E0ECD1B" Ref="R7"  Part="1"
 F 0 "R7" V 6500 1100 50  0000 L CNN
 F 1 "10K" V 6400 1050 50  0000 L CNN

Commit message: Changed buttons to better match our needs, be cheaper and match footprint
Parts:
- BTN1, BTN2, BTN3, BTN4: LCSC Part C406163 -> C145890; Vendor TC-1102T-C -> K2-1102ST-A4SC-04
- BTN5: LCSC Part C319406 -> C223762; Vendor 1TS005A-2400-5001 -> K2-1102SP-B4SC-04
- U5: symbol badge2-rescue:W25Q32JVSS-Memory_Flash -> badge2-rescue:W25Q32JVSS-Memory_Flash-badge2-rescue
Changed lines of the file:
@@
 F 1 "DOWN" H 6800 3644 50  0000 C CNN
 F 2 "Button_Switch_SMD:SW_Push_1P1T_NO_6x6mm_H9.5mm" H 6800 3650 50  0001 C CNN
-F 3 "" H 6800 3650 50  0001 C CNN
-F 4 "C406163" H 6800 3450 50  0001 C CNN "LCSC Part"
-F 5 "TC-1102T-C" H 6800 3450 50  0001 C CNN "Vendor"
+F 3 "https://datasheet.lcsc.com/szlcsc/1809211434_Korean-Hroparts-Elec-K2-1102ST-A4SC-04_C145890.pdf" H 6800 3650 50  0001 C CNN
+F 4 "C145890" H 6800 3450 50  0001 C CNN "LCSC Part"
+F 5 "K2-1102ST-A4SC-04" H 6800 3450 50  0001 C CNN "Vendor"
 	1    6800 3450
 	1    0    0    -1
@@
 F 1 "LEFT" H 6800 3244 50  0000 C CNN
 F 2 "Button_Switch_SMD:SW_Push_1P1T_NO_6x6mm_H9.5mm" H 6800 3250 50  0001 C CNN
-F 3 "" H 6800 3250 50  0001 C CNN
-F 4 "C406163" H 6800 3050 50  0001 C CNN "LCSC Part"
-F 5 "TC-1102T-C" H 6800 3050 50  0001 C CNN "Vendor"
+F 3 "https://datasheet.lcsc.com/szlcsc/1809211434_Korean-Hroparts-Elec-K2-1102ST-A4SC-04_C145890.pdf" H 6800 3250 50  0001 C CNN
+F 4 "C145890" H 6800 3050 50  0001 C CNN "LCSC Part"
+F 5 "K2-1102ST-A4SC-04" H 6800 3050 50  0001 C CNN "Vendor"
 	1    6800 3050
 	1    0    0    -1
@@
 F 1 "TOP" H 6800 2844 50  0000 C CNN
 F 2 "Button_Switch_SMD:SW_Push_1P1T_NO_6x6mm_H9.5mm" H 6800 2850 50  0001 C CNN
-F 3 "" H 6800 2850 50  0001 C CNN
-F 4 "C406163" H 6800 2650 50  0001 C CNN "LCSC Part"
-F 5 "TC-1102T-C" H 6800 2650 50  0001 C CNN "Vendor"
+F 3 "https://datasheet.lcsc.com/szlcsc/1809211434_Korean-Hroparts-Elec-K2-1102ST-A4SC-04_C145890.pdf" H 6800 2850 50  0001 C CNN
+F 4 "C145890" H 6800 2650 50  0001 C CNN "LCSC Part"
+F 5 "K2-1102ST-A4SC-04" H 6800 2650 50  0001 C CNN "Vendor"
 	1    6800 2650
 	1    0    0    -1
@@
 F 1 "RIGHT" H 6800 4044 50  0000 C CNN
 F 2 "Button_Switch_SMD:SW_Push_1P1T_NO_6x6mm_H9.5mm" H 6800 4050 50  0001 C CNN
-F 3 "" H 6800 4050 50  0001 C CNN
-F 4 "C406163" H 6800 3850 50  0001 C CNN "LCSC Part"
-F 5 "TC-1102T-C" H 6800 3850 50  0001 C CNN "Vendor"
+F 3 "https://datasheet.lcsc.com/szlcsc/1809211434_Korean-Hroparts-Elec-K2-1102ST-A4SC-04_C145890.pdf" H 6800 4050 50  0001 C CNN
+F 4 "C145890" H 6800 3850 50  0001 C CNN "LCSC Part"
+F 5 "K2-1102ST-A4SC-04" H 6800 3850 50  0001 C CNN "Vendor"
 	1    6800 3850
 	1    0    0    -1
@@
 F 1 "ACTION" H 2100 4444 50  0000 C CNN
 F 2 "Button_Switch_SMD:SW_Push_1P1T_NO_6x6mm_H9.5mm" H 2100 4450 50  0001 C CNN
-F 3 "" H 2100 4450 50  0001 C CNN
-F 4 "C319406" H 2100 4250 50  0001 C CNN "LCSC Part"
-F 5 "1TS005A-2400-5001" H 2100 4250 50  0001 C CNN "Vendor"
+F 3 "https://datasheet.lcsc.com/szlcsc/1809211432_Korean-Hroparts-Elec-K2-1102SP-B4SC-04_C223762.pdf" H 2100 4450 50  0001 C CNN
+F 4 "C223762" H 2100 4250 50  0001 C CNN "LCSC Part"
+F 5 "K2-1102SP-B4SC-04" H 2100 4250 50  0001 C CNN "Vendor"
 	1    2100 4250
 	0    -1   -1   0
@@
 	1700 2600 1600 2600
 $Comp
-L badge2-rescue:W25Q32JVSS-Memory_Flash U5
+L badge2-rescue:W25Q32JVSS-Memory_Flash-badge2-rescue U5
 U 1 1 5C51FC1A
 P 3000 5700
