File: pcbv2/badge2.kicad_pcb (KiCad board)
At the start: 2 copper layers, 137.9 x 57.6 mm, 68 parts, among them J1 Conn_02x04_Counter_Clockwise, J2 SAO_CONN, J3 USB_C_Receptacle_USB2.0, J4 Conn_01x08_Female, J6 Conn_ARM_JTAG_SWD_10, J7 PFC24/0.5mm, Q1 Si1308EDL, Q2 Si1308EDL, SW4 SW_SPDT, U1 MCP73831-2-OT, U2 AMS1117-3.3, U3 E73-2G4M08S1C, U4 TPS610986DSET, U5 GD25Q16C, U6 PMPB15XP,115, U7 LIS2DH12TR, U8 RT9013-XXXB

Commit message: feat(pcbv2): move SOICbite, add reset to PCB
move SOICbite to the other side of the board, add reset button to the PCB,
start routing flash and power LED
Parts:
- added BTN6: RESET, Button_Switch_SMD:SW_SPST_PTS810, F.Cu at (162.0, 117.0)
- moved J1 136.6 mm to (273.6, 103.2), turned to 90 degrees
Routing:
- net +3V3: track 30.4 -> 47.7 mm
- net Net-(U3-Pad40): track 0.00 -> 17.0 mm
- net Net-(U3-Pad42): track 0.00 -> 16.4 mm
- net Net-(U3-Pad36): track 0.00 -> 16.4 mm
- net Net-(U3-Pad34): track 0.00 -> 15.6 mm
- net Net-(U3-Pad38): track 0.00 -> 13.1 mm
- net Net-(D5-Pad1): track 0.00 -> 9.05 mm
- net /FLASH_SO: track 0.00 -> 8.70 mm
- net Net-(BTN6-Pad2): track 0.00 -> 8.28 mm

Commit message: cleanup(pcbv2): remove Cortex-M connector
Parts:
- removed J6: Conn_ARM_JTAG_SWD_10, Connector_PinHeader_1.27mm:PinHeader_2x05_P1.27mm_Vertical_SMD
- J1: value Conn_02x04_Counter_Clockwise -> SOICbite

Commit message: feat(pcbv2): replace flash memory
Upgrade flash to 128MBit (16MByte):
GD25Q16C → W25Q128JVS

The new flash chip has a different package (SOIC-8  208-mil), so the PCB was updated with the new footprint
Parts:
- U5: value GD25Q16C -> W25Q128JVSIQ; footprint Package_SO:SOIC-8_3.9x4.9mm_P1.27mm -> Package_SO:SOIC-8_5.23x5.23mm_P1.27mm
Connections:
- net /FLASH_SO renamed /FLASH_DO
- net Net-(U3-Pad34) renamed /FLASH_DI
- net Net-(U3-Pad36) renamed /FLASH_CLK
- net Net-(U3-Pad38) renamed /FLASH_CS
- net Net-(U3-Pad40) renamed /FLASH_IO2
- net Net-(U3-Pad42) renamed /FLASH_IO3
Routing:
- net /FLASH_DI: track 15.6 -> 17.8 mm
- net /FLASH_CLK: track 16.4 -> 18.5 mm
- net /FLASH_IO3: track 16.4 -> 17.3 mm
- net /FLASH_IO2: track 17.0 -> 16.1 mm
- net /FLASH_DO: track 8.70 -> 7.81 mm

Commit message: fix(pcbv2): reconnect VUSB pin
also add decoupling cap on VUSB, as recommended in nRF reference design
Parts:
- added C3: 4.7uF, Capacitor_SMD:C_0603_1608Metric, F.Cu at (159.3, 108.6)
- moved U5 1.80 mm to (165.8, 108.0)
Connections:
- U3 pad 27: Net-(U3-Pad27) -> +5V
Routing:
- net /FLASH_DI: track 17.8 -> 0.00 mm
- net /FLASH_IO3: track 17.3 -> 0.44 mm
- net /FLASH_CLK: track 18.5 -> 2.07 mm
- net /FLASH_IO2: track 16.1 -> 6.69 mm
- net /FLASH_CS: track 12.8 -> 4.63 mm
- net /FLASH_DO: track 7.81 -> 0.00 mm
- net +5V: track 2.66 -> 5.32 mm

Commit message: feat(pcbv2): replace SAO footprint with the official one
also add a 3D model
Parts:
- J2: footprint Connector_PinSocket_2.54mm:PinSocket_2x03_P2.54mm_Vertical -> badge:Badgelife-SAOv169-BADGE-2x3
- moved C38 4.24 mm to (221.7, 101.7)
- moved C39 4.24 mm to (221.7, 99.8)
- moved U7 4.24 mm to (217.2, 101.1)
- moved J2 2.89 mm to (205.4, 101.2), turned to 180 degrees
Routing:
- net GND: track 18.5 -> 15.6 mm
- net +3V3: track 47.7 -> 47.2 mm

Commit message: fix(pcbv2): SAO orientation
Make it compatible with last year's badge
Parts:
- turned J2 to 0 degrees
Changed lines of the file:
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@@
   )
   (module badge:Badgelife-SAOv169-BADGE-2x3 (layer B.Cu)
-    (at 205.43 101.23 180)
+    (at 205.43 101.23)
     (descr "Through hole straight IDC box header, 2x03, 2.54mm pitch, double rows")
     (tags "Through hole IDC box header THT 2x03 2.54mm double row")
@@
       (effects (font (size 1 1) (thickness 0.15)) (justify mirror))
     )
-    (pad 2 thru_hole rect (at -2.48 -1.29 270) (size 1.7272 1.7272) (drill 1.016) (layers *.Cu *.Mask)
+    (pad 2 thru_hole rect (at -2.48 -1.29 90) (size 1.7272 1.7272) (drill 1.016) (layers *.Cu *.Mask)
       (net 1 GND))
-    (pad 1 thru_hole oval (at -2.48 1.25 270) (size 1.7272 1.7272) (drill 1.016) (layers *.Cu *.Mask)
+    (pad 1 thru_hole oval (at -2.48 1.25 90) (size 1.7272 1.7272) (drill 1.016) (layers *.Cu *.Mask)
       (net 2 +3V3))
-    (pad 4 thru_hole oval (at 0.06 -1.29 270) (size 1.7272 1.7272) (drill 1.016) (layers *.Cu *.Mask)
+    (pad 4 thru_hole oval (at 0.06 -1.29 90) (size 1.7272 1.7272) (drill 1.016) (layers *.Cu *.Mask)
       (net 40 /SCL))
-    (pad 3 thru_hole oval (at 0.06 1.25 270) (size 1.7272 1.7272) (drill 1.016) (layers *.Cu *.Mask)
+    (pad 3 thru_hole oval (at 0.06 1.25 90) (size 1.7272 1.7272) (drill 1.016) (layers *.Cu *.Mask)
       (net 39 /SDA))
-    (pad 6 thru_hole circle (at 2.6 -1.29 270) (size 1.7272 1.7272) (drill 1.016) (layers *.Cu *.Mask)
+    (pad 6 thru_hole circle (at 2.6 -1.29 90) (size 1.7272 1.7272) (drill 1.016) (layers *.Cu *.Mask)
       (net 63 /SAO_GPIO2))
-    (pad 5 thru_hole circle (at 2.6 1.25 270) (size 1.7272 1.7272) (drill 1.016) (layers *.Cu *.Mask)
+    (pad 5 thru_hole circle (at 2.6 1.25 90) (size 1.7272 1.7272) (drill 1.016) (layers *.Cu *.Mask)
       (net 62 /SAO_GPIO1))
     (model 3d-models/SFH11-xxPC-D03-ST-BK.STEP

Commit message: feat(pcbv2): add cross hole
Parts:
- added CROSS1: , badge:cross-u5, F.Cu at (249.7, 136.7)
