File: pcbv2/badge2.kicad_pcb (KiCad board)
At the start: 2 copper layers, 137.9 x 57.6 mm, 70 parts, among them J1 SOICbite, J2 SAO_CONN, J3 USB_C_Receptacle_USB2.0, J4 Conn_01x08_Female, J7 PFC24/0.5mm, Q1 Si1308EDL, Q2 Si1308EDL, SW4 SW_SPDT, U1 MCP73831-2-OT, U2 AMS1117-3.3, U3 E73-2G4M08S1C, U4 TPS610986DSET, U5 W25Q128JVSIQ, U6 PMPB15XP,115, U7 LIS2DH12TR, U8 RT9013-XXXB

Commit message: Placed new AAA and JST battery holders on PCB
Parts:
- removed BT1: Battery_Cell, AA_battery_clip:BK-53_MPD_AAClip
- removed BT2: Battery_Cell, Connector_JST:JST_EH_S2B-EH_1x02_P2.50mm_Horizontal
- added REF**: bcaaapc, bcaaapc:bcaaapc, F.Cu at (206.8, 146.8)
- added REF**: JST_PH_B2B-PH-K_02x2.00mm_Straight, jst:JST_PH_B2B-PH-K_02x2.00mm_Straight, F.Cu at (163.6, 146.6)

Commit message: fix(pcbv2): sync pcb with schematic
Parts:
- BT1: renamed from REF**; value bcaaapc -> Battery_Cell
- BT2: renamed from REF**; value JST_PH_B2B-PH-K_02x2.00mm_Straight -> Battery_Cell
- D10: value LED -> LED Red
- D4, D5: value LED -> LED Green
- J4: value Conn_01x08_Female -> Conn_01x08_Female Through Hole Right Angle
- J7: value PFC24/0.5mm -> FH12A-24S-0.5SH
- R12, R13: value 470R -> 4.7K
- U8: value RT9013-XXXB -> RT9013-33GB
Changed lines of the file:
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@@
-(kicad_pcb (version 20171130) (host pcbnew 5.0.2-bee76a0~70~ubuntu18.04.1)
+(kicad_pcb (version 20171130) (host pcbnew "(5.1.4)-1")
   (general
     (thickness 1.6)
@@
     (zone_45_only no)
     (trace_min 0.15)
-    (segment_width 0.2)
-    (edge_width 0.15)
     (via_size 0.8)
     (via_drill 0.4)
@@
     (uvia_min_size 0.2)
     (uvia_min_drill 0.1)
+    (edge_width 0.15)
+    (segment_width 0.2)
     (pcb_text_width 0.3)
     (pcb_text_size 1.5 1.5)
@@
       (effects (font (size 1 1) (thickness 0.15)))
     )
-    (fp_text value Conn_01x08_Female (at -4.38 20.55) (layer F.Fab)
+    (fp_text value "Conn_01x08_Female Through Hole Right Angle" (at -4.38 20.55) (layer F.Fab)
       (effects (font (size 1 1) (thickness 0.15)))
     )
@@
       (effects (font (size 1 1) (thickness 0.15)))
     )
-    (fp_text value RT9013-XXXB (at 0 2.9) (layer F.Fab)
+    (fp_text value RT9013-33GB (at 0 2.9) (layer F.Fab)
       (effects (font (size 1 1) (thickness 0.15)))
     )
@@
       (effects (font (size 1 1) (thickness 0.15)))
     )
-    (fp_text value LED (at 0 1.43) (layer F.Fab)
+    (fp_text value "LED Red" (at 0 1.43) (layer F.Fab)
       (effects (font (size 1 1) (thickness 0.15)))
     )
@@
       (effects (font (size 1 1) (thickness 0.15)))
     )
-    (fp_text value PFC24/0.5mm (at 0 5.6 90) (layer F.Fab)
+    (fp_text value FH12A-24S-0.5SH (at 0 5.6 90) (layer F.Fab)
       (effects (font (size 1 1) (thickness 0.15)))
     )
@@
       (effects (font (size 1 1) (thickness 0.15)))
     )
-    (fp_text value LED (at 0 1.43) (layer F.Fab)
+    (fp_text value "LED Green" (at 0 1.43) (layer F.Fab)
       (effects (font (size 1 1) (thickness 0.15)))
     )
@@
       (effects (font (size 1 1) (thickness 0.15)))
     )
-    (fp_text value LED (at 0 1.43 90) (layer F.Fab)
+    (fp_text value "LED Green" (at 0 1.43 90) (layer F.Fab)
       (effects (font (size 1 1) (thickness 0.15)))
     )
@@
       (effects (font (size 1 1) (thickness 0.15)))
     )
-    (fp_text value 470R (at 0 1.43) (layer F.Fab)
+    (fp_text value 4.7K (at 0 1.43) (layer F.Fab)
       (effects (font (size 1 1) (thickness 0.15)))
     )
@@
       (effects (font (size 1 1) (thickness 0.15)))
     )
-    (fp_text value 470R (at 0 1.43 90) (layer F.Fab)
+    (fp_text value 4.7K (at 0 1.43 90) (layer F.Fab)
       (effects (font (size 1 1) (thickness 0.15)))
     )
@@
   (module bcaaapc:bcaaapc (layer F.Cu)
     (at 206.75 146.85)
-    (fp_text reference REF** (at 0 0.5) (layer F.SilkS)
+    (fp_text reference BT1 (at 0 0.5) (layer F.SilkS)
       (effects (font (size 1 1) (thickness 0.15)))
     )
-    (fp_text value bcaaapc (at 0 -0.5) (layer F.Fab)
+    (fp_text value Battery_Cell (at 0 -0.5) (layer F.Fab)
       (effects (font (size 1 1) (thickness 0.15)))
     )
@@
     (descr "JST PH series connector, B2B-PH-K, top entry type, through hole, Datasheet: http://www.jst-mfg.com/product/pdf/eng/ePH.pdf")
     (tags "connector jst ph")
-    (fp_text reference REF** (at 1.5 -2.8) (layer F.SilkS)
+    (fp_text reference BT2 (at 1.5 -2.8) (layer F.SilkS)
       (effects (font (size 1 1) (thickness 0.15)))
     )
-    (fp_text value JST_PH_B2B-PH-K_02x2.00mm_Straight (at 1 3.8) (layer F.Fab)
+    (fp_text value Battery_Cell (at 1 3.8) (layer F.Fab)
       (effects (font (size 1 1) (thickness 0.15)))
     )
@@
     (pad 1 thru_hole rect (at 2 0) (size 1.2 1.7) (drill 0.75) (layers *.Cu *.Mask)
       (net 66 "Net-(BT2-Pad1)"))
-    (pad GND thru_hole oval (at 0 0) (size 1.2 1.7) (drill 0.75) (layers *.Cu *.Mask))
+    (pad 2 thru_hole oval (at 0 0) (size 1.2 1.7) (drill 0.75) (layers *.Cu *.Mask)
+      (net 1 GND))
     (model ${KISYS3DMOD}/Connectors_JST.3dshapes/JST_PH_B2B-PH-K_02x2.00mm_Straight.wrl
       (at (xyz 0 0 0))

Commit message: feat(pcbv2): wiring
Parts:
- removed C36: 1uF, Capacitor_SMD:C_0603_1608Metric
- removed C4: 100nF, Capacitor_SMD:C_0603_1608Metric
- removed U2: AMS1117-3.3, Package_TO_SOT_SMD:SOT-223-3_TabPin2
- moved D4 105.7 mm to (272.6, 135.6), turned to 90 degrees
- moved R12 101.5 mm to (272.6, 131.4), turned to 90 degrees
- moved U6 38.0 mm to (235.1, 145.9), turned to 90 degrees
- moved BZ1 35.3 mm to (182.7, 115.0)
- moved C40 35.3 mm to (180.2, 115.6)
- moved Q2 35.3 mm to (182.6, 111.3)
- moved C2 19.9 mm to (163.7, 139.9), turned to 270 degrees
- moved C16 18.9 mm to (204.2, 122.2)
- moved C37 18.9 mm to (196.7, 126.7)
- moved C12 18.9 mm to (200.7, 119.1)
- moved C6 18.9 mm to (193.6, 123.4)
- moved L2 18.9 mm to (208.5, 122.2)
- moved R14 18.9 mm to (201.4, 126.7)
- moved U4 18.9 mm to (199.9, 121.6)
- moved U8 11.8 mm to (166.6, 140.2), turned to 90 degrees
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Connections:
- net /MISO renamed Net-(U3-Pad17)
- C2 pad 1: +3V3 -> Net-(C2-Pad1)
- J4 pad 5: Net-(J4-Pad5) -> /FM_~SEN
- J4 pad 7: Net-(J4-Pad7) -> /FM_GPIO1
- J4 pad 8: Net-(J4-Pad8) -> /FM_GPIO2
- SW4 pad 3: Net-(C36-Pad2) -> Net-(C2-Pad1)
- U3 pad 28: Net-(U3-Pad28) -> /FM_~SEN
- U3 pad 33: Net-(U3-Pad33) -> /FM_GPIO1
- U3 pad 35: Net-(U3-Pad35) -> /FM_GPIO2
- U8 pad 5: +3V3 -> Net-(C2-Pad1)
Routing:
- net Net-(SW4-Pad1): track 0.99 -> 38.5 mm
- net +3V3: track 47.2 -> 74.9 mm
- net +5V: track 5.32 -> 28.7 mm
- net Net-(BT2-Pad1): track 0.00 -> 18.7 mm
- net Net-(R4-Pad1): track 0.00 -> 4.37 mm
- net Net-(BT1-Pad1): track 4.08 -> 7.82 mm
- net Net-(C2-Pad1): track 0.00 -> 3.61 mm
- net Net-(R3-Pad1): track 0.00 -> 3.52 mm
- net GND: track 15.6 -> 19.1 mm
- net Net-(D4-Pad2): track 2.63 -> 0.00 mm
- net Net-(D10-Pad1): track 0.00 -> 2.03 mm

Commit message: feat(pcbv2): even more wiring
Parts:
- moved C12 38.4 mm to (173.6, 146.3)
- moved L2 36.8 mm to (177.5, 141.9), turned to 180 degrees
- moved C16 34.5 mm to (178.2, 144.8), turned to 180 degrees
- moved U4 33.5 mm to (173.3, 141.9), turned to 180 degrees
- moved C6 29.8 mm to (170.5, 142.2)
- moved C37 26.9 mm to (173.1, 139.5)
- moved R14 26.5 mm to (178.1, 139.4), turned to 180 degrees
Routing:
- net Net-(C2-Pad1): track 3.61 -> 109.6 mm
- net /V_BAT: track 15.8 -> 98.7 mm
- net Net-(BTN4-Pad1): track 0.00 -> 48.5 mm, vias 0 -> 1
- net Net-(BTN2-Pad1): track 0.00 -> 33.6 mm, vias 0 -> 1
- net Net-(BTN3-Pad1): track 0.00 -> 27.8 mm, vias 0 -> 1
- net Net-(L2-Pad2): track 22.6 -> 2.19 mm, vias 2 -> 0
- net Net-(BTN1-Pad1): track 0.00 -> 17.4 mm, vias 0 -> 1
- net /SDA: track 0.00 -> 13.0 mm
- net /SCL: track 0.00 -> 11.5 mm
- net Net-(C37-Pad1): track 9.71 -> 5.40 mm
- net +3V3: track 74.9 -> 76.5 mm, vias 2 -> 4

Commit message: feat(pcbv2): finish wiring
Parts:
- moved C40 11.1 mm to (188.6, 108.4), turned to 180 degrees
- moved BZ1 7.05 mm to (185.2, 108.4), turned to 270 degrees
- moved C3 5.84 mm to (158.6, 114.4), turned to 0 degrees
- moved BTN6 4.37 mm to (164.1, 113.2), turned to 180 degrees
- moved Q2 4.19 mm to (179.6, 108.4), turned to 0 degrees
- moved U7 0.46 mm to (217.1, 101.5), turned to 0 degrees
Routing:
- net +3V3: track 76.5 -> 352.3 mm, vias 4 -> 7
- net /SDA: track 13.0 -> 150.9 mm, vias 0 -> 1
- net Net-(BTN5-Pad2): track 0.00 -> 125.3 mm, vias 0 -> 1
- net /SWDCLK: track 0.00 -> 119.3 mm, vias 0 -> 1
- net /SWDIO: track 0.00 -> 118.2 mm, vias 0 -> 1
- net /SCL: track 11.5 -> 128.0 mm, vias 0 -> 1
- net /FM_~RST: track 0.00 -> 113.2 mm, vias 0 -> 2
- net /MOSI: track 2.35 -> 115.0 mm, vias 1 -> 2
- net /FM_~SEN: track 0.00 -> 101.9 mm, vias 0 -> 1
- net /DISPBUSY: track 2.20 -> 103.8 mm, vias 1 -> 2
- net /DISPRST: track 0.00 -> 98.2 mm, vias 0 -> 2
- net /SCLK: track 1.95 -> 100.0 mm, vias 0 -> 2
- net /FM_GPIO1: track 0.00 -> 95.0 mm, vias 0 -> 1
- net /FM_GPIO2: track 0.00 -> 94.8 mm, vias 0 -> 1
- net /NEOPIXEL: track 0.00 -> 90.4 mm, vias 0 -> 1
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Other:
- board text added: "CHARGE"
- board text added: "POWER"

Commit message: fix(pcbv2): add pull-down resistor to vibration motor
This ensures the vibration motor doesn't randomally go start before the MCU configures the respective GPIO to output

The new resistor is R9
Parts:
- added R9: 10K, Resistor_SMD:R_0603_1608Metric, F.Cu at (175.8, 108.5)
Routing:
- net /VIBRATOR: track 33.7 -> 35.6 mm
Changed lines of the file:
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@@
     (thickness 1.6)
     (drawings 13)
-    (tracks 921)
+    (tracks 923)
     (zones 0)
-    (modules 67)
+    (modules 68)
     (nets 84)
   )
@@
   )
   (setup
-    (last_trace_width 0.4)
+    (last_trace_width 0.16)
     (user_trace_width 0.16)
     (user_trace_width 0.4)
@@
     (add_net "Net-(U8-Pad4)")
   )
+  (module Resistor_SMD:R_0603_1608Metric (layer F.Cu)
+    (at 175.768 108.4835 270)
+    (descr "Resistor SMD 0603 (1608 Metric), square (rectangular) end terminal, IPC_7351 nominal, (Body size source: http://www.tortai-tech.com/upload/download/2011102023233369053.pdf), generated with kicad-footprint-generator")
+    (tags resistor)
+    (attr smd)
+    (fp_text reference R9 (at -2.3115 0 180) (layer F.SilkS)
+      (effects (font (size 1 1) (thickness 0.15)))
+    )
+    (fp_text value 10K (at 0 1.43 90) (layer F.Fab)
+      (effects (font (size 1 1) (thickness 0.15)))
+    )
+    (fp_text user %R (at 0 0 90) (layer F.Fab)
+      (effects (font (size 0.4 0.4) (thickness 0.06)))
+    )
+    (fp_line (start 1.48 0.73) (end -1.48 0.73) (layer F.CrtYd) (width 0.05))
+    (fp_line (start 1.48 -0.73) (end 1.48 0.73) (layer F.CrtYd) (width 0.05))
+    (fp_line (start -1.48 -0.73) (end 1.48 -0.73) (layer F.CrtYd) (width 0.05))
+    (fp_line (start -1.48 0.73) (end -1.48 -0.73) (layer F.CrtYd) (width 0.05))
+    (fp_line (start -0.162779 0.51) (end 0.162779 0.51) (layer F.SilkS) (width 0.12))
+    (fp_line (start -0.162779 -0.51) (end 0.162779 -0.51) (layer F.SilkS) (width 0.12))
+    (fp_line (start 0.8 0.4) (end -0.8 0.4) (layer F.Fab) (width 0.1))
+    (fp_line (start 0.8 -0.4) (end 0.8 0.4) (layer F.Fab) (width 0.1))
+    (fp_line (start -0.8 -0.4) (end 0.8 -0.4) (layer F.Fab) (width 0.1))
+    (fp_line (start -0.8 0.4) (end -0.8 -0.4) (layer F.Fab) (width 0.1))
+    (pad 2 smd roundrect (at 0.7875 0 270) (size 0.875 0.95) (layers F.Cu F.Paste F.Mask) (roundrect_rratio 0.25)
+      (net 1 GND))
+    (pad 1 smd roundrect (at -0.7875 0 270) (size 0.875 0.95) (layers F.Cu F.Paste F.Mask) (roundrect_rratio 0.25)
+      (net 46 /VIBRATOR))
+    (model ${KISYS3DMOD}/Resistor_SMD.3dshapes/R_0603_1608Metric.wrl
+      (at (xyz 0 0 0))
+      (scale (xyz 1 1 1))
+      (rotate (xyz 0 0 0))
+    )
+  )
   (module EBYTE:E73-2G4M08S1C (layer F.Cu)
     (at 150.3 102.725)
@@
     (descr "Through hole straight pin header, 1x02, 2.00mm pitch, single row")
     (tags "Through hole pin header THT 1x02 2.00mm single row")
-    (fp_text reference BZ1 (at 0.0635 4.191 90) (layer F.SilkS)
+    (fp_text reference BZ1 (at -2.228 0.796 180) (layer F.SilkS)
       (effects (font (size 1 1) (thickness 0.15)))
     )
@@
       (effects (font (size 1 1) (thickness 0.15)))
     )
-    (fp_line (start -0.5 -1) (end 1 -1) (layer F.Fab) (width 0.1))
-    (fp_line (start 1 -1) (end 1 3) (layer F.Fab) (width 0.1))
-    (fp_line (start 1 3) (end -1 3) (layer F.Fab) (width 0.1))
-    (fp_line (start -1 3) (end -1 -0.5) (layer F.Fab) (width 0.1))
-    (fp_line (start -1 -0.5) (end -0.5 -1) (layer F.Fab) (width 0.1))
-    (fp_line (start -1.06 3.06) (end 1.06 3.06) (layer F.SilkS) (width 0.12))
-    (fp_line (start -1.06 1) (end -1.06 3.06) (layer F.SilkS) (width 0.12))
-    (fp_line (start 1.06 1) (end 1.06 3.06) (layer F.SilkS) (width 0.12))
-    (fp_line (start -1.06 1) (end 1.06 1) (layer F.SilkS) (width 0.12))
-    (fp_line (start -1.06 0) (end -1.06 -1.06) (layer F.SilkS) (width 0.12))
-    (fp_line (start -1.06 -1.06) (end 0 -1.06) (layer F.SilkS) (width 0.12))
-    (fp_line (start -1.5 -1.5) (end -1.5 3.5) (layer F.CrtYd) (width 0.05))
-    (fp_line (start -1.5 3.5) (end 1.5 3.5) (layer F.CrtYd) (width 0.05))
-    (fp_line (start 1.5 3.5) (end 1.5 -1.5) (layer F.CrtYd) (width 0.05))
-    (fp_line (start 1.5 -1.5) (end -1.5 -1.5) (layer F.CrtYd) (width 0.05))
     (fp_text user %R (at 0 1) (layer F.Fab)
       (effects (font (size 1 1) (thickness 0.15)))
     )
-    (pad 1 thru_hole rect (at 0 0 270) (size 1.35 1.35) (drill 0.8) (layers *.Cu *.Mask)
-      (net 2 +3V3))
+    (fp_line (start 1.5 -1.5) (end -1.5 -1.5) (layer F.CrtYd) (width 0.05))
+    (fp_line (start 1.5 3.5) (end 1.5 -1.5) (layer F.CrtYd) (width 0.05))
+    (fp_line (start -1.5 3.5) (end 1.5 3.5) (layer F.CrtYd) (width 0.05))
+    (fp_line (start -1.5 -1.5) (end -1.5 3.5) (layer F.CrtYd) (width 0.05))
+    (fp_line (start -1.06 -1.06) (end 0 -1.06) (layer F.SilkS) (width 0.12))
+    (fp_line (start -1.06 0) (end -1.06 -1.06) (layer F.SilkS) (width 0.12))
+    (fp_line (start -1.06 1) (end 1.06 1) (layer F.SilkS) (width 0.12))
+    (fp_line (start 1.06 1) (end 1.06 3.06) (layer F.SilkS) (width 0.12))
+    (fp_line (start -1.06 1) (end -1.06 3.06) (layer F.SilkS) (width 0.12))
+    (fp_line (start -1.06 3.06) (end 1.06 3.06) (layer F.SilkS) (width 0.12))
+    (fp_line (start -1 -0.5) (end -0.5 -1) (layer F.Fab) (width 0.1))
+    (fp_line (start -1 3) (end -1 -0.5) (layer F.Fab) (width 0.1))
+    (fp_line (start 1 3) (end -1 3) (layer F.Fab) (width 0.1))
+    (fp_line (start 1 -1) (end 1 3) (layer F.Fab) (width 0.1))
+    (fp_line (start -0.5 -1) (end 1 -1) (layer F.Fab) (width 0.1))
     (pad 2 thru_hole oval (at 0 2 270) (size 1.35 1.35) (drill 0.8) (layers *.Cu *.Mask)
       (net 42 "Net-(BZ1-Pad2)"))
+    (pad 1 thru_hole rect (at 0 0 270) (size 1.35 1.35) (drill 0.8) (layers *.Cu *.Mask)
+      (net 2 +3V3))
     (model ${KISYS3DMOD}/Connector_PinHeader_2.00mm.3dshapes/PinHeader_1x02_P2.00mm_Vertical.wrl
       (at (xyz 0 0 0))
@@
   (segment (start 177.3125 139.36) (end 174.0075 139.36) (width 0.25) (layer F.Cu) (net 44) (status 30))
   (segment (start 173.905 141.9) (end 176.1 141.9) (width 0.25) (layer F.Cu) (net 45) (status 30))
-  (via (at 177.5 107.3) (size 0.8) (drill 0.4) (layers F.Cu B.Cu) (net 46))
-  (segment (start 178.15 107.3) (end 178.6 107.75) (width 0.16) (layer F.Cu) (net 46))
-  (segment (start 177.5 107.3) (end 178.15 107.3) (width 0.16) (layer F.Cu) (net 46))
+  (via (at 177.5 107.3) (size 0.8) (drill 0.4) (layers F.Cu B.Cu) (net 46) (status 1000000))
   (segment (start 154.269 105.84) (end 153.042476 105.84) (width 0.16) (layer F.Cu) (net 46))
   (segment (start 153.042476 105.84) (end 152.828876 105.6264) (width 0.16) (layer F.Cu) (net 46))
@@
   (segment (start 152.828876 105.6264) (end 151.6736 105.6264) (width 0.16) (layer F.Cu) (net 46))
   (segment (start 151.6736 105.6264) (end 151.2 106.1) (width 0.16) (layer F.Cu) (net 46))
-  (segment (start 164.636014 107.3) (end 177.5 107.3) (width 0.16) (layer B.Cu) (net 46))
   (segment (start 161.448562 103.648562) (end 162.458522 104.658522) (width 0.16) (layer B.Cu) (net 46))
   (segment (start 151.2 106.1) (end 151.619991 105.680009) (width 0.16) (layer B.Cu) (net 46))
@@
   (segment (start 162.458522 105.122508) (end 164.636014 107.3) (width 0.16) (layer B.Cu) (net 46))
   (segment (start 155.568323 103.648562) (end 161.448562 103.648562) (width 0.16) (layer B.Cu) (net 46))
+  (segment (start 164.636014 107.3) (end 177.5 107.3) (width 0.16) (layer B.Cu) (net 46))
+  (segment (start 177.5 107.3) (end 178.15 107.3) (width 0.16) (layer F.Cu) (net 46))
+  (segment (start 178.15 107.3) (end 178.6 107.75) (width 0.16) (layer F.Cu) (net 46))
+  (segment (start 177.5 107.3) (end 176.164 107.3) (width 0.16) (layer F.Cu) (net 46))
+  (segment (start 176.164 107.3) (end 175.768 107.696) (width 0.16) (layer F.Cu) (net 46))
   (segment (start 236.61 144.98) (end 236.035 144.98) (width 0.4) (layer F.Cu) (net 47) (status 20))
   (segment (start 238.217796 143.372204) (end 236.61 144.98) (width 0.4) (layer F.Cu) (net 47))

Commit message: feat(pcbv2): improve LiPo charging circuit
Add a transistor (Q3), that cuts the power from the LiPo when USB is connected,
allowing us to separate the battery from the rest of the circuit
while it's being charged.
Parts:
- added D8: MBR0530, Diode_SMD:D_SOD-123, F.Cu at (159.8, 139.0)
- added Q3: Q_PMOS_DGS, Package_TO_SOT_SMD:SOT-23, F.Cu at (160.2, 142.2)
- added R5: 10K, Resistor_SMD:R_0603_1608Metric, F.Cu at (157.4, 143.1)
Connections:
- U8 pad 1: Net-(BT2-Pad1) -> Net-(D8-Pad1)
- U8 pad 3: Net-(BT2-Pad1) -> Net-(D8-Pad1)
Routing:
- net GND: track 78.5 -> 90.2 mm
- net Net-(D8-Pad1): track 0.00 -> 11.4 mm
- net +5V: track 66.5 -> 71.9 mm
- net Net-(BT2-Pad1): track 18.7 -> 13.4 mm
