File: pcbv2/badge2.kicad_pcb (KiCad board)
At the start: 2 copper layers, 137.9 x 57.6 mm, 71 parts, among them J1 SOICbite, J2 SAO_CONN, J3 USB_C_Receptacle_USB2.0, J4 Conn_01x08_Female Through Hol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, J7 FH12A-24S-0.5SH, Q1 Si1308EDL, Q2 Si1308EDL, Q3 Q_PMOS_DGS, SW4 SW_SPDT, U1 MCP73831-2-OT, U3 E73-2G4M08S1C, U4 TPS610986DSET, U5 W25Q128JVSIQ, U6 PMPB15XP,115, U7 LIS2DH12TR, U8 RT9013-33GB

Commit message: fix(pcbv2): mark AAA battery polarity on silk layer
Other:
- board text added: "-"
Changed lines of the file:
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@@
   (general
     (thickness 1.6)
-    (drawings 15)
+    (drawings 17)
     (tracks 996)
     (zones 0)
@@
       (net 1 GND))
   )
+  (gr_text - (at 187.05 146.65) (layer F.SilkS)
+    (effects (font (size 2.5 2.5) (thickness 0.2)))
+  )
+  (gr_text + (at 226.45 146.7) (layer F.SilkS)
+    (effects (font (size 2.5 2.5) (thickness 0.2)))
+  )
   (gr_text + (at 185.275 109.825) (layer F.SilkS)

Commit message: feat(pcbv2): add AAA/LiPo symbols next to power switch
Parts:
- added SYM1: Val**, badge:symbol-aaa, F.Cu at (266.0, 135.3)
- added SYM2: Val**, badge:symbol-lipo, F.Cu at (266.0, 151.4)

Commit message: fix(pcbv2): reverse polarity of LiPo connector
Parts:
- R12, R13: value 4.7K -> 390R
Routing:
- net GND: track 108.0 -> 111.5 mm
- net Net-(BT2-Pad1): track 11.5 -> 9.87 mm
Changed lines of the file:
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@@
     (thickness 1.6)
     (drawings 17)
-    (tracks 996)
+    (tracks 997)
     (zones 0)
     (modules 73)
@@
   )
   (setup
-    (last_trace_width 0.25)
+    (last_trace_width 0.4)
     (user_trace_width 0.16)
     (user_trace_width 0.4)
@@
     (descr "JST PH series connector, B2B-PH-K, top entry type, through hole, Datasheet: http://www.jst-mfg.com/product/pdf/eng/ePH.pdf")
     (tags "connector jst ph")
-    (fp_text reference BT2 (at 0.05 -3.1) (layer F.SilkS)
+    (fp_text reference BT2 (at 2.55 -2.95) (layer F.SilkS)
       (effects (font (size 1 1) (thickness 0.15)))
     )
@@
     (fp_line (start -2.05 2.9) (end 4.05 2.9) (layer F.SilkS) (width 0.12))
     (fp_line (start -2.05 -1.8) (end -2.05 2.9) (layer F.SilkS) (width 0.12))
-    (pad 1 thru_hole oval (at 2 0) (size 1.2 1.7) (drill 0.75) (layers *.Cu *.Mask)
-      (net 61 "Net-(BT2-Pad1)"))
-    (pad 2 thru_hole rect (at 0 0) (size 1.2 1.7) (drill 0.75) (layers *.Cu *.Mask)
+    (pad 2 thru_hole oval (at 2 0) (size 1.2 1.7) (drill 0.75) (layers *.Cu *.Mask)
       (net 1 GND))
+    (pad 1 thru_hole rect (at 0 0) (size 1.2 1.7) (drill 0.75) (layers *.Cu *.Mask)
+      (net 61 "Net-(BT2-Pad1)"))
     (model ${KISYS3DMOD}/Connectors_JST.3dshapes/JST_PH_B2B-PH-K_02x2.00mm_Straight.wrl
       (at (xyz 0 0 0))
@@
       (effects (font (size 1 1) (thickness 0.15)))
     )
-    (fp_text value 4.7K (at 0 1.43 90) (layer F.Fab)
+    (fp_text value 390R (at 0 1.43 90) (layer F.Fab)
       (effects (font (size 1 1) (thickness 0.15)))
     )
@@
       (effects (font (size 1 1) (thickness 0.15)))
     )
-    (fp_text value 4.7K (at 0 1.43 90) (layer F.Fab)
+    (fp_text value 390R (at 0 1.43 90) (layer F.Fab)
       (effects (font (size 1 1) (thickness 0.15)))
     )
@@
     (effects (font (size 1.5 1.5) (thickness 0.3)) (justify mirror))
   )
-  (gr_text + (at 165.875 143.825) (layer F.SilkS)
+  (gr_text + (at 163.2 143.55) (layer F.SilkS)
     (effects (font (size 1 1) (thickness 0.2)))
   )
@@
   (via (at 148.3 142.7) (size 0.8) (drill 0.4) (layers F.Cu B.Cu) (net 1))
   (via (at 148.3 152.1) (size 0.8) (drill 0.4) (layers F.Cu B.Cu) (net 1))
-  (segment (start 163.6 146.6) (end 158.4 146.6) (width 0.4) (layer F.Cu) (net 1))
-  (segment (start 158 146.2) (end 155.7 146.2) (width 0.4) (layer F.Cu) (net 1))
-  (segment (start 158.4 146.6) (end 158 146.2) (width 0.4) (layer F.Cu) (net 1))
   (via (at 272.1 110.4) (size 0.8) (drill 0.4) (layers F.Cu B.Cu) (net 1))
   (via (at 272.1 114) (size 0.8) (drill 0.4) (layers F.Cu B.Cu) (net 1))
@@
   (segment (start 148.4 104) (end 149.702499 105.302499) (width 0.16) (layer F.Cu) (net 60))
   (segment (start 149.702499 105.302499) (end 149.702499 109.966003) (width 0.16) (layer F.Cu) (net 60))
-  (segment (start 164.5 145.25) (end 165.6 146.35) (width 0.4) (layer F.Cu) (net 61))
-  (segment (start 165.6 146.35) (end 165.6 146.6) (width 0.4) (layer F.Cu) (net 61))
-  (segment (start 161.45 145.25) (end 161.65 145.25) (width 0.4) (layer F.Cu) (net 61))
-  (segment (start 161.65 145.25) (end 164.5 145.25) (width 0.4) (layer F.Cu) (net 61))
+  (segment (start 165.6 146.35) (end 165.6 146.6) (width 0.4) (layer F.Cu) (net 1))
+  (segment (start 159.650001 147.850001) (end 164.6 147.85) (width 0.4) (layer F.Cu) (net 1))
+  (segment (start 158 146.2) (end 159.650001 147.850001) (width 0.4) (layer F.Cu) (net 1))
+  (segment (start 165.6 146.85) (end 165.6 146.6) (width 0.4) (layer F.Cu) (net 1))
+  (segment (start 164.6 147.85) (end 165.6 146.85) (width 0.4) (layer F.Cu) (net 1))
+  (segment (start 155.7 146.2) (end 158 146.2) (width 0.4) (layer F.Cu) (net 1))
   (segment (start 161.3 145.25) (end 161.25 145.2) (width 0.4) (layer F.Cu) (net 61))
-  (segment (start 161.3 145.25) (end 161.65 145.25) (width 0.4) (layer F.Cu) (net 61))
   (segment (start 158.7 145.1) (end 158.85 145.25) (width 0.4) (layer F.Cu) (net 61))
   (segment (start 158.7 144.7) (end 158.7 145.1) (width 0.4) (layer F.Cu) (net 61))
   (segment (start 155.7 145.25) (end 158.85 145.25) (width 0.4) (layer F.Cu) (net 61))
   (segment (start 158.85 145.25) (end 161.3 145.25) (width 0.4) (layer F.Cu) (net 61))
+  (segment (start 163.5 145.25) (end 163.6 145.35) (width 0.4) (layer F.Cu) (net 61))
+  (segment (start 163.6 145.35) (end 163.6 146.6) (width 0.4) (layer F.Cu) (net 61))
+  (segment (start 161.3 145.25) (end 163.5 145.25) (width 0.4) (layer F.Cu) (net 61))
   (segment (start 157.3125 150) (end 155.2875 150) (width 0.16) (layer F.Cu) (net 62) (status 30))
   (segment (start 153.5 148.3875) (end 151.8875 150) (width 0.16) (layer F.Cu) (net 63) (status 20))

Commit message: cleanup(pcbv2): remove "Rev 1.0" text
Other:
- board text removed: "Rev 1.0"
Changed lines of the file:
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@@
   (general
     (thickness 1.6)
-    (drawings 17)
+    (drawings 16)
     (tracks 997)
     (zones 0)
@@
     (effects (font (size 1 1) (thickness 0.15)))
   )
-  (gr_text "Rev 1.0" (at 259 101.65) (layer F.SilkS)
-    (effects (font (size 1.5 1.5) (thickness 0.3)))
-  )
   (gr_text POWER (at 270.7 133.4 90) (layer F.SilkS)

Commit message: fix(pcbv2): sprinkle vias
also connect some ground island (according to kicad)
Routing:
- net GND: track 111.5 -> 165.5 mm, vias 62 -> 79
Changed lines of the file:
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@@
     (thickness 1.6)
     (drawings 16)
-    (tracks 997)
+    (tracks 1019)
     (zones 0)
     (modules 73)
@@
   (segment (start 164.6 147.85) (end 165.6 146.85) (width 0.4) (layer F.Cu) (net 1))
   (segment (start 155.7 146.2) (end 158 146.2) (width 0.4) (layer F.Cu) (net 1))
+  (via (at 252.65 132.4) (size 0.8) (drill 0.4) (layers F.Cu B.Cu) (net 1))
+  (via (at 258.7 132.5) (size 0.8) (drill 0.4) (layers F.Cu B.Cu) (net 1))
+  (via (at 265.4 132.6) (size 0.8) (drill 0.4) (layers F.Cu B.Cu) (net 1))
+  (via (at 265.65 136.85) (size 0.8) (drill 0.4) (layers F.Cu B.Cu) (net 1))
+  (via (at 259 136.75) (size 0.8) (drill 0.4) (layers F.Cu B.Cu) (net 1))
+  (via (at 252.2 136.3) (size 0.8) (drill 0.4) (layers F.Cu B.Cu) (net 1))
+  (via (at 226.35 137.1) (size 0.8) (drill 0.4) (layers F.Cu B.Cu) (net 1))
+  (via (at 217.8 137.1) (size 0.8) (drill 0.4) (layers F.Cu B.Cu) (net 1))
+  (via (at 208.6 137.2) (size 0.8) (drill 0.4) (layers F.Cu B.Cu) (net 1))
+  (via (at 200.35 137.1) (size 0.8) (drill 0.4) (layers F.Cu B.Cu) (net 1))
+  (via (at 193.2 137) (size 0.8) (drill 0.4) (layers F.Cu B.Cu) (net 1))
+  (via (at 185.65 136.35) (size 0.8) (drill 0.4) (layers F.Cu B.Cu) (net 1))
+  (via (at 189.4 132.5) (size 0.8) (drill 0.4) (layers F.Cu B.Cu) (net 1))
+  (via (at 196.6 132.6) (size 0.8) (drill 0.4) (layers F.Cu B.Cu) (net 1))
+  (via (at 204.95 133.25) (size 0.8) (drill 0.4) (layers F.Cu B.Cu) (net 1))
+  (via (at 213.1 133.65) (size 0.8) (drill 0.4) (layers F.Cu B.Cu) (net 1))
+  (via (at 221.85 133.25) (size 0.8) (drill 0.4) (layers F.Cu B.Cu) (net 1))
+  (segment (start 235.487999 148.012001) (end 185.669001 148.012001) (width 0.4) (layer F.Cu) (net 1))
+  (segment (start 236.035 147.465) (end 235.487999 148.012001) (width 0.4) (layer F.Cu) (net 1))
+  (segment (start 184.507 146.85) (end 183.345 146.85) (width 0.4) (layer F.Cu) (net 1))
+  (segment (start 185.669001 148.012001) (end 184.507 146.85) (width 0.4) (layer F.Cu) (net 1))
+  (segment (start 236.035 146.85) (end 236.035 147.465) (width 0.4) (layer F.Cu) (net 1))
   (segment (start 161.3 145.25) (end 161.25 145.2) (width 0.4) (layer F.Cu) (net 61))
   (segment (start 158.7 145.1) (end 158.85 145.25) (width 0.4) (layer F.Cu) (net 61))

Commit message: feat(pcbv2): add I2C pullup resistors
R6/R7, 10k ohm
Parts:
- added R6: 10K, Resistor_SMD:R_0603_1608Metric, F.Cu at (225.8, 100.8)
- added R7: 10K, Resistor_SMD:R_0603_1608Metric, F.Cu at (197.9, 105.3)
Routing:
- net /SDA: track 150.9 -> 158.6 mm
- net +3V3: track 352.9 -> 355.5 mm
- net GND: track 165.5 -> 166.7 mm, vias 79 -> 94
- net /SCL: track 128.0 -> 129.0 mm
