File: pcbv2/lipo.sch (KiCad schematic (older format))
At the start: 8 parts, among them U1 MCP73831-2-OT, U8 RT9013-XXXB

Commit message: feat(pcbv2): replace keyboard buttons with 6x6 buttons
Now we have 4 buttons: top/left/right/down instead of the 3 keyboard buttons we used to have
Parts:
- BT2: footprint (none) -> Connector_JST:JST_EH_S2B-EH_1x02_P2.50mm_Horizontal
Changed lines of the file:
@@
 F 0 "BT2" H 6768 3496 50  0000 L CNN
 F 1 "Battery_Cell" H 6768 3405 50  0000 L CNN
-F 2 "" V 6650 3460 50  0001 C CNN
+F 2 "Connector_JST:JST_EH_S2B-EH_1x02_P2.50mm_Horizontal" V 6650 3460 50  0001 C CNN
 F 3 "~" V 6650 3460 50  0001 C CNN
 	1    6650 3400

Commit message: feat(pcbv2): add BOM part numbers
most parts there there, still missing a few
Parts:
- D10: value LED -> LED Red; LCSC Part (none) -> C2286
- R3: LCSC Part (none) -> C22975; Vendor (none) -> 0603WAF2001T5E
- R4: LCSC Part (none) -> C23162; Vendor (none) -> 0603WAF4701T5E
- U1: LCSC Part (none) -> C14879; Vendor (none) -> MCP73831T-2ATI
- U8: value RT9013-XXXB -> RT9013-33GB; LCSC Part (none) -> C47773
Changed lines of the file:
@@
 F 2 "Package_TO_SOT_SMD:SOT-23-5" H 5800 3050 50  0001 L CIN
 F 3 "http://ww1.microchip.com/downloads/en/DeviceDoc/20001984g.pdf" H 5600 3250 50  0001 C CNN
+F 4 "C14879" H 5750 3300 50  0001 C CNN "LCSC Part"
+F 5 "MCP73831T-2ATI" H 5750 3300 50  0001 C CNN "Vendor"
 	1    5750 3300
 	1    0    0    -1
@@
 F 2 "Resistor_SMD:R_0603_1608Metric" V 5130 3550 50  0001 C CNN
 F 3 "~" H 5200 3550 50  0001 C CNN
+F 4 "C22975" H 5200 3550 50  0001 C CNN "LCSC Part"
+F 5 "0603WAF2001T5E" H 5200 3550 50  0001 C CNN "Vendor"
 	1    5200 3550
 	1    0    0    -1
@@
 F 2 "Resistor_SMD:R_0603_1608Metric" V 6230 3550 50  0001 C CNN
 F 3 "~" H 6300 3550 50  0001 C CNN
+F 4 "C23162" H 6300 3550 50  0001 C CNN "LCSC Part"
+F 5 "0603WAF4701T5E" H 6300 3550 50  0001 C CNN "Vendor"
 	1    6300 3550
 	1    0    0    -1
@@
 P 6300 4000
 F 0 "D10" V 6247 4078 50  0000 L CNN
-F 1 "LED" V 6338 4078 50  0000 L CNN
+F 1 "LED Red" V 6338 4078 50  0000 L CNN
 F 2 "LED_SMD:LED_0603_1608Metric" H 6300 4000 50  0001 C CNN
 F 3 "~" H 6300 4000 50  0001 C CNN
+F 4 "C2286" V 6300 4000 50  0001 C CNN "LCSC Part"
 	1    6300 4000
 	0    1    1    0
@@
 P 8000 3400
 F 0 "U8" H 8000 3886 59  0000 C CNN
-F 1 "RT9013-XXXB" H 8000 3781 59  0000 C CNN
+F 1 "RT9013-33GB" H 8000 3781 59  0000 C CNN
 F 2 "Package_TO_SOT_SMD:SOT-23-5" H 8000 3400 50  0001 C CNN
 F 3 "" H 8000 3400 50  0001 C CNN
+F 4 "C47773" H 8000 3400 50  0001 C CNN "LCSC Part"
 	1    8000 3400
 	1    0    0    -1

Commit message: Added battery holders BOM data
Parts:
- BT2: footprint Connector_JST:JST_EH_S2B-EH_1x02_P2.50mm_Horizontal -> jst:JST_PH_B2B-PH-K_02x2.00mm_Straight; Digikey Part (none) -> B2B-PH-K-S(LF)(SN)
- U8: symbol RT9013:RT9013-XXXB -> badge2-rescue:RT9013-XXXB-RT9013
Changed lines of the file:
@@
 EESchema Schematic File Version 4
 LIBS:badge2-cache
-EELAYER 30 0
+EELAYER 26 0
 EELAYER END
 $Descr A4 11693 8268
@@
 F 0 "BT2" H 6768 3496 50  0000 L CNN
 F 1 "Battery_Cell" H 6768 3405 50  0000 L CNN
-F 2 "Connector_JST:JST_EH_S2B-EH_1x02_P2.50mm_Horizontal" V 6650 3460 50  0001 C CNN
-F 3 "~" V 6650 3460 50  0001 C CNN
+F 2 "jst:JST_PH_B2B-PH-K_02x2.00mm_Straight" V 6650 3460 50  0001 C CNN
+F 3 "http://www.jst-mfg.com/product/pdf/eng/ePH.pdf" V 6650 3460 50  0001 C CNN
+F 4 "B2B-PH-K-S(LF)(SN)" H 6650 3400 50  0001 C CNN "Digikey Part"
 	1    6650 3400
 	1    0    0    -1
@@
 	6300 4150 6300 4350
 $Comp
-L RT9013:RT9013-XXXB U8
+L badge2-rescue:RT9013-XXXB-RT9013 U8
 U 1 1 5D9DA7E0
 P 8000 3400

Commit message: fix(pcbv2): broken schematic symbols
Parts:
- U8: symbol badge2-rescue:RT9013-XXXB-RT9013 -> RT9013:RT9013-XXXB
Changed lines of the file:
@@
 EESchema Schematic File Version 4
 LIBS:badge2-cache
-EELAYER 26 0
+EELAYER 30 0
 EELAYER END
 $Descr A4 11693 8268
@@
 	6300 4150 6300 4350
 $Comp
-L badge2-rescue:RT9013-XXXB-RT9013 U8
+L RT9013:RT9013-XXXB U8
 U 1 1 5D9DA7E0
 P 8000 3400
