File: pcbv2/Epaper.sch (KiCad schematic (older format))
At the start: 20 parts, among them J7 PFC24/0.5mm, Q1 Si1308EDL

Commit message: feat(pcbv2): add part numbers to schematics
mostly LCSC / Digikey. Some components still missing, will
add them soon.
Parts:
- C27: LCSC Part (none) -> C272771
- D1, D2, D3: LCSC Part (none) -> C77336
- J7: value PFC24/0.5mm -> FH12A-24S-0.5SH; Digikey Part (none) -> HFK24CT-ND; LCSC Part (none) -> C122394
- L1: LCSC Part (none) -> C295164; Vendor (none) -> NLV32T-680J-EF
Changed lines of the file:
@@
 F 2 "Diode_SMD:D_SOD-123" H 3500 2450 50  0001 C CNN
 F 3 "~" H 3500 2450 50  0001 C CNN
+F 4 "C77336" H 3500 2450 50  0001 C CNN "LCSC Part"
 	1    3500 2450
 	-1   0    0    1
@@
 F 2 "Diode_SMD:D_SOD-123" H 3600 2800 50  0001 C CNN
 F 3 "~" H 3600 2800 50  0001 C CNN
+F 4 "C77336" H 3600 2800 50  0001 C CNN "LCSC Part"
 	1    3600 2800
 	1    0    0    -1
@@
 F 2 "Diode_SMD:D_SOD-123" H 3550 3600 50  0001 C CNN
 F 3 "~" H 3550 3600 50  0001 C CNN
+F 4 "C77336" H 3550 3600 50  0001 C CNN "LCSC Part"
 	1    3550 3600
 	-1   0    0    1
@@
 F 2 "Inductor_SMD:L_1210_3225Metric" H 2500 3600 50  0001 C CNN
 F 3 "~" H 2500 3600 50  0001 C CNN
+F 4 "C295164" V 2500 3600 50  0001 C CNN "LCSC Part"
+F 5 "NLV32T-680J-EF" V 2500 3600 50  0001 C CNN "Vendor"
 	1    2500 3600
 	0    -1   -1   0
@@
 P 8100 3550
 F 0 "J7" H 8180 3542 50  0000 L CNN
-F 1 "PFC24/0.5mm" H 8180 3451 50  0000 L CNN
+F 1 "FH12A-24S-0.5SH" H 8180 3451 50  0000 L CNN
 F 2 "connectors:EPD-FPC-1x24-P0.50mm_Horizontal" H 8100 3550 50  0001 C CNN
 F 3 "~" H 8100 3550 50  0001 C CNN
+F 4 "HFK24CT-ND" H 8100 3550 50  0001 C CNN "Digikey Part"
+F 5 "C122394" H 8100 3550 50  0001 C CNN "LCSC Part"
 	1    8100 3550
 	1    0    0    -1
@@
 F 2 "Capacitor_SMD:C_0603_1608Metric" H 6538 3800 50  0001 C CNN
 F 3 "~" H 6500 3950 50  0001 C CNN
+F 4 "C272771" V 6500 3950 50  0001 C CNN "LCSC Part"
 	1    6500 3950
 	0    1    1    0

Commit message: feat(pcbv2): add BOM part numbers
most parts there there, still missing a few
Parts:
- C26: LCSC Part (none) -> C14663; Vendor (none) -> CC0603KRX7R9BB104
- C27: LCSC Part C272771 -> C15849; Vendor (none) -> CL10A105KB8NNNC
- Q1: Digikey Part (none) -> SI1308EDL-T1-GE3CT-ND; LCSC Part (none) -> C150506
- R10: LCSC Part (none) -> C25804; Vendor (none) -> 0603WAF1002T5E
- R11: LCSC Part (none) -> C23411; Vendor (none) -> 0603WAF470LT5E
Changed lines of the file:
@@
 F 2 "Package_TO_SOT_SMD:SOT-323_SC-70" H 3050 4850 50  0001 C CNN
 F 3 "~" H 2850 4750 50  0001 C CNN
+F 4 "C150506" H 2850 4750 50  0001 C CNN "LCSC Part"
+F 5 "SI1308EDL-T1-GE3CT-ND" H 2850 4750 50  0001 C CNN "Digikey Part"
 	1    2850 4750
 	1    0    0    -1
@@
 F 2 "Resistor_SMD:R_0603_1608Metric" V 2280 5600 50  0001 C CNN
 F 3 "~" H 2350 5600 50  0001 C CNN
+F 4 "C25804" H 2350 5600 50  0001 C CNN "LCSC Part"
+F 5 "0603WAF1002T5E" H 2350 5600 50  0001 C CNN "Vendor"
 	1    2350 5600
 	1    0    0    -1
@@
 F 2 "Resistor_SMD:R_0603_1608Metric" V 2880 5600 50  0001 C CNN
 F 3 "~" H 2950 5600 50  0001 C CNN
+F 4 "C23411" H 2950 5600 50  0001 C CNN "LCSC Part"
+F 5 "0603WAF470LT5E" H 2950 5600 50  0001 C CNN "Vendor"
 	1    2950 5600
 	1    0    0    -1
@@
 F 2 "Capacitor_SMD:C_0603_1608Metric" H 6538 3600 50  0001 C CNN
 F 3 "~" H 6500 3750 50  0001 C CNN
+F 4 "C14663" V 6500 3750 50  0001 C CNN "LCSC Part"
+F 5 "CC0603KRX7R9BB104" V 6500 3750 50  0001 C CNN "Vendor"
 	1    6500 3750
 	0    1    1    0
@@
 F 2 "Capacitor_SMD:C_0603_1608Metric" H 6538 3800 50  0001 C CNN
 F 3 "~" H 6500 3950 50  0001 C CNN
-F 4 "C272771" V 6500 3950 50  0001 C CNN "LCSC Part"
+F 4 "C15849" V 6500 3950 50  0001 C CNN "LCSC Part"
+F 5 "CL10A105KB8NNNC" V 6500 3950 50  0001 C CNN "Vendor"
 	1    6500 3950
 	0    1    1    0
