File: pcbv2/accelerometer.sch (KiCad schematic (older format))
At the start: 3 parts, among them U7 LIS2DH12TR

Commit message: feat(pcbv2): add part numbers to schematics
mostly LCSC / Digikey. Some components still missing, will
add them soon.
Parts:
- U7: Description (none) -> MEMS digital output motion sensor: ultra low-power high per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; Digikey Part (none) -> 497-14851-1-ND; Field4 LGA-12 STMicroelectronics -> (none); Field5 https://www.digikey.com/product-detail/en/stmicroelectronic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 -> (none); Field6 STMicroelectronics -> (none); Field7 LIS2DH12TR -> (none); Field8 MEMS digital output motion sensor: ultra low-power high per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 -> (none); LCSC Part (none) -> C110926
Changed lines of the file:
@@
 F 1 "LIS2DH12TR" H 8950 6079 50  0000 C CNN
 F 2 "Package_LGA:LGA-12_2x2mm_P0.5mm" H 8950 5400 50  0001 L BNN
-F 3 "497-14851-1-ND" H 8950 5400 50  0001 L BNN
-F 4 "LGA-12 STMicroelectronics" H 8950 5400 50  0001 L BNN "Field4"
-F 5 "https://www.digikey.com/product-detail/en/stmicroelectronics/LIS2DH12TR/497-14851-1-ND/4899838?utm_source=snapeda&utm_medium=aggregator&utm_campaign=symbol" H 8950 5400 50  0001 L BNN "Field5"
-F 6 "STMicroelectronics" H 8950 5400 50  0001 L BNN "Field6"
-F 7 "LIS2DH12TR" H 8950 5400 50  0001 L BNN "Field7"
-F 8 "MEMS digital output motion sensor: ultra low-power high performance 3-axes femto accelerometer" H 8950 5400 50  0001 L BNN "Field8"
+F 3 "~" H 8950 5400 50  0001 L BNN
+F 4 "497-14851-1-ND" H 8950 5400 50  0001 L BNN "Digikey Part"
+F 5 "MEMS digital output motion sensor: ultra low-power high performance 3-axes femto accelerometer" H 8950 5400 50  0001 L BNN "Description"
+F 6 "C110926" H 8950 5400 50  0001 C CNN "LCSC Part"
 	1    8950 5400
 	1    0    0    -1
