File: pcbv2/power.sch (KiCad schematic (older format))
At the start: 21 parts, among them Q3 Q_PMOS_DGS, SW4 SW_SPDT, U1 MCP73831-2-OT, U4 TPS610986DSET, U6 PMPB15XP,115, U8 RT9013-33GB

Commit message: doc(pcbv2): explain battery load sharing system
add link to the relevant application note from the schematic
Other:
- note added: "Battery Load Sharing System design based on Microchip's AN1149\nhttp://ww1.microchip.com/downloads/en/appnotes/01149c.pdf"
Changed lines of the file:
@@
 EESchema Schematic File Version 4
-LIBS:badge2-cache
 EELAYER 30 0
 EELAYER END
@@
 	0    1    1    0
 $EndComp
+Text Notes 4300 1650 0    50   ~ 0
+Battery Load Sharing System design based on Microchip's AN1149\nhttp://ww1.microchip.com/downloads/en/appnotes/01149c.pdf
+Wire Notes Line
+	4250 1450 6900 1450
+Wire Notes Line
+	6900 1450 6900 1700
+Wire Notes Line
+	6900 1700 4250 1700
+Wire Notes Line
+	4250 1700 4250 1450
 $EndSCHEMATC
